File: eaglecad/controller_rev3.brd (EAGLE design)
At the start: 30 x 50 mm, 91 parts, among them J1 1.27MM-SWD-CONNECTOR, U100 STM32F042K6, U101 TCAN330, U200 TPS63070, U300 STSPIN230, U301 TSV991ILT, U302 AS5047P, U400 STSPIN250, U401 TSV991ILT, X101 16MHZ-2.5x2mm

Commit message: part placement on rev3
Parts:
- moved C310 110.1 mm to (130.5, 25.9), flipped to the top
- moved C305 104.0 mm to (14.0, 28.4), flipped to the top, turned to 270 degrees
- moved R302 102.4 mm to (15.7, 28.3), flipped to the top
- moved C410 10.7 mm to (22.6, 34.2), flipped to the top
- moved R418 10.7 mm to (21.4, 31.4), turned to 270 degrees
- moved L201 9.86 mm to (2.30, 9.69), turned to 90 degrees
- moved C411 9.39 mm to (22.4, 31.4), turned to 90 degrees
- moved R419 9.39 mm to (25.5, 34.5), turned to 270 degrees
- moved C409 8.91 mm to (22.0, 32.9), flipped to the top, turned to 180 degrees
- moved C408 8.80 mm to (26.5, 32.3), turned to 90 degrees
- moved R417 8.77 mm to (22.9, 29.8), turned to 0 degrees
- moved EN 7.95 mm to (5.70, 15.1), flipped to the top, turned to 0 degrees
- moved U401 7.50 mm to (24.4, 31.9), turned to 270 degrees
- moved JP401 6.78 mm to (25.2, 12.7), turned to 0 degrees
- moved R410 6.48 mm to (23.5, 27.8), turned to 90 degrees
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
Commit message: rev 3 progress
Parts:
- removed JP101: (no value), pinhead:1X04
- added JP103: (no value), SparkFun-Connectors:6_PIN_SERIAL_TARGET_SIDE_W_SILK
- added JP301: (no value), pinhead-2:1X03M
- JP1: device pinhead:1X03 -> pinhead:1X02
- JP102: device SparkFun-Connectors:6_PIN_SERIAL_TARGET_SIDE_W_SILK -> pinhead:1X02
- moved R207 120.0 mm to (5.30, 14.1), flipped to the top
- moved C310 117.5 mm to (14.3, 44.0), flipped to the bottom
- moved C103 117.4 mm to (7.30, 28.1), turned to 270 degrees
- moved C101 110.0 mm to (6.10, 28.0), flipped to the top, turned to 90 degrees
- moved R315 108.2 mm to (16.2, 44.0), turned to 270 degrees
- moved U302 106.2 mm to (15.0, 27.0), turned to 270 degrees
- moved C102 101.8 mm to (15.0, 32.0), flipped to the top, turned to 180 degrees
- moved H1 99.7 mm to (48.9, 5.90)
- moved JP102 97.9 mm to (15.0, 5.70), turned to 0 degrees
- moved C105 87.2 mm to (27.7, 19.1), turned to 180 degrees
- moved X101 86.8 mm to (27.7, 21.2), turned to 90 degrees
- moved C104 86.7 mm to (27.6, 23.3), turned to 0 degrees
- moved 3.3V 39.8 mm to (-16.2, 26.2)
- moved C206 39.6 mm to (-19.1, 24.0), turned to 180 degrees
- moved C207 39.4 mm to (-19.1, 26.0)
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Connections:
- net CAN_H: now also JP102.1; no longer JP101.2
- net CAN_L: now also JP102.2; no longer JP101.3
- net GND: now also JP1.2, JP103.P$6; no longer JP101.4, JP102.P$6
- net PA2/USART2_TX: now also JP103.P$2; no longer JP102.P$2
- net PA3/USART2_RX: now also JP103.P$3; no longer JP102.P$3
- net TPS-FB: no longer PG.TP
- net TPS-PG: now also PG.TP
- net U: now also JP301.1; no longer JP1.1
- net V: now also JP301.2; no longer JP1.2
- net V_BATT: now also JP1.1, JP103.P$4; no longer JP101.1
- net W: now also JP301.3; no longer JP1.3
Routing:
- net OUT1: track 0.00 -> 12.4 mm, vias 0 -> 2
- net OUT2: track 0.00 -> 11.7 mm, vias 0 -> 2
- net SENSE_MAG: track 0.00 -> 9.81 mm, vias 0 -> 7
- net N$19: track 0.00 -> 9.64 mm
- net N$25: track 0.00 -> 9.43 mm
- net GND: track 1.49 -> 10.2 mm, vias 0 -> 14
- net U: track 9.33 -> 17.2 mm
- net N$8: track 0.00 -> 7.35 mm
- net N$27: track 0.00 -> 5.64 mm
- net V: track 7.52 -> 12.4 mm
- net W: track 8.47 -> 12.1 mm
- net N$15: track 0.00 -> 3.07 mm
- net N$17: track 0.00 -> 2.92 mm
- net 3.3V: track 0.00 -> 2.17 mm, vias 0 -> 3
- net N$2: track 0.00 -> 0.95 mm

Commit message: progress rev 3
Parts:
- moved C206 25.6 mm to (2.70, 10.5), flipped to the bottom
- moved C207 25.6 mm to (2.70, 12.5), flipped to the bottom
- moved 3.3V 23.8 mm to (1.80, 10.6)
- moved C205 22.8 mm to (2.50, 14.3), flipped to the bottom
- moved R205 21.7 mm to (4.81, 15.6), turned to 0 degrees
- moved FB2 20.7 mm to (1.80, 12.3)
- moved R206 19.0 mm to (3.30, 14.1), turned to 270 degrees
- moved R302 13.8 mm to (23.4, 27.4), turned to 0 degrees
- moved C305 13.0 mm to (21.5, 26.8), turned to 270 degrees
- moved R303 10.8 mm to (3.30, 22.7), turned to 180 degrees
- moved C302 9.41 mm to (3.40, 20.9), turned to 180 degrees
- moved C301 8.44 mm to (3.40, 19.4), turned to 180 degrees
- moved C303 7.65 mm to (3.40, 17.9), turned to 180 degrees
- moved R405 6.44 mm to (15.5, 18.0), turned to 90 degrees
- moved R406 6.44 mm to (14.5, 18.0)
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Routing:
- net CAN_H: track 0.00 -> 13.6 mm
- net PB1/INWL: track 0.00 -> 13.1 mm, vias 0 -> 2
- net PA7/INUL: track 0.00 -> 12.2 mm, vias 0 -> 2
- net CAN_L: track 0.00 -> 12.2 mm
- net PB0/INVL: track 0.00 -> 10.0 mm, vias 0 -> 2
- net TPS-VIN: track 0.00 -> 8.95 mm
- net PA8/INUH/PWM_MAG: track 0.00 -> 8.13 mm
- net CAN_RX: track 0.00 -> 7.60 mm
- net TPS-EN: track 0.00 -> 7.33 mm
- net TPS-FB: track 0.00 -> 7.10 mm
- net PA10/INWH: track 0.00 -> 6.30 mm
- net PA9/INVH/DIR_MAG: track 0.00 -> 6.21 mm
- net GND: track 10.2 -> 16.4 mm, vias 14 -> 36
- net PA15/CAN_SILENT: track 0.00 -> 6.15 mm, vias 0 -> 2
- net CAN_TX: track 0.00 -> 4.84 mm
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- added copper zone on layer 1, net TPS-L1
- added copper zone on layer 1, net TPS-L2

Commit message: rev3 needs design review
Parts:
- moved J1 100.9 mm to (33.9, 8.70), turned to 0 degrees
- moved JP302 85.4 mm to (32.5, 30.1), turned to 90 degrees
- moved JP103 74.2 mm to (36.3, 25.2)
- moved C103 21.3 mm to (25.2, 16.6), turned to 0 degrees
- moved C102 20.5 mm to (25.1, 21.8), flipped to the bottom, turned to 270 degrees
- moved BOOT 14.6 mm to (23.6, 18.8), flipped to the bottom
- moved C310 13.7 mm to (14.3, 25.8), turned to 0 degrees
- moved R101 12.1 mm to (23.2, 20.6), flipped to the bottom
- moved C106 11.1 mm to (13.4, 18.0), turned to 270 degrees
- moved C101 11.1 mm to (16.8, 25.1), turned to 270 degrees
- moved R315 9.78 mm to (15.6, 29.7), turned to 180 degrees
- moved C308 8.72 mm to (9.97, 27.9), turned to 180 degrees
- moved R308 8.51 mm to (7.70, 25.9), turned to 0 degrees
- moved C309 6.87 mm to (10.3, 29.1), turned to 0 degrees
- moved R314 6.33 mm to (9.30, 26.4), turned to 90 degrees
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Routing:
- net NRESET: track 0.00 -> 26.6 mm, vias 0 -> 1
- net SWCLK: track 0.00 -> 26.1 mm, vias 0 -> 2
- net PA1/CURR_FDB_BLDC: track 0.00 -> 23.7 mm
- net SWDIO: track 0.00 -> 22.9 mm, vias 0 -> 1
- net 3.3V: track 4.65 -> 26.7 mm, vias 6 -> 23
- net N$13: track 0.00 -> 19.3 mm
- net PB4/SPI1_MISO: track 0.00 -> 16.6 mm, vias 0 -> 3
- net N$4: track 0.00 -> 16.0 mm
- net PA4/FAULT_BLDC: track 0.00 -> 15.8 mm, vias 0 -> 2
- net SENSE_BLDC: track 0.00 -> 14.3 mm, vias 0 -> 7
- net GND: track 16.4 -> 29.5 mm, vias 36 -> 223
- net PA3/USART2_RX: track 0.00 -> 12.9 mm, vias 0 -> 1
- net PA5/SPI1_SCK: track 0.00 -> 12.3 mm, vias 0 -> 1
- net PA6/SPI1_NSS: track 0.00 -> 12.2 mm, vias 0 -> 1
- net PA2/USART2_TX: track 0.00 -> 11.9 mm, vias 0 -> 1
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- added copper zone on layer 1, net 3.3V
- added copper zone on layer 15, net 3.3V
- added copper zone on layer 16, net 3.3V
- added copper zone on layer 1, net GND
- added copper zone on layer 16, net GND
- added copper zone on layer 2, net GND
- added copper zone on layer 15, net V_BATT
Other:
- board size 30 x 50 mm -> 38 x 35 mm

Commit message: some more cleanup on rev 3
Parts:
- removed H1, H2, H3, H4: STAND-OFFTIGHT, SparkFun-Hardware:STAND-OFF-TIGHT
Routing:
- net GND: vias 223 -> 225
Changed lines of the file:
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@@
 <layer number="13" name="Route13" color="4" fill="5" visible="no" active="no"/>
 <layer number="14" name="Route14" color="1" fill="6" visible="no" active="no"/>
-<layer number="15" name="Route15" color="14" fill="1" visible="yes" active="yes"/>
+<layer number="15" name="Route15" color="14" fill="1" visible="no" active="yes"/>
 <layer number="16" name="Bottom" color="1" fill="1" visible="yes" active="yes"/>
 <layer number="17" name="Pads" color="2" fill="1" visible="yes" active="yes"/>
@@
 <layer number="28" name="bValues" color="7" fill="1" visible="no" active="yes"/>
 <layer number="29" name="tStop" color="7" fill="3" visible="no" active="yes"/>
-<layer number="30" name="bStop" color="7" fill="6" visible="yes" active="yes"/>
+<layer number="30" name="bStop" color="7" fill="6" visible="no" active="yes"/>
 <layer number="31" name="tCream" color="7" fill="4" visible="no" active="yes"/>
 <layer number="32" name="bCream" color="7" fill="5" visible="no" active="yes"/>
@@
 </element>
 <element name="U400" library="U-ST-STSPIN250-Brushed-DC-controller" package="VFQPN" value="STSPIN250" x="20.4" y="10.52"/>
-<element name="H1" library="SparkFun-Hardware" library_urn="urn:adsk.eagle:library:519" package="STAND-OFF-TIGHT" package3d_urn="urn:adsk.eagle:package:38629/1" value="STAND-OFFTIGHT" x="48.9" y="5.9" rot="R270"/>
-<element name="H2" library="SparkFun-Hardware" library_urn="urn:adsk.eagle:library:519" package="STAND-OFF-TIGHT" package3d_urn="urn:adsk.eagle:package:38629/1" value="STAND-OFFTIGHT" x="111" y="16.4"/>
-<element name="H3" library="SparkFun-Hardware" library_urn="urn:adsk.eagle:library:519" package="STAND-OFF-TIGHT" package3d_urn="urn:adsk.eagle:package:38629/1" value="STAND-OFFTIGHT" x="111" y="38.2" rot="R90"/>
-<element name="H4" library="SparkFun-Hardware" library_urn="urn:adsk.eagle:library:519" package="STAND-OFF-TIGHT" package3d_urn="urn:adsk.eagle:package:38629/1" value="STAND-OFFTIGHT" x="129.6" y="38.2" rot="R90"/>
 <element name="JP103" library="SparkFun-Connectors" library_urn="urn:adsk.eagle:library:513" package="6_PIN_SERIAL_TARGET_SIDE_W_SILK" package3d_urn="urn:adsk.eagle:package:37995/1" value="" x="36.3" y="25.2" rot="R90"/>
 <element name="JP401" library="pinhead" library_urn="urn:adsk.eagle:library:325" package="1X02" package3d_urn="urn:adsk.eagle:package:22435/2" value="" x="15" y="9.3" rot="R180"/>
@@
 <via x="28.2" y="21.7" extent="1-16" drill="0.254"/>
 <via x="28.9" y="20.9" extent="1-16" drill="0.254"/>
-<via x="29.2" y="19.6" extent="1-16" drill="0.254"/>
+<via x="29.23" y="19.6" extent="1-16" drill="0.254"/>
 <via x="26.5" y="17.2" extent="1-16" drill="0.254"/>
 <via x="26.5" y="16.6" extent="1-16" drill="0.254"/>
@@
 <via x="35" y="30" extent="1-16" drill="0.254"/>
 <via x="35" y="32.5" extent="1-16" drill="0.254"/>
+<via x="35.4" y="12.5" extent="1-16" drill="0.254"/>
+<via x="26.1" y="25.5" extent="1-16" drill="0.254"/>
 </signal>
 <signal name="CRYSTALIN">

Commit message: Rev 3 Ready for final sendout (Don't forget the stencils)
Parts:
- moved C401 0.40 mm to (21.0, 6.10)
- moved C402 0.40 mm to (22.5, 6.10)
- moved C403 0.40 mm to (24.0, 6.10)
- moved R403 0.40 mm to (19.2, 6.00)
- moved C207 0.30 mm to (2.70, 12.8)
- moved C205 0.30 mm to (2.50, 14.6)
Routing:
- net GND: track 29.5 -> 38.4 mm, vias 225 -> 207
- net 3.3V: track 26.7 -> 30.7 mm
- net SENSE_MAG: track 12.4 -> 8.67 mm, vias 7 -> 5
- net V_BATT: track 5.13 -> 2.46 mm, vias 15 -> 12
- net OUT2: track 11.7 -> 13.7 mm
- net SENSE_BLDC: track 14.3 -> 13.3 mm, vias 7 -> 5
- net OUT1: track 12.4 -> 12.7 mm, vias 2 -> 1
- added copper zone on layer 1, net SENSE_BLDC
- added copper zone on layer 16, net SENSE_BLDC
- added copper zone on layer 1, net SENSE_MAG
- added copper zone on layer 16, net SENSE_MAG
- added copper zone on layer 1, net V_BATT
