File: eaglecad/controller_rev4.sch (EAGLE design)
At the start: 91 parts, among them J1 1.27MM-SWD-CONNECTOR, U101 TCAN330, U200 TPS63070, U300 STSPIN230, U301 TSV991ILT, U302 AS5047P, U400 STSPIN250, U401 TSV991ILT, X101 16MHZ-2.5x2mm

Commit message: f4 updates
Connections:
- removed net CRYSTALIN: C105.1, X101.1
- removed net CRYSTALOUT: C104.1, X101.2
- new net N$1: C104.2, U$1.PH0-OSC_IN, X101.2
- new net N$4: C105.2, U$1.PH1-OSC_OUT, X101.1
- net 3.3V: now also U$1.VBAT, U$1.VDD, U$1.VDDA/VREF+
- net BOOT: now also U$1.BOOT0
- net CAN_RX: now also U$1.PA11
- net CAN_TX: now also U$1.PA12
- net GND: now also C104.1, C105.1, U$1.VSS, U$1.VSSA/VREF-; no longer C104.2, C105.2
- net NRESET: now also U$1.NRST
- net PA15/CAN_SILENT: now also U$1.PA15
- net PA2/USART2_TX: now also U$1.PA0
- net PA3/USART2_RX: now also U$1.PA1
- net SWCLK: now also U$1.PA14
- net SWDIO: now also U$1.PA13
Other:
- note removed: "Change to 3 pin for final rev"
- note removed: "Place on breakoff"
- moved on the sheet: BOOT, C101, C102, C103, C104, C105, C106, J1, JP1, JP102, JP103, R101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

Commit message: F4 updates
Parts:
- added C107: 2.2u, rcl_custom:C-EU0402-B-NOSILK
Connections:
- new net N$6: C107.2, U$1.VCAP_1
- net GND: now also C107.1
Changed lines of the file:
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@@
 <part name="TP3" library="testpad" library_urn="urn:adsk.eagle:library:385" deviceset="TP" device="TP06R" package3d_urn="urn:adsk.eagle:package:27954/1"/>
 <part name="U$1" library="oresat-misc" deviceset="STM32F446X" device=""/>
+<part name="C107" library="rcl_custom" deviceset="C-EU" device="0402-B-NOSILK" value="2.2u">
+<attribute name="DIS" value="Digi-Key"/>
+<attribute name="DPN" value="1276-1001-1-ND"/>
+<attribute name="MFR" value="Samsung"/>
+<attribute name="MPN" value="CL05B104KO5NNNC"/>
+</part>
 </parts>
 <sheets>
@@
 </instance>
 <instance part="U$1" gate="G$1" x="243.84" y="83.82" smashed="yes"/>
+<instance part="C107" gate="CE" x="210.82" y="114.3" smashed="yes" rot="R90">
+<attribute name="DIS" x="210.82" y="114.3" size="1.778" layer="96" rot="R90" display="off"/>
+<attribute name="DPN" x="210.82" y="114.3" size="1.778" layer="96" rot="R90" display="off"/>
+<attribute name="MFR" x="210.82" y="114.3" size="1.778" layer="96" rot="R90" display="off"/>
+<attribute name="MPN" x="210.82" y="114.3" size="1.778" layer="96" rot="R90" display="off"/>
+<attribute name="NAME" x="210.566" y="115.189" size="1.778" layer="95" rot="MR0"/>
+<attribute name="VALUE" x="213.614" y="115.189" size="1.778" layer="96"/>
+</instance>
 </instances>
 <busses>
@@
 <wire x1="208.28" y1="104.14" x2="205.74" y2="104.14" width="0.1524" layer="91"/>
 <wire x1="205.74" y1="104.14" x2="205.74" y2="101.6" width="0.1524" layer="91"/>
+<pinref part="C107" gate="CE" pin="1"/>
+<wire x1="208.28" y1="114.3" x2="205.74" y2="114.3" width="0.1524" layer="91"/>
+<wire x1="205.74" y1="114.3" x2="205.74" y2="104.14" width="0.1524" layer="91"/>
+<junction x="205.74" y="104.14"/>
 </segment>
 <segment>
@@
 </segment>
 </net>
+<net name="N$6" class="0">
+<segment>
+<pinref part="U$1" gate="G$1" pin="VCAP_1"/>
+<pinref part="C107" gate="CE" pin="2"/>
+<wire x1="215.9" y1="114.3" x2="220.98" y2="114.3" width="0.1524" layer="91"/>
+</segment>
+</net>

Commit message: F4 uPdateS
Parts:
- added C304, C404: 1n, rcl_custom:C-EU0402-B-NOSILK
- added R301, R401: 18k, rcl_custom:R-US_0402-B-NOSILK
Connections:
- net 3.3V: now also R301.1, R401.1
- net GND: now also C304.1, C404.1
- net STBY/RESET_BLDC: now also C304.2, R301.2
- net STBY/RESET_MAG: now also C404.2, R401.2
Changed lines of the file:
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@@
 <attribute name="MPN" value="CL05B104KO5NNNC"/>
 </part>
+<part name="R301" library="rcl_custom" deviceset="R-US_" device="0402-B-NOSILK" value="18k">
+<attribute name="DIS" value="Digi-Key"/>
+<attribute name="DPN" value="1276-4275-1-ND"/>
+<attribute name="MFR" value="Samsung"/>
+<attribute name="MPN" value="RC1005F6653CS"/>
+</part>
+<part name="C304" library="rcl_custom" deviceset="C-EU" device="0402-B-NOSILK" value="1n">
+<attribute name="DIS" value="Digi-Key"/>
+<attribute name="DPN" value="1276-1001-1-ND"/>
+<attribute name="MFR" value="Samsung"/>
+<attribute name="MPN" value="CL05B104KO5NNNC"/>
+</part>
+<part name="GND7" library="supply1" library_urn="urn:adsk.eagle:library:371" deviceset="GND" device=""/>
+<part name="SUPPLY5" library="SparkFun-PowerSymbols" library_urn="urn:adsk.eagle:library:530" deviceset="3.3V" device=""/>
+<part name="R401" library="rcl_custom" deviceset="R-US_" device="0402-B-NOSILK" value="18k">
+<attribute name="DIS" value="Digi-Key"/>
+<attribute name="DPN" value="1276-4275-1-ND"/>
+<attribute name="MFR" value="Samsung"/>
+<attribute name="MPN" value="RC1005F6653CS"/>
+</part>
+<part name="C404" library="rcl_custom" deviceset="C-EU" device="0402-B-NOSILK" value="1n">
+<attribute name="DIS" value="Digi-Key"/>
+<attribute name="DPN" value="1276-1001-1-ND"/>
+<attribute name="MFR" value="Samsung"/>
+<attribute name="MPN" value="CL05B104KO5NNNC"/>
+</part>
+<part name="GND8" library="supply1" library_urn="urn:adsk.eagle:library:371" deviceset="GND" device=""/>
+<part name="SUPPLY8" library="SparkFun-PowerSymbols" library_urn="urn:adsk.eagle:library:530" deviceset="3.3V" device=""/>
 </parts>
 <sheets>
@@
 <attribute name="TP_SIGNAL_NAME" x="90.17" y="217.17" size="1.778" layer="97"/>
 </instance>
+<instance part="R301" gate="R" x="119.38" y="220.98" smashed="yes" rot="R270">
+<attribute name="DIS" x="119.38" y="220.98" size="1.778" layer="96" rot="R270" display="off"/>
+<attribute name="DPN" x="119.38" y="220.98" size="1.778" layer="96" rot="R270" display="off"/>
+<attribute name="MFR" x="119.38" y="220.98" size="1.778" layer="96" rot="R270" display="off"/>
+<attribute name="MPN" x="119.38" y="220.98" size="1.778" layer="96" rot="R270" display="off"/>
+<attribute name="NAME" x="120.8786" y="224.79" size="1.778" layer="95" rot="R270"/>
+<attribute name="VALUE" x="116.078" y="224.79" size="1.778" layer="96" rot="R270"/>
+</instance>
+<instance part="C304" gate="CE" x="119.38" y="210.82" smashed="yes" rot="R180">
+<attribute name="DIS" x="119.38" y="210.82" size="1.778" layer="96" rot="R180" display="off"/>
+<attribute name="DPN" x="119.38" y="210.82" size="1.778" layer="96" rot="R180" display="off"/>
+<attribute name="MFR" x="119.38" y="210.82" size="1.778" layer="96" rot="R180" display="off"/>
+<attribute name="MPN" x="119.38" y="210.82" size="1.778" layer="96" rot="R180" display="off"/>
+<attribute name="NAME" x="117.856" y="210.439" size="1.778" layer="95" rot="R180"/>
+<attribute name="VALUE" x="117.856" y="215.519" size="1.778" layer="96" rot="R180"/>
+</instance>
+<instance part="GND7" gate="1" x="119.38" y="205.74" smashed="yes">
+<attribute name="VALUE" x="116.84" y="203.2" size="1.778" layer="96"/>
+</instance>
+<instance part="SUPPLY5" gate="G$1" x="119.38" y="226.06" smashed="yes">
+<attribute name="VALUE" x="119.38" y="228.854" size="1.778" layer="96" align="bottom-center"/>
+</instance>
 </instances>
 <busses>
@@
 <pinref part="C303" gate="CE" pin="2"/>
 <wire x1="214.376" y1="204.216" x2="214.376" y2="205.74" width="0.1524" layer="91"/>
+</segment>
+<segment>
+<pinref part="C304" gate="CE" pin="1"/>
+<pinref part="GND7" gate="1" pin="GND"/>
 </segment>
 </net>
@@
 <wire x1="345.44" y1="114.3" x2="345.44" y2="118.11" width="0.1524" layer="91"/>
 <pinref part="C310" gate="CE" pin="2"/>
+</segment>
+<segment>
+<pinref part="R301" gate="R" pin="1"/>
+<pinref part="SUPPLY5" gate="G$1" pin="3.3V"/>
 </segment>
 </net>
@@
 <wire x1="132.08" y1="215.9" x2="132.08" y2="200.66" width="0.1524" layer="91"/>
 <wire x1="132.08" y1="200.66" x2="142.24" y2="200.66" width="0.1524" layer="91"/>
-<wire x1="132.08" y1="215.9" x2="88.9" y2="215.9" width="0.1524" layer="91"/>
+<wire x1="132.08" y1="215.9" x2="119.38" y2="215.9" width="0.1524" layer="91"/>
 <label x="86.36" y="215.9" size="1.778" layer="95" rot="R180" xref="yes"/>
 <pinref part="U300" gate="G$1" pin="STBY/RESET"/>
 <pinref part="TP2" gate="G$1" pin="TP"/>
+<wire x1="119.38" y1="215.9" x2="88.9" y2="215.9" width="0.1524" layer="91"/>
 <wire x1="88.9" y1="215.9" x2="86.36" y2="215.9" width="0.1524" layer="91"/>
 <junction x="88.9" y="215.9"/>
+<pinref part="R301" gate="R" pin="2"/>
+<junction x="119.38" y="215.9"/>
+<pinref part="C304" gate="CE" pin="2"/>
 </segment>
 </net>
@@
 <attribute name="TP_SIGNAL_NAME" x="153.67" y="229.87" size="1.778" layer="97"/>
 </instance>
+<instance part="R401" gate="R" x="177.8" y="233.68" smashed="yes" rot="R270">
+<attribute name="DIS" x="177.8" y="233.68" size="1.778" layer="96" rot="R270" display="off"/>
+<attribute name="DPN" x="177.8" y="233.68" size="1.778" layer="96" rot="R270" display="off"/>
+<attribute name="MFR" x="177.8" y="233.68" size="1.778" layer="96" rot="R270" display="off"/>
+<attribute name="MPN" x="177.8" y="233.68" size="1.778" layer="96" rot="R270" display="off"/>
+<attribute name="NAME" x="179.2986" y="237.49" size="1.778" layer="95" rot="R270"/>
+<attribute name="VALUE" x="174.498" y="237.49" size="1.778" layer="96" rot="R270"/>
+</instance>
+<instance part="C404" gate="CE" x="177.8" y="223.52" smashed="yes" rot="R180">
+<attribute name="DIS" x="177.8" y="223.52" size="1.778" layer="96" rot="R180" display="off"/>
+<attribute name="DPN" x="177.8" y="223.52" size="1.778" layer="96" rot="R180" display="off"/>
+<attribute name="MFR" x="177.8" y="223.52" size="1.778" layer="96" rot="R180" display="off"/>
+<attribute name="MPN" x="177.8" y="223.52" size="1.778" layer="96" rot="R180" display="off"/>
+<attribute name="NAME" x="176.276" y="223.139" size="1.778" layer="95" rot="R180"/>
+<attribute name="VALUE" x="176.276" y="228.219" size="1.778" layer="96" rot="R180"/>
+</instance>
+<instance part="GND8" gate="1" x="177.8" y="215.9" smashed="yes">
+<attribute name="VALUE" x="175.26" y="213.36" size="1.778" layer="96"/>
+</instance>
+<instance part="SUPPLY8" gate="G$1" x="177.8" y="238.76" smashed="yes">
+<attribute name="VALUE" x="177.8" y="241.554" size="1.778" layer="96" align="bottom-center"/>
+</instance>
 </instances>
 <busses>
@@
 <pinref part="C403" gate="CE" pin="2"/>
 <wire x1="261.62" y1="227.33" x2="261.62" y2="228.6" width="0.1524" layer="91"/>
+</segment>
+<segment>
+<pinref part="C404" gate="CE" pin="1"/>
+<pinref part="GND8" gate="1" pin="GND"/>
+<wire x1="177.8" y1="218.44" x2="177.8" y2="220.98" width="0.1524" layer="91"/>
 </segment>
 </net>
@@
 <wire x1="171.45" y1="167.64" x2="171.45" y2="170.18" width="0.1524" layer="91"/>
 </segment>
+<segment>
+<pinref part="R401" gate="R" pin="1"/>
+<pinref part="SUPPLY8" gate="G$1" pin="3.3V"/>
+</segment>
 </net>
 <net name="STBY/RESET_MAG" class="0">
 <segment>
-<wire x1="189.23" y1="228.6" x2="152.4" y2="228.6" width="0.1524" layer="91"/>
+<wire x1="189.23" y1="228.6" x2="177.8" y2="228.6" width="0.1524" layer="91"/>
+<wire x1="177.8" y1="228.6" x2="152.4" y2="228.6" width="0.1524" layer="91"/>
 <wire x1="152.4" y1="228.6" x2="146.05" y2="228.6" width="0.1524" layer="91"/>
 <wire x1="189.23" y1="228.6" x2="189.23" y2="210.82" width="0.1524" layer="91"/>
@@
 <pinref part="TP3" gate="G$1" pin="TP"/>
 <junction x="152.4" y="228.6"/>
-</segment>
-</net>
+<pinref part="R401" gate="R" pin="2"/>
+<junction x="177.8" y="228.6"/>
+<pinref part="C404" gate="CE" pin="2"/>
+<junction x="177.8" y="228.6"/>
+</segment>
+</net>

Commit message: F4 updates
Connections:
- net PA0/CURR_FDB_MAG renamed MAG_CURR_FDB
- net PA1/CURR_FDB_BLDC renamed BLDC_CURR_FDB
- net PA10/INWH renamed BLDC_INWH
- net PA15/CAN_SILENT renamed CAN_SILENT
- net PA2/USART2_TX renamed USART2_TX
- net PA3/USART2_RX renamed USART2_RX
- net PA4/FAULT_BLDC renamed BLDC_FAULT
- net PA5/SPI1_SCK renamed SPI1_SCK
- net PA6/SPI1_NSS renamed SPI1_NSS
- net PA7/INUL renamed BLDC_INUL
- net PB0/INVL renamed BLDC_INVL
- net PB1/INWL renamed BLDC_INWL
- net PB3/EN_MAG renamed MAG_EN
- net PB4/SPI1_MISO renamed SPI1_MISO
- net PB6/EN_BLDC renamed BLDC_EN
- net PB7/FAULT_MAG renamed MAG_FAULT
- removed net PA8/INUH/PWM_MAG: R406.2, U$1.PA8, U300.INUH
- removed net PA9/INVH/DIR_MAG: R405.2, U$1.PA9, U300.INVH
- removed net STBY/RESET_BLDC: C304.2, R301.2, TP2.TP, U300.STBY/RESET
- removed net STBY/RESET_MAG: C404.2, R401.2, TP3.TP, U400.STBY/RESET
- new net BLDC_INUH: U$1.PA8, U300.INUH
- new net BLDC_INVH: U$1.PA9, U300.INVH
- new net BLDC_STBY: C304.2, R301.2, TP2.TP, U$1.PC8, U300.STBY/RESET
- new net MAG_DIR: R405.2, U$1.PB5
- new net MAG_PWM: R406.2, U$1.PB4
- new net MAG_STBY: C404.2, R401.2, TP3.TP, U$1.PB6, U400.STBY/RESET

Commit message: F4 update
Parts:
- removed 3.3V, EN, FB2, PG, VSEL: TPTP15SQ, testpad:TPTP15SQ
- removed C201, C202: 10u, oresat-rcl:C-EU0805-B-NOSILK
- removed C203: 10u, oresat-rcl:C-EU0603-B-NOSILK
- removed C204: 100n, rcl_custom:C-EU0402-B-NOSILK
- removed C205: 22u, oresat-rcl:C-EU0603-B-NOSILK
- removed C206, C207: 22u, oresat-rcl:C-EU0805-B-NOSILK
- removed L201: 1.5 uH, L-Coilcraft-XFL4020:L-COILCRAFT-XFL4020
- removed R201: 0, rcl_custom:R-US_0805-B-NOSILK
- removed R202, R204: 10k, rcl_custom:R-US_0402-B-NOSILK
- removed R203, R207: NP, rcl_custom:R-US_0402-B-NOSILK
- removed R205: 470k, rcl_custom:R-US_0402-B-NOSILK
- removed R206: 150k, rcl_custom:R-US_0402-B-NOSILK
- removed U200: TPS63070, ic-pwr-tps63070x:TPS63070X
- added C1: 10u, oresat-rcl:C-EU0603-B-NOSILK
- added C10, C11: 22u, oresat-rcl:C-EU0805-B-NOSILK
- added C2: 100n, rcl_custom:C-EU0402-B-NOSILK
- added C3, C7: 10u, oresat-rcl:C-EU0805-B-NOSILK
- added C9: 22u, oresat-rcl:C-EU0603-B-NOSILK
- added L1: 1.5 uH, L-Coilcraft-XFL4020:L-COILCRAFT-XFL4020
- added R1, R4: 10k, rcl_custom:R-US_0402-B-NOSILK
- added R2: 470k, rcl_custom:R-US_0402-B-NOSILK
- added R3: 150k, rcl_custom:R-US_0402-B-NOSILK
- added R6: NP, rcl_custom:R-US_0402-B-NOSILK
- added U2: TPS63070, ic-pwr-tps63070x:TPS63070X
Connections:
- removed net TPS-EN: EN.TP, R202.1, R203.2, U200.EN, U200.PS/SYNC
- removed net TPS-FB: R205.1, R206.2, U200.FB
- removed net TPS-L1: L201.1, U200.L1
- removed net TPS-L2: L201.2, U200.L2
- removed net TPS-PG: PG.TP, R207.1, U200.PG
- removed net TPS-VAUX: C204.1, U200.VAUX
- removed net TPS-VIN: C201.1, C202.1, C203.1, R201.1, R202.2, U200.VIN
- removed net TSP-FB2: FB2.TP, U200.FB2
- removed net TSP-VSEL: R204.2, U200.VSEL, VSEL.TP
- new net TPS-EN2: R1.1, R6.2, U2.EN, U2.PS/SYNC
- new net TPS-FB2: R2.1, R3.2, U2.FB
- new net TPS-L5: L1.1, U2.L1
- new net TPS-L6: L1.2, U2.L2
- new net TPS-VAUX2: C2.1, U2.VAUX
- new net TPS-VSEL2: R4.2, U2.VSEL
- new net VBUS: C1.1, C3.1, C7.1, R1.2, U2.VIN
- net 3.3V: now also C10.1, C11.1, C9.1, R2.2, U2.VOUT; no longer 3.3V.TP, C205.1, C206.1, C207.1, R205.2, R207.2, U200.VOUT
- net GND: now also C1.2, C10.2, C11.2, C2.2, C3.2, C7.2, C9.2, R3.1, R4.1, R6.1, U2.GND, U2.PGND; no longer C201.2, C202.2, C203.2, C204.2, C205.2, C206.2, C207.2, R203.1, R204.1, R206.1, U200.GND, U200.PGND
- net V_BATT: no longer R201.2

Commit message: L4 updates
Parts:
- U$1: value STM32F446X -> STM32L452XX_QFPN48; device oresat-misc:STM32F446X -> oresat-ACS_driver_board:STM32L452XX_QFPN48
Connections:
- net 3.3V: no longer U$1.VBAT, U$1.VDD, U$1.VDDA/VREF+
- net BLDC_CURR_FDB: now also U$1.PA1; no longer U$1.PA3
- net BLDC_EN: now also U$1.PA12; no longer U$1.PC6
- net BLDC_FAULT: now also U$1.PA11; no longer U$1.PC7
- net BLDC_INUH: now also U$1.PB13; no longer U$1.PA8
- net BLDC_INUL: now also U$1.PA8; no longer U$1.PB13
- net BLDC_INVH: now also U$1.PB14; no longer U$1.PA9
- net BLDC_INVL: now also U$1.PA9; no longer U$1.PB14
- net BLDC_INWH: now also U$1.PB15; no longer U$1.PA10
- net BLDC_INWL: now also U$1.PA10; no longer U$1.PB15
- net BLDC_STBY: now also U$1.PB12; no longer U$1.PC8
- net BOOT: no longer U$1.BOOT0
- net CAN_RX: no longer U$1.PA11
- net CAN_SILENT: no longer U$1.PA15
- net CAN_TX: no longer U$1.PA12
- net GND: no longer U$1.VSS, U$1.VSSA/VREF-
- net MAG_CURR_FDB: now also U$1.PA0; no longer U$1.PA2
- net MAG_DIR: now also U$1.PB3; no longer U$1.PB5
- net MAG_PWM: now also U$1.PA15; no longer U$1.PB4
- net MAG_STBY: now also U$1.PB7; no longer U$1.PB6
- net N$1: no longer U$1.PH0-OSC_IN
- net N$4: no longer U$1.PH1-OSC_OUT
- net N$6: no longer U$1.VCAP_1
- net NRESET: no longer U$1.NRST
- net SWCLK: no longer U$1.PA14
- net SWDIO: no longer U$1.PA13
- net USART2_RX: no longer U$1.PA1
- net USART2_TX: no longer U$1.PA0

Commit message: Schematic Overhal and chip opperation verification
Parts:
- removed C106: 100n, rcl_custom:C-EU0402-B-NOSILK
- removed C107: 2.2u, rcl_custom:C-EU0402-B-NOSILK
- removed JP302: (no value), pinhead:PINHD-1X2
- removed R1: 10k, rcl_custom:R-US_0402-B-NOSILK
- removed R303, R403: 0, oresat-rcl:R-US_0805-B-NOSILK
- removed R314, R419: 0, rcl_custom:R-US_0402-B-NOSILK
- removed R6: NP, rcl_custom:R-US_0402-B-NOSILK
- added JP2: (no value), pinhead:PINHD-1X2
- added R201: 10k, rcl_custom:R-US_0402-B-NOSILK
- added R202: NP, rcl_custom:R-US_0402-B-NOSILK
- added U$2, U$3: DEBUG_CON, oresat-ACS_driver_board:DEBUG_CON
- C103: value 100n -> 10n
- C104: value 20p -> 10p
- C105: value 20p -> 100n; DPN 1276-6601-1-ND -> 1276-1001-1-ND; MPN CL05C200JB51PNC -> CL05B104KO5NNNC
- U300: device U-ST-STSPIN230-BLDC-controller:STSPIN230 -> oresat-ACS_driver_board:STSPIN230
- U301, U401: device TSV991ILT:TSV991ILT -> oresat-ACS_driver_board:TSV991ILT
- U400: device U-ST-STSPIN250-Brushed-DC-controller:STSPIN250 -> oresat-ACS_driver_board:STSPIN250
- X101: value 16MHZ-2.5x2mm -> ABM10-16MHz
- renumbered C1 to C203, C10 to C206, C11 to C207, C2 to C204, C3 to C201, C7 to C202, C9 to C205, L1 to L201, R2 to R204, R3 to R205, R4 to R203, U2 to U200
Connections:
- net BLDC-I-IN+ renamed N$9
- net MAG-I-IN+ renamed N$7
- net NRESET renamed NRESET_D
- net USART2_RX renamed USART_RX_D
- net USART2_TX renamed USART_TX_D
- removed net BLDC-I-IN-: C307.1, R312.1, R313.2, U301.IN-
- removed net BLDC-I-OUT: C307.2, R313.1, R314.2, U301.OUT
- removed net MAG-I-IN-: C411.1, R417.1, R418.2, U401.IN-
- removed net MAG-I-OUT: C411.2, R418.1, R419.2, U401.OUT
- removed net N$6: C107.2
- removed net N$7 (its old number): C301.1, C302.1, C303.1, R303.1, U300.VS
- removed net N$8: C401.1, C402.1, C403.1, R403.1, U400.VS
- new net N$11: C411.2, R417.2, R418.1, U401.IN-
- new net N$12: C307.2, R312.2, R313.1, U301.IN-
- new net NRST: U$1.NRST
- new net QUAD_A_D: JP2.1
- new net QUAD_B_D: JP2.2
- new net SWCLK_D: J1.SWDCLK/TCK
- new net SWDIO_D: J1.SWDIO/TMS
- new net UART_RX: U$1.PA3
- new net UART_XT: U$1.PA2
- net 250_REF: now also C407.1; no longer C407.2
- net 3.3V: now also C101.1, C102.1, C103.1, C105.2, C308.1, C310.1, U$1.VBAT, U$1.VDD, U$1.VDDA, U$2.2, U$3.2; no longer C101.2, C102.2, C103.2, C106.2, C308.2, C310.2
- net BLDC_CURR_FDB: now also C307.1, R313.2, U301.OUT; no longer R314.1
- net BLDC_FAULT: now also C305.1; no longer C305.2
- net BLDC_STBY: now also C304.1; no longer C304.2
- net BOOT: now also U$1.PH3-BOOT0
- net CAN_RX: now also U$1.PB5
- net CAN_SILENT: now also U$1.PB4
- net CAN_TX: now also U$1.PB6
- net GND: now also C101.2, C102.2, C103.2, C304.2, C305.2, C308.2, C310.2, C404.2, C405.2, C406.2, C407.2, R202.1, R312.1, R417.1, U$1.VDDUSB, U$1.VSS, U$1.VSSA, U$2.10, U$3.10; no longer C101.1, C102.1, C103.1, C104.1, C106.1, C107.1, C304.1, C305.1, C308.1, C310.1, C404.1, C405.1, C406.1, C407.1, R312.2, R417.2, R6.1
- net MAG_CURR_FDB: now also C411.1, R418.2, U401.OUT; no longer R419.1
- net MAG_FAULT: now also C405.1; no longer C405.2
- net MAG_STBY: now also C404.1; no longer C404.2
- net N$1: now also U$1.PH1-OSC_OUT, X101.1; no longer X101.2
- net N$2: now also C406.1; no longer C406.2
- net N$4: now also C104.1, U$1.PH0-OSC_IN, X101.2; no longer C105.2, X101.1
- net QUAD_A: no longer JP302.1
- net QUAD_B: no longer JP302.2
- net SWCLK: now also U$1.PA14; no longer J1.SWDCLK/TCK
- net SWDIO: now also U$1.PA13; no longer J1.SWDIO/TMS
- net TPS-EN2: now also R201.1, R202.2; no longer R1.1, R6.2
- net VBUS: now also C301.1, C302.1, C303.1, C401.1, C402.1, C403.1, JP1.1, JP103.VCC, R201.2, U$3.1, U300.VS, U400.VS; no longer R1.2
- net V_BATT: now also U$2.1; no longer JP1.1, JP103.VCC, R303.2, R403.2
Other:
- note added: "Debug Breakout Board"
- note removed: "All caps are ceramic 10% X5R >= 16V Vwv unless marked"
- note removed: "All resistors 0402 +/- 1% unless marked"
- note removed: "CAN_SHDN and CAN_LSTN pins have internal pull-down resistors. If CAN_SHDN is pulled high it shuts the IC off. If CAN_LSTN is pulled high it puts the IC intro receive-only mode. Leave CAN_SHDN disconnected."
- note removed: "Current feedback to STM32."
- note removed: "NP FOR FLIGHT"
- note removed: "NRST pull-up built in"
- note removed: "Quadrature output leads for motor spec test case"
- note removed: "STM32 Current Feedback"
