File: eaglecad/controller_rev4.sch (EAGLE design)
At the start: 85 parts, among them J1 1.27MM-SWD-CONNECTOR, U101 TCAN330, U200 TPS63070, U300 STSPIN230, U301 TSV991ILT, U302 AS5047P, U400 STSPIN250, U401 TSV991ILT, X101 ABM10-16MHz

Commit message: Prelim final rev completed + design overhaul
Parts:
- removed J1: 1.27MM-SWD-CONNECTOR, J-CNC-3220-10-0100-00-ARM-SWD-port:1.27MM-SWD-CONNECTOR
- removed JP103: (no value), SparkFun-Connectors:6_PIN_SERIAL_TARGETSILK
- removed JP2: (no value), pinhead:PINHD-1X2
- removed R312, R417, R418: 2.2k, rcl_custom:R-US_0402-B-NOSILK
- removed R315: 10k, rcl_custom:R-US_0402-B-NOSILK
- added JP501: (no value), pinhead:PINHD-1X2
- added JP502: (no value), SparkFun-Connectors:6_PIN_SERIAL_TARGETSILK
- added JP503: 1.27MM-SWD-CONNECTOR, J-CNC-3220-10-0100-00-ARM-SWD-port:1.27MM-SWD-CONNECTOR
- added R303: 2.2k, rcl_custom:R-US_0402-B-NOSILK
- added R304: 680, rcl_custom:R-US_0402-B-NOSILK
- added R403, R404: 330, rcl_custom:R-US_0402-B-NOSILK
- C306: value 680p -> 4.7u; device rcl_custom:C-EU0402-B-NOSILK -> oresat-rcl:C-EU0603-B-NOSILK
- C307, C408: value 680p -> 100n
- C308: value 100n -> 680p
- C309, C410: value 4.7u -> 680p; device oresat-rcl:C-EU0603-B-NOSILK -> rcl_custom:C-EU0402-B-NOSILK
- C406: value 22n -> 2.2n
- C407: value 2.2n -> 22n
- C409: value 100n -> 4.7u; device rcl_custom:C-EU0402-B-NOSILK -> oresat-rcl:C-EU0603-B-NOSILK
- R309: value 680 -> 10k
- R405: value 330 -> 100k
- R406: value 330 -> 18k
- R409: value 100k -> 2.2k
- R410: value 18k -> 680
- R414: value 680 -> 2.2k
- renumbered JP1 to JP101, R310 to R305, R311 to R306, R313 to R307, R415 to R411, R416 to R412, U$1 to U100
Connections:
- removed net UART_XT: U100.PA2
- new net UART_TX: U$2.6, U100.PA2
- net 250_REF: now also C406.1, R405.2, R406.1; no longer C407.1, R409.2, R410.1
- net 3.3V: now also C306.1, C307.1, C408.1, JP503.VTREF, R303.2, R309.1, R405.1, R409.2; no longer C308.1, C309.1, C410.1, J1.VTREF, R308.2, R315.1, R409.1, R413.2
- net AS5047_MOSI: now also R309.2; no longer R315.2
- net BLDC_CURR_FDB: now also C309.1; no longer C307.1
- net GND: now also C307.2, JP502.GND, JP503.GND, JP503.GND@2, R308.1, R406.2, R414.1; no longer C309.2, J1.GND, J1.GND@2, JP103.GND, R312.1, R410.2, R417.1
- net MAG_CURR_FDB: now also R413.2; no longer R418.2
- net MAG_DIR: now also R403.2; no longer R405.2
- net MAG_PWM: now also R404.2; no longer R406.2
- net N$11: now also R413.1, R414.2; no longer R417.2, R418.1
- net N$12: now also C309.2, R308.2; no longer C307.2, R312.2
- net N$2: now also C407.1; no longer C406.1
- net N$3: now also R404.1; no longer R406.1
- net N$5: now also R403.1; no longer R405.1
- net N$7: now also C410.1, R409.1, R410.2; no longer C408.1, R413.1, R414.2
- net N$9: now also C308.1, R303.1, R304.2; no longer C306.1, R308.1, R309.2
- net NRESET_D: now also JP503.!RESET, U$3.7; no longer J1.!RESET
- net NRST: now also U$2.7
- net QUAD_A: now also U$2.4
- net QUAD_A_D: now also JP501.1, U$3.4; no longer JP2.1
- net QUAD_B: now also U$2.3
- net QUAD_B_D: now also JP501.2, U$3.3; no longer JP2.2
- net SENSE_BLDC: now also R304.1; no longer R309.1
- net SENSE_MAG: now also R410.1; no longer R414.1
- net SWCLK: now also U$2.9
- net SWCLK_D: now also JP503.SWDCLK/TCK, U$3.9; no longer J1.SWDCLK/TCK
- net SWDIO: now also U$2.8
- net SWDIO_D: now also JP503.SWDIO/TMS, U$3.8; no longer J1.SWDIO/TMS
- net UART_RX: now also U$2.5
- net USART_RX_D: now also JP502.RXI, U$3.5; no longer JP103.RXI
- net USART_TX_D: now also JP502.TXO, U$3.6; no longer JP103.TXO
- net VBUS: now also JP502.VCC; no longer JP103.VCC
Other:
- moved on the sheet: C306, C307, C308, C309, C406, C407, C408, C409, C410, R308, R309, R405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
