File: eaglecad/oresat-card.sch (EAGLE design)
At the start: 96 parts, among them J1 J-SAMTEC-TFM-110-X1-XXX-D-RA, J2 U.FL, J3 U.FL, J4 U.FL, J6 J-SAMTEC-TFM-120-X1-XXX-D-RA, Q1 DMP2240UDM, Q3 MOSFET-PCH-SOT23-6, Q4 MOSFET-PCH-SOT23-6, Q5 PMV45EN, Q6 PMV45EN, U3 MAX7310ATE, U4 MAX4211CETE, U5 TPS62111RSA, U7 MCP1703A

Commit message: mods
Connections:
- net CB-RESET: now also U4.CIN2+; no longer U4.CIN2-
- net N$596: now also U4.CIN1+; no longer U4.CIN1-
- net N$597: now also U4.CIN1-; no longer U4.CIN1+
- net N$599: now also U4.CIN2-; no longer U4.CIN2+
Other:
- moved on the sheet: R30, R34, TP11, TP12
Changed lines of the file:
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@@
 <attribute name="VALUE" x="285.75" y="199.39" size="1.778" layer="96"/>
 </instance>
-<instance part="R30" gate="R" x="304.8" y="152.4" smashed="yes" rot="R90">
-<attribute name="DIS" x="304.8" y="152.4" size="1.778" layer="96" rot="R90" display="off"/>
-<attribute name="DPN" x="304.8" y="152.4" size="1.778" layer="96" rot="R90" display="off"/>
-<attribute name="MFR" x="304.8" y="152.4" size="1.778" layer="96" rot="R90" display="off"/>
-<attribute name="MPN" x="304.8" y="152.4" size="1.778" layer="96" rot="R90" display="off"/>
-<attribute name="NAME" x="303.53" y="147.32" size="1.778" layer="95" rot="R90"/>
-<attribute name="VALUE" x="303.53" y="152.4" size="1.778" layer="96" rot="R90"/>
-</instance>
-<instance part="GND33" gate="1" x="304.8" y="144.78" smashed="yes" rot="MR0">
-<attribute name="VALUE" x="307.34" y="142.24" size="1.778" layer="96" rot="MR0"/>
+<instance part="R30" gate="R" x="307.34" y="152.4" smashed="yes" rot="R90">
+<attribute name="DIS" x="307.34" y="152.4" size="1.778" layer="96" rot="R90" display="off"/>
+<attribute name="DPN" x="307.34" y="152.4" size="1.778" layer="96" rot="R90" display="off"/>
+<attribute name="MFR" x="307.34" y="152.4" size="1.778" layer="96" rot="R90" display="off"/>
+<attribute name="MPN" x="307.34" y="152.4" size="1.778" layer="96" rot="R90" display="off"/>
+<attribute name="NAME" x="306.07" y="147.32" size="1.778" layer="95" rot="R90"/>
+<attribute name="VALUE" x="306.07" y="152.4" size="1.778" layer="96" rot="R90"/>
+</instance>
+<instance part="GND33" gate="1" x="307.34" y="144.78" smashed="yes" rot="MR0">
+<attribute name="VALUE" x="309.88" y="142.24" size="1.778" layer="96" rot="MR0"/>
 </instance>
 <instance part="R31" gate="R" x="327.66" y="185.42" smashed="yes" rot="R180">
@@
 <attribute name="VALUE" x="323.85" y="179.07" size="1.778" layer="96"/>
 </instance>
-<instance part="R34" gate="R" x="327.66" y="167.64" smashed="yes" rot="R90">
-<attribute name="DIS" x="327.66" y="167.64" size="1.778" layer="96" rot="R90" display="off"/>
-<attribute name="DPN" x="327.66" y="167.64" size="1.778" layer="96" rot="R90" display="off"/>
-<attribute name="MFR" x="327.66" y="167.64" size="1.778" layer="96" rot="R90" display="off"/>
-<attribute name="MPN" x="327.66" y="167.64" size="1.778" layer="96" rot="R90" display="off"/>
-<attribute name="NAME" x="326.39" y="162.56" size="1.778" layer="95" rot="R90"/>
-<attribute name="VALUE" x="326.39" y="168.91" size="1.778" layer="96" rot="R90"/>
-</instance>
-<instance part="GND34" gate="1" x="327.66" y="160.02" smashed="yes" rot="MR0">
-<attribute name="VALUE" x="330.2" y="157.48" size="1.778" layer="96" rot="MR0"/>
+<instance part="R34" gate="R" x="327.66" y="162.56" smashed="yes" rot="R90">
+<attribute name="DIS" x="327.66" y="162.56" size="1.778" layer="96" rot="R90" display="off"/>
+<attribute name="DPN" x="327.66" y="162.56" size="1.778" layer="96" rot="R90" display="off"/>
+<attribute name="MFR" x="327.66" y="162.56" size="1.778" layer="96" rot="R90" display="off"/>
+<attribute name="MPN" x="327.66" y="162.56" size="1.778" layer="96" rot="R90" display="off"/>
+<attribute name="NAME" x="326.39" y="157.48" size="1.778" layer="95" rot="R90"/>
+<attribute name="VALUE" x="326.39" y="163.83" size="1.778" layer="96" rot="R90"/>
+</instance>
+<instance part="GND34" gate="1" x="327.66" y="154.94" smashed="yes" rot="MR0">
+<attribute name="VALUE" x="330.2" y="152.4" size="1.778" layer="96" rot="MR0"/>
 </instance>
 <instance part="GND35" gate="1" x="337.82" y="172.72" smashed="yes" rot="MR0">
@@
 <attribute name="NAME" x="298.45" y="179.07" size="1.778" layer="95" font="vector"/>
 </instance>
-<instance part="TP11" gate="G$1" x="314.96" y="172.72" smashed="yes">
-<attribute name="NAME" x="311.15" y="168.91" size="1.778" layer="95" font="vector"/>
-</instance>
-<instance part="TP12" gate="G$1" x="309.88" y="167.64" smashed="yes">
-<attribute name="NAME" x="306.07" y="163.83" size="1.778" layer="95" font="vector"/>
+<instance part="TP11" gate="G$1" x="314.96" y="167.64" smashed="yes">
+<attribute name="NAME" x="313.69" y="163.83" size="1.778" layer="95" font="vector"/>
+</instance>
+<instance part="TP12" gate="G$1" x="332.74" y="172.72" smashed="yes">
+<attribute name="NAME" x="328.93" y="168.91" size="1.778" layer="95" font="vector"/>
 </instance>
 <instance part="TP13" gate="G$1" x="190.5" y="144.78" smashed="yes">
@@
 <net name="CB-RESET" class="0">
 <segment>
-<pinref part="U4" gate="G$1" pin="CIN2-"/>
-<pinref part="R30" gate="R" pin="2"/>
-<wire x1="299.72" y1="157.48" x2="304.8" y2="157.48" width="0.1524" layer="91"/>
-<wire x1="304.8" y1="157.48" x2="312.42" y2="157.48" width="0.1524" layer="91"/>
-<junction x="304.8" y="157.48"/>
-<wire x1="312.42" y1="157.48" x2="312.42" y2="132.08" width="0.1524" layer="91"/>
+<wire x1="312.42" y1="162.56" x2="312.42" y2="132.08" width="0.1524" layer="91"/>
 <wire x1="312.42" y1="132.08" x2="213.36" y2="132.08" width="0.1524" layer="91"/>
 <wire x1="213.36" y1="132.08" x2="213.36" y2="142.24" width="0.1524" layer="91"/>
@@
 <junction x="213.36" y="142.24"/>
 <label x="144.78" y="142.24" size="1.778" layer="95"/>
-<label x="299.72" y="158.75" size="1.778" layer="95"/>
+<pinref part="U4" gate="G$1" pin="CIN2+"/>
+<wire x1="312.42" y1="162.56" x2="307.34" y2="162.56" width="0.1524" layer="91"/>
+<label x="316.23" y="149.86" size="1.778" layer="95" rot="R90"/>
+<pinref part="R30" gate="R" pin="2"/>
+<wire x1="307.34" y1="162.56" x2="299.72" y2="162.56" width="0.1524" layer="91"/>
+<wire x1="307.34" y1="157.48" x2="307.34" y2="162.56" width="0.1524" layer="91"/>
+<junction x="307.34" y="162.56"/>
 </segment>
 </net>
@@
 <pinref part="R31" gate="R" pin="1"/>
 <pinref part="R32" gate="R" pin="2"/>
-<pinref part="U4" gate="G$1" pin="CIN1-"/>
-<wire x1="299.72" y1="167.64" x2="309.88" y2="167.64" width="0.1524" layer="91"/>
-<wire x1="309.88" y1="167.64" x2="317.5" y2="167.64" width="0.1524" layer="91"/>
-<wire x1="317.5" y1="167.64" x2="317.5" y2="154.94" width="0.1524" layer="91"/>
-<wire x1="317.5" y1="154.94" x2="332.74" y2="154.94" width="0.1524" layer="91"/>
-<wire x1="332.74" y1="154.94" x2="332.74" y2="185.42" width="0.1524" layer="91"/>
 <junction x="332.74" y="185.42"/>
+<wire x1="332.74" y1="172.72" x2="332.74" y2="185.42" width="0.1524" layer="91"/>
 <wire x1="332.74" y1="185.42" x2="337.82" y2="185.42" width="0.1524" layer="91"/>
+<pinref part="U4" gate="G$1" pin="CIN1+"/>
+<wire x1="299.72" y1="172.72" x2="332.74" y2="172.72" width="0.1524" layer="91"/>
 <pinref part="TP12" gate="G$1" pin="1"/>
-<junction x="309.88" y="167.64"/>
 </segment>
 </net>
@@
 <pinref part="R33" gate="R" pin="1"/>
 <pinref part="R34" gate="R" pin="2"/>
-<pinref part="U4" gate="G$1" pin="CIN1+"/>
-<wire x1="299.72" y1="172.72" x2="314.96" y2="172.72" width="0.1524" layer="91"/>
-<wire x1="314.96" y1="172.72" x2="327.66" y2="172.72" width="0.1524" layer="91"/>
-<wire x1="327.66" y1="172.72" x2="327.66" y2="177.8" width="0.1524" layer="91"/>
-<junction x="327.66" y="172.72"/>
+<wire x1="314.96" y1="167.64" x2="327.66" y2="167.64" width="0.1524" layer="91"/>
+<wire x1="327.66" y1="167.64" x2="327.66" y2="177.8" width="0.1524" layer="91"/>
+<junction x="327.66" y="167.64"/>
 <pinref part="TP11" gate="G$1" pin="1"/>
-<junction x="314.96" y="172.72"/>
+<pinref part="U4" gate="G$1" pin="CIN1-"/>
+<wire x1="314.96" y1="167.64" x2="299.72" y2="167.64" width="0.1524" layer="91"/>
+<junction x="314.96" y="167.64"/>
 </segment>
 </net>
@@
 <pinref part="R33" gate="R" pin="2"/>
 <wire x1="299.72" y1="177.8" x2="304.8" y2="177.8" width="0.1524" layer="91"/>
-<pinref part="U4" gate="G$1" pin="CIN2+"/>
 <wire x1="304.8" y1="177.8" x2="317.5" y2="177.8" width="0.1524" layer="91"/>
-<wire x1="299.72" y1="162.56" x2="304.8" y2="162.56" width="0.1524" layer="91"/>
-<wire x1="304.8" y1="162.56" x2="304.8" y2="177.8" width="0.1524" layer="91"/>
+<wire x1="304.8" y1="157.48" x2="304.8" y2="177.8" width="0.1524" layer="91"/>
 <junction x="304.8" y="177.8"/>
-</segment>
-</net>
+<pinref part="U4" gate="G$1" pin="CIN2-"/>
+<wire x1="304.8" y1="157.48" x2="299.72" y2="157.48" width="0.1524" layer="91"/>
+</segment>
+</net>

Commit message: card
Parts:
- removed C10: 1u, oresat-rcl:C-EU0603-B-NOSILK
- removed C12: 22u, oresat-rcl:C-EU0805-B-NOSILK
- removed C7: 10u, oresat-rcl:C-EU0805-B-NOSILK
- removed D2: GREEN, SparkFun-LED:LED-GREEN0603
- removed L2: 6.8u, L-ECS-MPI4040:L-ECS-MPI4040
- removed R10: NP, rcl_custom:R-US_0402-B-NOSILK
- removed R2: 2.7k, rcl_custom:R-US_0402-B-NOSILK
- removed R7: 10k, rcl_custom:R-US_0402-B-NOSILK
- removed TP16, TP17, TP19: TEST-POINT, Tova:TEST-POINT
- removed U5: TPS62111RSA, U-TI-TPS6211x-SPS-buck:TPS6211X
Connections:
- removed net N$271: D2.A, R2.1
- removed net TPS62111-PG: TP16.1, U5.PG
- removed net TPS62111-SYNC: R10.2, R7.1, TP19.1, U5.SYNC
- removed net TPS62111_SW: L2.1, U5.SW
- net 3.3V: no longer C12.1, L2.2, R2.2, TP17.1, U5.FB
- net GND: no longer C10.2, C12.2, C7.2, D2.C, R10.1, U5.GND, U5.LBI, U5.LBO
- net VBUSP: no longer C10.1, C7.1, R7.2, U5.EN, U5.VIN
Other:
- note removed: "0805"
- note removed: "3.3V Card Switching Supply"
- note removed: "ECS-MPI4040R4-6R8-R"
- note removed: "NOTE: This is outdated, REF should be connected to the inverting terminals, not the noninverting"
