File: eaglecad/design_block-readable.sch (EAGLE design)
At the start: 260 parts, among them J6 J-SAMTEC-TFM-120-X1-XXX-D-RA, Q10 DMP2240UDM, Q11 MOSFET-PCH-SOT23-6, Q12 MOSFET-PCH-SOT23-6, Q13 PMV45EN, Q14 PMV45EN, Q15 DMP2240UDM, Q16 MOSFET-PCH-SOT23-6, Q17 MOSFET-PCH-SOT23-6, Q18 PMV45EN, Q19 PMV45EN, Q20 DMP2240UDM, Q21 MOSFET-PCH-SOT23-6, Q22 MOSFET-PCH-SOT23-6, Q23 PMV45EN, Q24 PMV45EN, Q25 DMP2240UDM, Q6 MOSFET-PCH-SOT23-6, Q7 MOSFET-PCH-SOT23-6, Q8 PMV45EN, Q9 PMV45EN, U10 MAX7310ATE, U11 MAX4211CETE, U12 MCP1703A, U13 MAX7310ATE, U14 MAX4211CETE, U15 MCP1703A, U3 MAX7310ATE, U4 MAX4211CETE, U6 MCP1703A, U7 MAX7310ATE, U8 MAX4211CETE, U9 MCP1703A

Commit message: ACS card updates
Parts:
- removed C10, C15, C16, C21, C22, C27, C28, C9: 1u, oresat-rcl:C-EU0603-B-NOSILK
- removed C11, C12, C17, C18, C23, C24, C29, C30: TBD, rcl_custom:C-EU0402-B-NOSILK
- removed C13, C19, C25, C7: 100n, rcl_custom:C-EU0402-B-NOSILK
- removed C14, C20, C26, C8: NP, rcl_custom:C-EU0402-B-NOSILK
- removed D10, D4, D6, D8: AMBER, SparkFun-LED:LED-GREEN0603
- removed D3, D5, D7, D9: GREEN, SparkFun-LED:LED-GREEN0603
- removed H1, H2, H3, H4: STAND-OFFTIGHT, SparkFun-Hardware:STAND-OFFTIGHT
- removed J6: J-SAMTEC-TFM-120-X1-XXX-D-RA, J-Samtec-TFM-120-X1-XXX-D-RA:J-SAMTEC-TFM-120-X1-XXX-D-RA
- removed JP10: (no value), pinhead:PINHD-2X5
- removed Q10, Q15, Q20, Q25: DMP2240UDM, Q-MOSFET-PCH-dual-SOT23-6:MOSFET-PCH-SOT23-6
- removed Q11, Q12, Q16, Q17, Q21, Q22, Q6, Q7: MOSFET-PCH-SOT23-6, Q-MOSFET-PCH-SOT23-6:MOSFET-PCH-SOT23-6
- removed Q13, Q14, Q18, Q19, Q23, Q24, Q8, Q9: PMV45EN, Tova:PMV45EN
- removed R100, R106, R135, R141, R170, R36, R65, R71: 2.7k, rcl_custom:R-US_0402-B-NOSILK
- removed R101, R102, R103, R122, R123, R124, R126, R131, R134, R136, R137, R138, R157, R158, R159, R161, R166, R169, R171, R172, R173, R52, R53, R54, R56, R61, R64, R66, R67, R68, R87, R88, R89, R91, R96, R99: 10k, rcl_custom:R-US_0402-B-NOSILK
- removed R104, R105, R139, R140, R174, R175, R69, R70: 47k, rcl_custom:R-US_0402-B-NOSILK
- removed R107, R120, R121, R142, R155, R156, R37, R50, R51, R72, R85, R86: 100, rcl_custom:R-US_0402-B-NOSILK
- removed R108, R109, R110, R111, R112, R113, R114, R115, R116, R117, R118, R119, R128, R130, R132, R133, R143, R144, R145, R146, R147, R148, R149, R150, R151, R152, R153, R154, R163, R165, R167, R168, R38, R39, R40, R41, R42, R43, R44, R45, R46, R47, R48, R49, R58, R60, R62, R63, R73, R74, R75, R76, R77, R78, R79, R80, R81, R82, R83, R84, R93, R95, R97, R98: NP, rcl_custom:R-US_0402-B-NOSILK
- removed R125, R160, R55, R90: 100m, rcl:R-US_R1206
- removed R127, R129, R162, R164, R57, R59, R92, R94: 0, rcl_custom:R-US_0402-B-NOSILK
- removed TP13, TP14, TP15, TP16, TP17, TP18, TP19, TP20, TP21, TP22, TP23, TP24, TP25, TP26, TP27, TP28, TP29, TP30, TP31, TP32, TP33, TP34, TP35, TP36, TP37, TP38, TP39, TP40, TP41, TP42, TP43, TP44, TP45, TP46, TP47, TP48, TP49, TP50, TP51, TP52, TP53, TP54, TP55, TP56, TP57, TP58, TP59, TP60: TEST-POINT, Tova:TEST-POINT
- removed U$1: CARD-CONNECTOR_B, oresat-ACS_driver_board:CARD-CONNECTOR_B
- removed U$2: ORESAT-CARD-V1.1-3XRF, oresat-cards:ORESAT-CARD-V1.1-3XRF
- removed U10, U13, U3, U7: MAX7310ATE, U-Maxim-MAX7310-I2C-GPIO-expander:MAX7310
- removed U11, U14, U4, U8: MAX4211CETE, U-Maxim-MAX4211-power-monitor:MAX4211
- removed U12, U15, U6, U9: MCP1703A, v-reg:XC63FPM
- added C1: 100n, rcl_custom:C-EU0402-B-NOSILK
- added C2, C3: TBD, rcl_custom:C-EU0402-B-NOSILK
- added C4, C5: 1u, oresat-rcl:C-EU0603-B-NOSILK
- added C6: NP, rcl_custom:C-EU0402-B-NOSILK
- added D1: AMBER, SparkFun-LED:LED-GREEN0603
- added D2: GREEN, SparkFun-LED:LED-GREEN0603
- added Q1: DMP2240UDM, Q-MOSFET-PCH-dual-SOT23-6:MOSFET-PCH-SOT23-6
- added Q2, Q4: MOSFET-PCH-SOT23-6, Q-MOSFET-PCH-SOT23-6:MOSFET-PCH-SOT23-6
- added Q3, Q5: PMV45EN, Tova:PMV45EN
- added R1, R10, R11, R12, R2, R25, R26, R3, R30, R31, R4, R5, R6, R7, R8, R9: NP, rcl_custom:R-US_0402-B-NOSILK
- added R13, R18, R19, R20, R23, R24, R32, R33, R34: 10k, rcl_custom:R-US_0402-B-NOSILK
- added R14, R15: 47k, rcl_custom:R-US_0402-B-NOSILK
- added R16, R17, R22: 100, rcl_custom:R-US_0402-B-NOSILK
- added R21, R35: 2.7k, rcl_custom:R-US_0402-B-NOSILK
- added R27: 100m, rcl:R-US_R1206
- added R28, R29: 0, rcl_custom:R-US_0402-B-NOSILK
- added TP1, TP10, TP11, TP12, TP2, TP3, TP4, TP5, TP6, TP7, TP8, TP9: TEST-POINT, Tova:TEST-POINT
- added U1: MAX7310ATE, U-Maxim-MAX7310-I2C-GPIO-expander:MAX7310
- added U2: MAX4211CETE, U-Maxim-MAX4211-power-monitor:MAX4211
- added U5: MCP1703A, v-reg:XC63FPM
Connections:
- removed net !FAULT_Q1: Q9.D, R64.1, TP18.1, U3.IO2
- removed net !FAULT_Q2: Q14.D, R99.1, TP30.1, U7.IO2
- removed net !FAULT_Q3: Q19.D, R134.1, TP42.1, U10.IO2
- removed net !FAULT_Q4: Q24.D, R169.1, TP54.1, U13.IO2
- removed net !SD: J6.39, J6.40, JP10.10, JP10.9
- removed net AD0_Q1: R38.1, R39.2, R40.2, R41.1, U3.AD0
- removed net AD0_Q2: R73.1, R74.2, R75.2, R76.1, U7.AD0
- removed net AD0_Q3: R108.1, R109.2, R110.2, R111.1, U10.AD0
- removed net AD0_Q4: R143.1, R144.2, R145.2, R146.1, U13.AD0
- removed net AD1_Q1: R42.1, R43.2, R44.2, R45.1, U3.AD1
- removed net AD1_Q2: R77.1, R78.2, R79.2, R80.1, U7.AD1
- removed net AD1_Q3: R112.1, R113.2, R114.2, R115.1, U10.AD1
- removed net AD1_Q4: R147.1, R148.2, R149.2, R150.1, U13.AD1
- removed net AD2_Q1: R46.1, R47.2, R48.2, R49.1, U3.AD2
- removed net AD2_Q2: R81.1, R82.2, R83.2, R84.1, U7.AD2
- removed net AD2_Q3: R116.1, R117.2, R118.2, R119.1, U10.AD2
- removed net AD2_Q4: R151.1, R152.2, R153.2, R154.1, U13.AD2
- removed net BOOT_Q1: U3.IO5
- removed net BOOT_Q2: U7.IO5
- removed net BOOT_Q3: U10.IO5
- removed net BOOT_Q4: U13.IO5
- removed net CAN2_H: J6.17, J6.18, JP10.5, JP10.6
- removed net CAN2_L: J6.19, J6.20, JP10.7, JP10.8
- removed net CB-RESET_Q1: R56.2, TP17.1, U3.IO1, U4.CIN2+
- removed net CB-RESET_Q2: R91.2, TP29.1, U7.IO1, U8.CIN2+
- removed net CB-RESET_Q3: R126.2, TP41.1, U10.IO1, U11.CIN2+
- removed net CB-RESET_Q4: R161.2, TP53.1, U13.IO1, U14.CIN2+
- removed net CB_CTRL_Q1: Q6.G, Q9.G, R61.1, U4.COUT1, U4.COUT2, U4.LE
- removed net CB_CTRL_Q2: Q11.G, Q14.G, R96.1, U8.COUT1, U8.COUT2, U8.LE
- removed net CB_CTRL_Q3: Q16.G, Q19.G, R131.1, U11.COUT1, U11.COUT2, U11.LE
- removed net CB_CTRL_Q4: Q21.G, Q24.G, R166.1, U14.COUT1, U14.COUT2, U14.LE
- removed net MAX4211-3V3_Q1: C10.1, U4.VCC, U6.OUT
- removed net MAX4211-3V3_Q2: C16.1, U8.VCC, U9.OUT
- removed net MAX4211-3V3_Q3: C22.1, U11.VCC, U12.OUT
- removed net MAX4211-3V3_Q4: C28.1, U14.VCC, U15.OUT
- removed net N$1: J6.34
- removed net N$21: D3.A, R36.1
- removed net N$22: R52.1, U3.!RESET
- removed net N$23: Q7.G, Q8.D, R53.1
- removed net N$24: Q7.D, R55.1, U4.RS+
- removed net N$25: R57.1, R58.2, TP15.1, U4.CIN1+
- removed net N$26: R59.1, R60.2, TP14.1, U4.CIN1-
- removed net N$27: R57.2, U4.IOUT
- removed net N$271: J6.33
- removed net N$28: R59.2, U4.CIN2-, U4.REF
- removed net N$29: TP13.1, U4.POUT
- removed net N$30: R63.1, U4.INHIBIT
- removed net N$300: J6.2
- removed net N$31: C8.1, R62.2, R63.2
- removed net N$32: C9.1, Q6.S, R55.2, R61.2, U4.RS-, U6.IN
- removed net N$33: R65.2, TP22.1, U3.IO7
- removed net N$34: D4.A, R65.1
- removed net N$35: C11.1, Q10.1.S, R51.2
- removed net N$36: C11.2, Q10.1.G, Q10.2.D, R66.2
- removed net N$37: C12.2, Q10.2.G, R67.2, R68.1
- removed net N$38: R69.1, R70.1, TP21.1, U3.IO6
- removed net N$400: J6.35
- removed net N$406: J6.36
- removed net N$41: D5.A, R71.1
- removed net N$42: R87.1, U7.!RESET
- removed net N$43: Q12.G, Q13.D, R88.1
- removed net N$44: Q12.D, R90.1, U8.RS+
- removed net N$45: R92.1, R93.2, TP27.1, U8.CIN1+
- removed net N$46: R94.1, R95.2, TP26.1, U8.CIN1-
- removed net N$47: R92.2, U8.IOUT
- removed net N$479: J6.9
- removed net N$48: R94.2, U8.CIN2-, U8.REF
- removed net N$480: J6.4
- removed net N$482: J6.5
- removed net N$49: TP25.1, U8.POUT
- removed net N$498: J6.1
- removed net N$499: J6.7
- removed net N$50: R98.1, U8.INHIBIT
- removed net N$500: J6.6
- removed net N$503: J6.8
- removed net N$504: J6.10
- removed net N$51: C14.1, R97.2, R98.2
- removed net N$52: C15.1, Q11.S, R90.2, R96.2, U8.RS-, U9.IN
- removed net N$53: R100.2, TP34.1, U7.IO7
- removed net N$54: D6.A, R100.1
- removed net N$55: C17.1, Q15.1.S, R86.2
- removed net N$56: C17.2, Q15.1.G, Q15.2.D, R101.2
- removed net N$58: C18.2, Q15.2.G, R102.2, R103.1
- removed net N$59: R104.1, R105.1, TP33.1, U7.IO6
- removed net N$61: D7.A, R106.1
- removed net N$62: R122.1, U10.!RESET
- removed net N$63: Q17.G, Q18.D, R123.1
- removed net N$64: Q17.D, R125.1, U11.RS+
- removed net N$65: R127.1, R128.2, TP39.1, U11.CIN1+
- removed net N$66: R129.1, R130.2, TP38.1, U11.CIN1-
- removed net N$67: R127.2, U11.IOUT
- removed net N$68: R129.2, U11.CIN2-, U11.REF
- removed net N$69: TP37.1, U11.POUT
- removed net N$70: R133.1, U11.INHIBIT
- removed net N$71: C20.1, R132.2, R133.2
- removed net N$72: C21.1, Q16.S, R125.2, R131.2, U11.RS-, U12.IN
- removed net N$73: R135.2, TP46.1, U10.IO7
- removed net N$74: D8.A, R135.1
- removed net N$75: C23.1, Q20.1.S, R121.2
- removed net N$76: C23.2, Q20.1.G, Q20.2.D, R136.2
- removed net N$77: C24.2, Q20.2.G, R137.2, R138.1
- removed net N$78: R139.1, R140.1, TP45.1, U10.IO6
- removed net N$80: D9.A, R141.1
- removed net N$81: R157.1, U13.!RESET
- removed net N$82: Q22.G, Q23.D, R158.1
- removed net N$83: Q22.D, R160.1, U14.RS+
- removed net N$84: R162.1, R163.2, TP51.1, U14.CIN1+
- removed net N$85: R164.1, R165.2, TP50.1, U14.CIN1-
- removed net N$86: R162.2, U14.IOUT
- removed net N$87: R164.2, U14.CIN2-, U14.REF
- removed net N$88: TP49.1, U14.POUT
- removed net N$89: R168.1, U14.INHIBIT
- removed net N$90: C26.1, R167.2, R168.2
- removed net N$91: C27.1, Q21.S, R160.2, R166.2, U14.RS-, U15.IN
- removed net N$92: R170.2, TP58.1, U13.IO7
- removed net N$93: D10.A, R170.1
- removed net N$94: C29.1, Q25.1.S, R156.2
- removed net N$95: C29.2, Q25.1.G, Q25.2.D, R171.2
- removed net N$96: C30.2, Q25.2.G, R172.2, R173.1
- removed net N$97: R174.1, R175.1, TP57.1, U13.IO6
- removed net ON/!OFF_Q1: Q8.G, R54.2, TP16.1, U3.IO0
- removed net ON/!OFF_Q2: Q13.G, R89.2, TP28.1, U7.IO0
- removed net ON/!OFF_Q3: Q18.G, R124.2, TP40.1, U10.IO0
- removed net ON/!OFF_Q4: Q23.G, R159.2, TP52.1, U13.IO0
- removed net PEN-SCL-FILT_Q1: R39.1, R43.1, R47.1, R50.2, TP23.1, U3.SCL
- removed net PEN-SCL-FILT_Q2: R74.1, R78.1, R82.1, R85.2, TP35.1, U7.SCL
- removed net PEN-SCL-FILT_Q3: R109.1, R113.1, R117.1, R120.2, TP47.1, U10.SCL
- removed net PEN-SCL-FILT_Q4: R144.1, R148.1, R152.1, R155.2, TP59.1, U13.SCL
- removed net PEN-SDA-FILT_Q1: Q10.1.D, R41.2, R45.2, R49.2, R67.1, TP24.1, U3.SDA
- removed net PEN-SDA-FILT_Q2: Q15.1.D, R102.1, R76.2, R80.2, R84.2, TP36.1, U7.SDA
- removed net PEN-SDA-FILT_Q3: Q20.1.D, R111.2, R115.2, R119.2, R137.1, TP48.1, U10.SDA
- removed net PEN-SDA-FILT_Q4: Q25.1.D, R146.2, R150.2, R154.2, R172.1, TP60.1, U13.SDA
- removed net SCL_Q1: R70.2, U3.IO3
- removed net SCL_Q2: R105.2, U7.IO3
- removed net SCL_Q3: R140.2, U10.IO3
- removed net SCL_Q4: R175.2, U13.IO3
- removed net SDA_Q1: R69.2, U3.IO4
- removed net SDA_Q2: R104.2, U7.IO4
- removed net SDA_Q3: R139.2, U10.IO4
- removed net SDA_Q4: R174.2, U13.IO4
- removed net SPARE4: J6.3
- removed net VBUSP_Q1: C8.2, Q6.D, R36.2, TP19.1
- removed net VBUSP_Q2: C14.2, Q11.D, R71.2, TP31.1
- removed net VBUSP_Q3: C20.2, Q16.D, R106.2, TP43.1
- removed net VBUSP_Q4: C26.2, Q21.D, R141.2, TP55.1
- removed net VPD_Q1: C12.1, C7.2, Q10.2.S, R37.2, R38.2, R42.2, R46.2, R52.2, R64.2, R68.2, TP20.1, U3.V+
- removed net VPD_Q2: C13.2, C18.1, Q15.2.S, R103.2, R72.2, R73.2, R77.2, R81.2, R87.2, R99.2, TP32.1, U7.V+
- removed net VPD_Q3: C19.2, C24.1, Q20.2.S, R107.2, R108.2, R112.2, R116.2, R122.2, R134.2, R138.2, TP44.1, U10.V+
- removed net VPD_Q4: C25.2, C30.1, Q25.2.S, R142.2, R143.2, R147.2, R151.2, R157.2, R169.2, R173.2, TP56.1, U13.V+
- new net !FAULT_Q_: Q5.D, R34.1, TP12.1, U1.IO2
- new net AD0_Q_: R10.2, R11.1, R12.2, R9.1, U1.AD0
- new net AD1_Q_: R5.1, R6.2, R7.1, R8.2, U1.AD1
- new net AD2_Q_: R1.1, R2.2, R3.1, R4.2, U1.AD2
- new net BOOT_Q_: U1.IO5
- new net CB-RESET_Q_: R32.2, TP11.1, U1.IO1, U2.CIN2+
- new net CB_CTRL_Q_: Q4.G, Q5.G, R33.1, U2.COUT1, U2.COUT2, U2.LE
- new net MAX4211-3V3_Q_: C5.1, U2.VCC, U5.OUT
- new net N$10: TP2.1, U2.POUT
- new net N$11: R26.1, U2.INHIBIT
- new net N$12: C6.1, R25.2, R26.2
- new net N$13: C4.1, Q4.S, R27.2, R33.2, U2.RS-, U5.IN
- new net N$14: R21.2, TP9.1, U1.IO7
- new net N$15: D1.A, R21.1
- new net N$16: C2.1, Q1.1.S, R17.2
- new net N$17: C2.2, Q1.1.G, Q1.2.D, R18.2
- new net N$18: C3.2, Q1.2.G, R19.2, R20.1
- new net N$19: R14.1, R15.1, TP8.1, U1.IO6
- new net N$2: D2.A, R35.1
- new net N$3: R13.1, U1.!RESET
- new net N$4: Q2.G, Q3.D, R23.1
- new net N$5: Q2.D, R27.1, U2.RS+
- new net N$6: R28.1, R30.2, TP4.1, U2.CIN1+
- new net N$7: R29.1, R31.2, TP3.1, U2.CIN1-
- new net N$8: R28.2, U2.IOUT
- new net N$9: R29.2, U2.CIN2-, U2.REF
- new net ON/!OFF_Q_: Q3.G, R24.2, TP10.1, U1.IO0
- new net PEN-SCL-FILT_Q_: R10.1, R16.2, R2.1, R6.1, TP6.1, U1.SCL
- new net PEN-SDA-FILT_Q_: Q1.1.D, R11.2, R19.1, R3.2, R7.2, TP7.1, U1.SDA
- new net SCL_Q_: R15.2, U1.IO3
- new net SDA_Q_: R14.2, U1.IO4
- new net VBUSP_Q_: C6.2, Q4.D, R35.2, TP5.1
- new net VPD_Q_: C1.2, C3.1, Q1.2.S, R1.2, R13.2, R20.2, R22.2, R34.2, R5.2, R9.2, TP1.1, U1.V+
- net GND: now also C1.1, C4.2, C5.2, D1.C, D2.C, Q3.S, Q5.S, R12.1, R18.1, R24.1, R25.1, R30.1, R31.1, R32.1, R4.1, R8.1, U1.GND, U2.GND, U5.GND; no longer C10.2, C13.1, C15.2, C16.2, C19.1, C21.2, C22.2, C25.1, C27.2, C28.2, C7.1, C9.2, D10.C, D3.C, D4.C, D5.C, D6.C, D7.C, D8.C, D9.C, J6.27, J6.28, J6.29, J6.30, J6.31, J6.32, J6.37, J6.38, Q13.S, Q14.S, Q18.S, Q19.S, Q23.S, Q24.S, Q8.S, Q9.S, R101.1, R110.1, R114.1, R118.1, R124.1, R126.1, R128.1, R130.1, R132.1, R136.1, R145.1, R149.1, R153.1, R159.1, R161.1, R163.1, R165.1, R167.1, R171.1, R40.1, R44.1, R48.1, R54.1, R56.1, R58.1, R60.1, R62.1, R66.1, R75.1, R79.1, R83.1, R89.1, R91.1, R93.1, R95.1, R97.1, U10.GND, U11.GND, U12.GND, U13.GND, U14.GND, U15.GND, U3.GND, U4.GND, U6.GND, U7.GND, U8.GND, U9.GND
- net OPD_PWR: now also R22.1; no longer J6.15, J6.16, R107.1, R142.1, R37.1, R72.1
- net OPD_SCL: now also R16.1; no longer J6.13, J6.14, R120.1, R155.1, R50.1, R85.1
- net OPD_SDA: now also R17.1; no longer J6.11, J6.12, R121.1, R156.1, R51.1, R86.1
- net VBUS: now also Q2.S, R23.2; no longer J6.21, J6.22, J6.23, J6.24, J6.25, J6.26, JP10.1, JP10.2, JP10.3, JP10.4, Q12.S, Q17.S, Q22.S, Q7.S, R123.2, R158.2, R53.2, R88.2
Other:
- note removed: "3.1"
- note removed: "All caps are 0402 ceramic 10% X5R Vw>=16V unless marked"
- note removed: "All resistors 0402 +/- 1% unless marked"
- note removed: "Main OreSat Card Connector"
- note removed: "OreSat Power Domain signals (See power sheet)"
- note removed: "OreSat Proto-Card"
