File: eaglecad/controller_rev4.2.sch (EAGLE design)
At the start: 84 parts, among them J1 J-SAMTEC-TFM-110-X1-XXX-D-RA, J2 U.FL, J3 U.FL, J4 U.FL, J6 J-SAMTEC-TFM-120-X1-XXX-D-RA, Q1 DMP2240UDM, Q3 MOSFET-PCH-SOT23-6, Q4 MOSFET-PCH-SOT23-6, Q5 PMV45EN, Q6 PMV45EN, U3 MAX7310ATE, U4 MAX4211CETE, U7 MCP1703A

Commit message: Board connector update
Parts:
- removed C1: 100n, rcl_custom:C-EU0402-B-NOSILK
- removed C2: NP, rcl_custom:C-EU0402-B-NOSILK
- removed C4, C5: 1u, oresat-rcl:C-EU0603-B-NOSILK
- removed C6, C8: TBD, rcl_custom:C-EU0402-B-NOSILK
- removed CM1, CM2, CM3: J-MOLEX-SMPM-73300-003X, J-Molex-SMPM-73300-003X:J-MOLEX-SMPM-73300-003X
- removed D1: GREEN, SparkFun-LED:LED-GREEN0603
- removed D4: AMBER, SparkFun-LED:LED-GREEN0603
- removed H1, H2, H3, H4: STAND-OFFTIGHT, SparkFun-Hardware:STAND-OFFTIGHT
- removed J1: J-SAMTEC-TFM-110-X1-XXX-D-RA, J-Samtec-TFM-110-X1-XXX-D-RA:J-SAMTEC-TFM-110-X1-XXX-D-RA
- removed J2, J3, J4: U.FL, SparkFun-Connectors:U.FL2PIN
- removed J6: J-SAMTEC-TFM-120-X1-XXX-D-RA, J-Samtec-TFM-120-X1-XXX-D-RA:J-SAMTEC-TFM-120-X1-XXX-D-RA
- removed JP1: (no value), pinhead:PINHD-1X6
- removed JP10: (no value), pinhead:PINHD-2X5
- removed JP11: (no value), pinhead:PINHD-2X6
- removed JP3: (no value), pinhead:PINHD-1X3
- removed JP5, JP6: (no value), pinhead:PINHD-1X5
- removed JP9: (no value), pinhead:PINHD-1X10
- removed Q1: DMP2240UDM, Q-MOSFET-PCH-dual-SOT23-6:MOSFET-PCH-SOT23-6
- removed Q3, Q4: MOSFET-PCH-SOT23-6, Q-MOSFET-PCH-SOT23-6:MOSFET-PCH-SOT23-6
- removed Q5, Q6: PMV45EN, Tova:PMV45EN
- removed R1, R12: 2.7k, rcl_custom:R-US_0402-B-NOSILK
- removed R11, R13, R14, R19, R20, R21, R22, R23, R32, R34, R36, R37, R5, R6, R8, R9: NP, rcl_custom:R-US_0402-B-NOSILK
- removed R15, R16, R18, R26, R27, R28, R30, R35, R38: 10k, rcl_custom:R-US_0402-B-NOSILK
- removed R24, R25, R4: 100, rcl_custom:R-US_0402-B-NOSILK
- removed R29: 100m, rcl:R-US_R1206
- removed R31, R33: 0, rcl_custom:R-US_0402-B-NOSILK
- removed TP10, TP11, TP12, TP13, TP14, TP18, TP20, TP5, TP6, TP8, TP9: TEST-POINT, Tova:TEST-POINT
- removed U3: MAX7310ATE, U-Maxim-MAX7310-I2C-GPIO-expander:MAX7310
- removed U4: MAX4211CETE, U-Maxim-MAX4211-power-monitor:MAX4211
- removed U7: MCP1703A, v-reg:XC63FPM
- added C101, C102, C106, C107, C204, C307, C310, C408: 100n, rcl_custom:C-EU0402-B-NOSILK
- added C103, C305, C405: 10n, rcl_custom:C-EU0402-B-NOSILK
- added C104, C105: 20p, rcl_custom:C-EU0402-B-NOSILK
- added C201, C202, C206, C207: 22u, oresat-rcl:C-EU0805-B-NOSILK
- added C203, C205: 10u, oresat-rcl:C-EU0603-B-NOSILK
- added C301, C302, C401, C402: 22u, oresat-rcl:C-EU0603-B-NOSILK
- added C303, C403: 2.2u, oresat-rcl:C-EU0603-B-NOSILK
- added C304, C404: 1n, rcl_custom:C-EU0402-B-NOSILK
- added C306, C409: 4.7u, oresat-rcl:C-EU0603-B-NOSILK
- added C308, C309, C410, C411: 680p, rcl_custom:C-EU0402-B-NOSILK
- added C406: 2.2n, rcl_custom:C-EU0402-B-NOSILK
- added C407: 22n, rcl_custom:C-EU0402-B-NOSILK
- added C501: DEBUG_CON, oresat-ACS_driver_board:DEBUG_CON
- added JP301: (no value), pinhead-2:PINHD-1X03_2.00
- added L201: 1.5 uH, L-Coilcraft-XFL4020:L-COILCRAFT-XFL4020
- added R101, R201, R203, R309: 10k, rcl_custom:R-US_0402-B-NOSILK
- added R202: NP, rcl_custom:R-US_0402-B-NOSILK
- added R204: 470k, rcl_custom:R-US_0402-B-NOSILK
- added R205: 150k, rcl_custom:R-US_0402-B-NOSILK
- added R301, R302, R401, R402, R406: 18k, rcl_custom:R-US_0402-B-NOSILK
- added R303, R307, R308, R409, R413, R414: 2.2k, rcl_custom:R-US_0402-B-NOSILK
- added R304, R410: 680, rcl_custom:R-US_0402-B-NOSILK
- added R305, R306, R411, R412: 0.68, oresat-rcl:R-US_0805-B-NOSILK
- added R403, R404: 330, rcl_custom:R-US_0402-B-NOSILK
- added R405: 100k, rcl_custom:R-US_0402-B-NOSILK
- added R407: 1k, rcl_custom:R-US_0402-B-NOSILK
- added R408: 47k, rcl_custom:R-US_0402-B-NOSILK
- added U100: STM32L452XX_QFPN48, oresat-ACS_driver_board:STM32L452XX_QFPN48
- added U101: TCAN330, TCAN330:TCAN330
- added U200: TPS63070, ic-pwr-tps63070x:TPS63070X
- added U300: STSPIN230, oresat-ACS_driver_board:STSPIN230
- added U301, U401: TSV991ILT, oresat-ACS_driver_board:TSV991ILT
- added U302: AS5047P, U-AMS-AS5047P-encoder:AS5047P
- added U400: STSPIN250, oresat-ACS_driver_board:STSPIN250
- added X101: ABM10-16MHz, low-gain-radio:CRYSTAL-WITH-GND
- TP1, TP2, TP3, TP4: value TEST-POINT -> TPTP06R; device Tova:TEST-POINT -> testpad:TPTP06R
- U$1: value ORESAT-CARD-V1.1-3XRF -> DRIVER-FLEX_CONN; device oresat-cards:ORESAT-CARD-V1.1-3XRF -> oresat-ACS_driver_board:DRIVER-FLEX_CONN
Connections:
- removed net !FAULT: Q6.D, R38.1, TP8.1, U3.IO2
- removed net !SHUTDOWN: J6.39, J6.40, JP1.3, JP10.10, JP10.9
- removed net AD0: R5.1, R6.2, R8.2, R9.1, U3.AD0
- removed net AD1: R11.1, R13.2, R14.2, R19.1, U3.AD1
- removed net AD2: R20.1, R21.2, R22.2, R23.1, U3.AD2
- removed net AUX_!SHUTDOWN: J1.19, J1.20, JP9.10
- removed net AUX_CAN1_H: J1.13, J1.14, JP9.7
- removed net AUX_CAN1_L: J1.15, J1.16, JP9.8
- removed net AUX_CAN2_H: J1.1, J1.2, JP9.1
- removed net AUX_CAN2_L: J1.3, J1.4, JP9.2
- removed net AUX_GND1: J1.17, J1.18, JP9.9
- removed net AUX_GND2: J1.11, J1.12, JP9.6
- removed net AUX_GND3: J1.10, J1.9, JP9.5
- removed net AUX_VBUS1: J1.7, J1.8, JP9.4
- removed net AUX_VBUS2: J1.5, J1.6, JP9.3
- removed net CAN1_H: J6.33, J6.34, JP1.1, JP10.5, JP10.6
- removed net CAN1_L: J6.35, J6.36, JP1.2, JP10.7, JP10.8
- removed net CAN2_H: J6.21, J6.22, JP11.11
- removed net CAN2_L: J6.23, J6.24, JP11.12
- removed net CB-RESET: R30.2, TP14.1, U3.IO1, U4.CIN2+
- removed net CB_CTRL: Q3.G, Q6.G, R35.1, U4.COUT1, U4.COUT2, U4.LE
- removed net MAX4211-3V3: C5.1, U4.VCC, U7.OUT
- removed net N$270: D1.A, R1.1
- removed net N$300: CM3.CENTER, J4.SIGNAL
- removed net N$398: C4.1, Q3.S, R29.2, R35.2, U4.RS-, U7.IN
- removed net N$480: TP2.1, U3.IO3
- removed net N$482: TP3.1, U3.IO4
- removed net N$518: TP4.1, U3.IO5
- removed net N$523: TP5.1, U3.IO6
- removed net N$573: R12.2, TP10.1, U3.IO7
- removed net N$575: D4.A, R12.1
- removed net N$579: C6.1, Q1.1.S, R25.2
- removed net N$580: C6.2, Q1.1.G, Q1.2.D, R15.2
- removed net N$581: C8.2, Q1.2.G, R16.2, R18.1
- removed net N$589: R26.1, U3.!RESET
- removed net N$590: Q4.G, Q5.D, R27.1
- removed net N$593: Q4.D, R29.1, U4.RS+
- removed net N$596: R31.1, R32.2, TP12.1, U4.CIN1+
- removed net N$597: R33.1, R34.2, TP11.1, U4.CIN1-
- removed net N$598: R31.2, U4.IOUT
- removed net N$599: R33.2, U4.CIN2-, U4.REF
- removed net N$600: TP6.1, U4.POUT
- removed net N$603: C2.1, R36.2, R37.2
- removed net N$604: R37.1, U4.INHIBIT
- removed net ON/!OFF: Q5.G, R28.2, TP13.1, U3.IO0
- removed net OPD_PWR: J6.19, J6.20, R4.1
- removed net OPD_SCL: J6.17, J6.18, R24.1
- removed net OPD_SDA: J6.15, J6.16, R25.1
- removed net PEN-SCL-FILT: R13.1, R21.1, R24.2, R6.1, TP18.1, U3.SCL
- removed net PEN-SDA-FILT: Q1.1.D, R16.1, R19.2, R23.2, R9.2, TP20.1, U3.SDA
- removed net RF1: CM1.CENTER, J2.SIGNAL
- removed net RF2: CM2.CENTER, J3.SIGNAL
- removed net SPARE1: J6.13, J6.14, JP11.8
- removed net SPARE2: J6.11, J6.12, JP11.7
- removed net SPARE3: J6.10, J6.9, JP11.6
- removed net SPARE4: J6.7, J6.8, JP11.5
- removed net SPARE5: J6.5, J6.6, JP11.4
- removed net SPARE6: J6.3, J6.4, JP11.3
- removed net SPARE7: J6.1, J6.2, JP11.2
- removed net VBUSP: C2.2, JP1.5, JP3.1, JP3.2, JP3.3, Q3.D, R1.2, TP9.1
- removed net VPD: C1.2, C8.1, Q1.2.S, R11.2, R18.2, R20.2, R26.2, R38.2, R4.2, R5.2, TP1.1, U3.V+
- new net 250_REF: C406.1, R405.2, R406.1, U400.REF
- new net 250_TOFF: R407.1, R408.1, U400.TOFF
- new net AS5047_MOSI: R309.2, U302.MOSI
- new net BLDC_CURR_FDB: C309.1, R307.2, U100.PA1, U301.OUT
- new net BLDC_EN: R302.2, U100.PA12
- new net BLDC_FAULT: C305.1, R302.1, U100.PA11, U300.EN/FAULT
- new net BLDC_INUH: U100.PB13, U300.INUH
- new net BLDC_INUL: U100.PA8, U300.INUL
- new net BLDC_INVH: U100.PB14, U300.INVH
- new net BLDC_INVL: U100.PA9, U300.INVL
- new net BLDC_INWH: U100.PB15, U300.INWH
- new net BLDC_INWL: U100.PA10, U300.INWL
- new net BLDC_STBY: C304.1, R301.2, TP2.TP, U100.PB12, U300.STBY/RESET
- new net BOOT: R101.2, TP4.TP, U$1.BOOT, U100.PH3-BOOT0
- new net B_IN+: C308.1, R303.1, R304.2, U301.IN+
- new net B_IN-: C309.2, R307.1, R308.2, U301.IN-
- new net CAN_H: U$1.CAN_H, U101.CANH
- new net CAN_L: U$1.CAN_L, U101.CANL
- new net CAN_RX: U100.PB5, U101.RXD
- new net CAN_SHDN: TP1.TP, U101.SHDN
- new net CAN_SILENT: U100.PB4, U101.S
- new net CAN_TX: U100.PB6, U101.TXD
- new net CLK1: C104.1, U100.PH0-OSC_IN, X101.2
- new net CLK2: C105.1, U100.PH1-OSC_OUT, X101.1
- new net DEBUG_1: C501.3, U100.PB2
- new net DEBUG_2: C501.4, U100.PB1
- new net I2C_SCL: U$1.SCL, U100.PB10
- new net I2C_SDA: U$1.SDA, U100.PB11
- new net MAG_CURR_FDB: C411.1, R413.2, U100.PA0, U401.OUT
- new net MAG_DIR: R403.2, U100.PB3
- new net MAG_EN: R402.2, U100.PB9
- new net MAG_FAULT: C405.1, R402.1, U100.PB8, U400.EN/FAULT
- new net MAG_PWM: R404.2, U100.PA15
- new net MAG_STBY: C404.1, R401.2, TP3.TP, U100.PB7, U400.STBY/RESET
- new net M_IN+: C410.1, R409.1, R410.2, U401.IN+
- new net M_IN-: C411.2, R413.1, R414.2, U401.IN-
- new net M_PH: R403.1, U400.PH
- new net M_PWM: R404.1, U400.PWM
- new net NRST: C106.1, C501.7, U100.NRST
- new net OUT1: U$1.MAG2, U400.OUTA1, U400.OUTB1
- new net OUT2: U$1.MAG1, U400.OUTA2, U400.OUTB2
- new net SENSE_BLDC: R304.1, R305.2, R306.2, U300.SENSEU, U300.SENSEVW
- new net SENSE_MAG: R410.1, R411.1, R412.1, U400.SENSEA, U400.SENSEB
- new net SPI1_CS: U100.PA4, U302.CSN
- new net SPI1_MISO: U100.PA6, U302.MISO
- new net SPI1_SCK: U100.PA5, U302.SCLK
- new net SWCLK: C501.9, U100.PA14
- new net SWDIO: C501.8, U100.PA13
- new net TOFF1: C407.1, R407.2
- new net TPS-EN2: R201.1, R202.2, U200.EN, U200.PS/SYNC
- new net TPS-FB2: R204.1, R205.2, U200.FB
- new net TPS-L5: L201.1, U200.L1
- new net TPS-L6: L201.2, U200.L2
- new net TPS-VAUX2: C204.1, U200.VAUX
- new net TPS-VSEL2: R203.2, U200.VSEL
- new net U: JP301.1, U300.OUTU
- new net UART_RX: C501.5, U100.PA3
- new net UART_TX: C501.6, U100.PA2
- new net V: JP301.2, U300.OUTV
- new net V_BATT: U$1.VCC
- new net W: JP301.3, U300.OUTW
- net 3.3V: now also C101.1, C102.1, C103.1, C107.1, C205.1, C206.1, C207.1, C306.1, C307.1, C310.1, C408.1, C409.1, C501.2, R204.2, R301.1, R303.2, R309.1, R401.1, R405.1, R409.2, U100.VBAT, U100.VDD, U100.VDDA, U101.VCC, U200.VOUT, U301.VCC, U302.VDD, U302.VDD3V, U401.VCC; no longer JP1.4, JP5.1, JP5.2, JP5.3, JP5.4, JP5.5, JP6.1, JP6.2, JP6.3, JP6.4, JP6.5
- net GND: now also C101.2, C102.2, C103.2, C104.2, C105.2, C106.2, C107.2, C201.2, C202.2, C203.2, C204.2, C205.2, C206.2, C207.2, C301.2, C302.2, C303.2, C304.2, C305.2, C306.2, C307.2, C308.2, C310.2, C401.2, C402.2, C403.2, C404.2, C405.2, C406.2, C407.2, C408.2, C409.2, C410.2, C501.10, R101.1, R202.1, R203.1, R205.1, R305.1, R306.1, R308.1, R406.2, R408.2, R411.2, R412.2, R414.1, U$1.GND, U100.VDDUSB, U100.VSS, U100.VSSA, U101.GND, U200.GND, U200.PGND, U300.GND, U301.GND, U302.GND, U302.TEST, U400.GND, U400.TEST0, U400.TEST1, U401.GND, X101.SHIELD; no longer C1.1, C4.2, C5.2, CM1.SHIELD, CM1.SHIELD1, CM1.SHIELD2, CM1.SHIELD3, CM2.SHIELD, CM2.SHIELD1, CM2.SHIELD2, CM2.SHIELD3, CM3.SHIELD, CM3.SHIELD1, CM3.SHIELD2, CM3.SHIELD3, D1.C, D4.C, J2.GND, J3.GND, J4.GND, J6.29, J6.30, J6.31, J6.32, J6.37, J6.38, JP1.6, JP11.10, JP11.9, Q5.S, Q6.S, R14.1, R15.1, R22.1, R28.1, R30.1, R32.1, R34.1, R36.1, R8.1, U3.GND, U4.GND, U7.GND
- net VBUS: now also C201.1, C202.1, C203.1, C301.1, C302.1, C303.1, C401.1, C402.1, C403.1, C501.1, R201.2, U200.VIN, U300.VS, U400.VS; no longer J6.25, J6.26, J6.27, J6.28, JP10.1, JP10.2, JP10.3, JP10.4, Q4.S, R27.2
Other:
- note added: "0805"
- note added: "3.3V SPS"
- note added: "4.2"
- note added: "ACS Controller"
- note added: "ASC BOARD CONNECTORS"
- note added: "BLDC ENCODER"
- note added: "BLDC Motor Driver"
- note added: "CON501"
- note added: "CONNECTION TO ACS DRIVER PROG. ADDAPTER"
- note added: "CONNECTION TO STANDARD ORESAT CARD"
- note added: "Correct command is FF!"
- note added: "DEBUG CONN"
- note added: "Magnetorquer Driver"
- note added: "STM32 Control"
- note added: "STM32 PWM"
- note added: "STM32 SPI"
- note added: "TO BLDC MOTOR"
- note added: "TO ORESAT CARD CONNECTION"
- note added: "Voltage divider biases the REF pin to 0.50V."
- note removed: "(3.3V)"
- note removed: "3.1"
- note removed: "Address selection for Card (See MAX7310 datasheet)"
- note removed: "All caps are 0402 ceramic 10% X5R Vw>=16V unless marked"
- note removed: "All resistors 0402 +/- 1% unless marked"
- note removed: "Auxiliary Connector"
- note removed: "Breakouts"
- note removed: "Card Power Switch and Circuit Breaker"
- note removed: "Main OreSat Card Connector"
- note removed: "Main Power Switch"
- note removed: "OreSat Power Domain (OPD) Controller"
- note removed: "OreSat Power Domain (OPD) Power Supply (3.3V)"
- note removed: "OreSat Power Domain signals (See power sheet)"
- note removed: "OreSat Power Enable (PEN)"
- note removed: "OreSat Proto-Card"
- note removed: "RF connections and test points"
- note removed: "Vbus = (6.0,7.2,8.4)V"

Commit message: rev4.2 ready for review
Parts:
- removed TP1, TP2, TP3, TP4: TPTP06R, testpad:TPTP06R
Connections:
- removed net V_BATT: U$1.VCC
- net BLDC_STBY: no longer TP2.TP
- net BOOT: no longer TP4.TP
- net CAN_SHDN: no longer TP1.TP
- net MAG_STBY: no longer TP3.TP
- net OUT1: now also U$1.MAG1; no longer U$1.MAG2
- net OUT2: now also U$1.MAG2; no longer U$1.MAG1
- net VBUS: now also U$1.VCC
Other:
- note added: "SHUTDOWN FEATURE NOT USED"
Changed lines of the file:
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@@
 </part>
 <part name="JP301" library="pinhead-2" deviceset="PINHD-1X03" device="_2.00"/>
-<part name="TP1" library="testpad" library_urn="urn:adsk.eagle:library:385" deviceset="TP" device="TP06R" package3d_urn="urn:adsk.eagle:package:27954/1" value="TPTP06R"/>
-<part name="TP2" library="testpad" library_urn="urn:adsk.eagle:library:385" deviceset="TP" device="TP06R" package3d_urn="urn:adsk.eagle:package:27954/1"/>
-<part name="TP3" library="testpad" library_urn="urn:adsk.eagle:library:385" deviceset="TP" device="TP06R" package3d_urn="urn:adsk.eagle:package:27954/1"/>
 <part name="R301" library="rcl_custom" deviceset="R-US_" device="0402-B-NOSILK" value="18k">
 <attribute name="DIS" value="Digi-Key"/>
@@
 <part name="GND17" library="supply1" deviceset="GND" device=""/>
 <part name="U$1" library="oresat-ACS_driver_board" deviceset="DRIVER-FLEX_CONN" device=""/>
-<part name="TP4" library="testpad" library_urn="urn:adsk.eagle:library:385" deviceset="TP" device="TP06R" package3d_urn="urn:adsk.eagle:package:27954/1" value="TPTP06R"/>
 </parts>
 <sheets>
@@
 <text x="78.74" y="139.7" size="1.778" layer="95">CON501</text>
 <text x="76.2" y="106.68" size="1.778" layer="96">DEBUG CONN</text>
+<text x="210.82" y="42.418" size="1.778" layer="97">SHUTDOWN FEATURE NOT USED</text>
 </plain>
 <instances>
@@
 <attribute name="VALUE" x="95.504" y="62.23" size="1.778" layer="96" rot="MR0"/>
 </instance>
-<instance part="TP1" gate="G$1" x="226.06" y="45.72" smashed="yes">
-<attribute name="NAME" x="227.33" y="44.45" size="1.778" layer="95"/>
-<attribute name="TP_SIGNAL_NAME" x="227.33" y="44.45" size="1.778" layer="97"/>
-</instance>
 <instance part="C203" gate="CE" x="176.53" y="226.06" smashed="yes">
 <attribute name="DIS" x="176.53" y="226.06" size="1.778" layer="96" display="off"/>
@@
 </instance>
 <instance part="U$1" gate="G$1" x="88.9" y="81.28" smashed="yes" rot="MR0"/>
-<instance part="TP4" gate="G$1" x="142.24" y="81.28" smashed="yes">
-<attribute name="NAME" x="139.954" y="82.042" size="1.778" layer="95"/>
-<attribute name="TP_SIGNAL_NAME" x="143.51" y="80.01" size="1.778" layer="97"/>
-</instance>
 </instances>
 <busses>
@@
 <segment>
 <pinref part="U101" gate="G$1" pin="SHDN"/>
-<label x="208.28" y="43.18" size="1.778" layer="95"/>
-<pinref part="TP1" gate="G$1" pin="TP"/>
-<wire x1="226.06" y1="43.18" x2="208.28" y2="43.18" width="0.1524" layer="91"/>
+<wire x1="210.058" y1="43.18" x2="208.28" y2="43.18" width="0.1524" layer="91"/>
 </segment>
 </net>
@@
 <wire x1="93.98" y1="134.62" x2="87.884" y2="134.62" width="0.1524" layer="91"/>
 </segment>
+<segment>
+<pinref part="U$1" gate="G$1" pin="VCC"/>
+<pinref part="SUPPLY2" gate="G$1" pin="V_BATT"/>
+<wire x1="88.9" y1="91.44" x2="92.964" y2="91.44" width="0.1524" layer="91"/>
+<wire x1="92.964" y1="91.44" x2="92.964" y2="92.71" width="0.1524" layer="91"/>
+</segment>
 </net>
 <net name="TPS-EN2" class="0">
@@
 <wire x1="144.78" y1="101.6" x2="144.78" y2="78.74" width="0.1524" layer="91"/>
 <pinref part="U$1" gate="G$1" pin="BOOT"/>
-<wire x1="144.78" y1="78.74" x2="142.24" y2="78.74" width="0.1524" layer="91"/>
 <pinref part="R101" gate="R" pin="2"/>
 <junction x="144.78" y="78.74"/>
-<pinref part="TP4" gate="G$1" pin="TP"/>
-<wire x1="142.24" y1="78.74" x2="88.9" y2="78.74" width="0.1524" layer="91"/>
-<junction x="142.24" y="78.74"/>
+<wire x1="144.78" y1="78.74" x2="88.9" y2="78.74" width="0.1524" layer="91"/>
 </segment>
 </net>
@@
 <net name="OUT2" class="0">
 <segment>
-<wire x1="90.424" y1="76.2" x2="91.44" y2="76.2" width="0.1524" layer="91"/>
+<label x="92.964" y="73.66" size="1.27" layer="95" xref="yes"/>
+<pinref part="U$1" gate="G$1" pin="MAG2"/>
+<wire x1="92.964" y1="73.66" x2="88.9" y2="73.66" width="0.1524" layer="91"/>
+</segment>
+</net>
+<net name="OUT1" class="0">
+<segment>
 <label x="92.964" y="76.2" size="1.27" layer="95" xref="yes"/>
 <pinref part="U$1" gate="G$1" pin="MAG1"/>
-<wire x1="91.44" y1="76.2" x2="92.964" y2="76.2" width="0.1524" layer="91"/>
-<wire x1="90.424" y1="76.2" x2="88.9" y2="76.2" width="0.1524" layer="91"/>
-</segment>
-</net>
-<net name="OUT1" class="0">
-<segment>
-<wire x1="90.424" y1="73.66" x2="91.44" y2="73.66" width="0.1524" layer="91"/>
-<label x="92.964" y="73.66" size="1.27" layer="95" xref="yes"/>
-<pinref part="U$1" gate="G$1" pin="MAG2"/>
-<wire x1="91.44" y1="73.66" x2="92.964" y2="73.66" width="0.1524" layer="91"/>
-<wire x1="90.424" y1="73.66" x2="88.9" y2="73.66" width="0.1524" layer="91"/>
+<wire x1="92.964" y1="76.2" x2="88.9" y2="76.2" width="0.1524" layer="91"/>
 </segment>
 </net>
@@
 <wire x1="132.08" y1="17.78" x2="132.08" y2="81.28" width="0.1524" layer="91"/>
 <wire x1="132.08" y1="81.28" x2="88.9" y2="81.28" width="0.1524" layer="91"/>
-</segment>
-</net>
-<net name="V_BATT" class="0">
-<segment>
-<pinref part="U$1" gate="G$1" pin="VCC"/>
-<pinref part="SUPPLY2" gate="G$1" pin="V_BATT"/>
-<wire x1="88.9" y1="91.44" x2="92.964" y2="91.44" width="0.1524" layer="91"/>
-<wire x1="92.964" y1="91.44" x2="92.964" y2="92.71" width="0.1524" layer="91"/>
 </segment>
 </net>
@@
 <attribute name="VALUE" x="252.73" y="185.42" size="1.778" layer="96"/>
 </instance>
-<instance part="TP2" gate="G$1" x="88.9" y="218.44" smashed="yes">
-<attribute name="NAME" x="87.63" y="219.71" size="1.778" layer="95"/>
-<attribute name="TP_SIGNAL_NAME" x="90.17" y="217.17" size="1.778" layer="97"/>
-</instance>
 <instance part="R301" gate="R" x="116.84" y="220.98" smashed="yes" rot="R270">
 <attribute name="DIS" x="116.84" y="220.98" size="1.778" layer="96" rot="R270" display="off"/>
@@
 <segment>
 <label x="86.36" y="215.9" size="1.778" layer="95" rot="R180" xref="yes"/>
-<pinref part="TP2" gate="G$1" pin="TP"/>
-<wire x1="88.9" y1="215.9" x2="86.36" y2="215.9" width="0.1524" layer="91"/>
 <pinref part="R301" gate="R" pin="2"/>
 <pinref part="C304" gate="CE" pin="1"/>
-<wire x1="88.9" y1="215.9" x2="116.84" y2="215.9" width="0.1524" layer="91"/>
-<junction x="88.9" y="215.9"/>
+<wire x1="86.36" y1="215.9" x2="116.84" y2="215.9" width="0.1524" layer="91"/>
 <junction x="116.84" y="215.9"/>
 <wire x1="116.84" y1="215.9" x2="119.38" y2="215.9" width="0.1524" layer="91"/>
@@
 <attribute name="VALUE" x="246.38" y="121.92" size="1.778" layer="96"/>
 </instance>
-<instance part="TP3" gate="G$1" x="99.06" y="193.04" smashed="yes">
-<attribute name="NAME" x="97.79" y="194.31" size="1.778" layer="95"/>
-<attribute name="TP_SIGNAL_NAME" x="100.33" y="191.77" size="1.778" layer="97"/>
-</instance>
 <instance part="R401" gate="R" x="121.92" y="195.58" smashed="yes" rot="R270">
 <attribute name="DIS" x="121.92" y="195.58" size="1.778" layer="96" rot="R270" display="off"/>
@@
 <net name="MAG_STBY" class="0">
 <segment>
-<wire x1="99.06" y1="190.5" x2="92.71" y2="190.5" width="0.1524" layer="91"/>
 <label x="92.71" y="190.5" size="1.778" layer="95" rot="R180" xref="yes"/>
-<pinref part="TP3" gate="G$1" pin="TP"/>
 <pinref part="R401" gate="R" pin="2"/>
 <pinref part="C404" gate="CE" pin="1"/>
-<wire x1="99.06" y1="190.5" x2="121.92" y2="190.5" width="0.1524" layer="91"/>
-<junction x="99.06" y="190.5"/>
+<wire x1="92.71" y1="190.5" x2="121.92" y2="190.5" width="0.1524" layer="91"/>
 <junction x="121.92" y="190.5"/>
 <wire x1="121.92" y1="190.5" x2="124.46" y2="190.5" width="0.1524" layer="91"/>
@@
 will not be understood (or retained) with this version.
 </note>
-<note version="8.3" severity="warning">
-Since Version 8.3, EAGLE supports the association of 3D packages
-with devices in libraries, schematics, and board files. Those 3D
-packages will not be understood (or retained) with this version.
-</note>
 </compatibility>
