File: eaglecad/oresat-proto-card.brd (EAGLE design)
At the start: 99.8 x 94.7 mm, 135 parts, among them J6 J-SAMTEC-TFM-120-X1-XXX-D-RA, Q1 DMP2240UDM, Q10 DMP2240UDM, Q2 MOSFET-PCH-SOT23-6, Q3 MOSFET-PCH-SOT23-6, Q4 MOSFET-PCH-SOT23-6, Q5 PMV45EN, Q6 PMV45EN, Q7 MOSFET-PCH-SOT23-6, Q8 PMV45EN, Q9 PMV45EN, U1 MAX7310ATE, U2 MAX4211CETE, U3 MAX7310ATE, U4 MAX4211CETE, U5 MCP1703A, U7 MCP1703A

Commit message: Oresat Card
Parts:
- moved BJ_Q2 135.5 mm to (117.2, 29.1)
- moved TP17 4.00 mm to (129.5, 21.3)
- moved R61 3.10 mm to (132.0, 17.4), turned to 270 degrees
- moved D2 1.90 mm to (128.5, 23.8)
- moved R58 0.67 mm to (139.9, 19.4), turned to 90 degrees
- moved C9 0.20 mm to (140.7, 16.9)
- moved R57 0.10 mm to (138.9, 19.4)
Routing:
- net N$13: track 0.00 -> 15.8 mm
- net CB_CTRL_Q2: track 0.00 -> 13.1 mm, vias 0 -> 2
- net N$5: track 0.00 -> 11.5 mm, vias 0 -> 2
- net MAX4211-3V3_Q2: track 0.00 -> 9.97 mm, vias 0 -> 2
- net N$6: track 3.53 -> 9.33 mm, vias 0 -> 1
- net N$8: track 0.00 -> 5.77 mm
- net N$4: track 0.00 -> 5.72 mm
- net N$9: track 4.16 -> 8.68 mm, vias 0 -> 2
- net VBUSP_Q2: track 0.00 -> 4.48 mm
- net N$2: track 0.00 -> 3.12 mm
- net VBUS: track 5.08 -> 7.93 mm
- net N$11: track 0.00 -> 2.05 mm
- net N$12: track 0.00 -> 1.90 mm
- added copper zone on layer 16, net N$5
- added copper zone on layer 16, net VBUSP_Q2

Commit message: ACS card updates
Parts:
- removed BJ_Q1, BJ_Q2: CARD-SIDE_CARD-CONNECTOR, oresat-ACS_driver_board:14-PIN_FFC-PORT
- removed C1, C3: 100n, rcl_custom:.0402-B-NOSILK
- removed C2, R10, R11, R13, R14, R17, R19, R20, R21, R22, R23, R32, R34, R5, R6, R7, R8, R9: NP, rcl_custom:.0402-B-NOSILK
- removed C4, C5: 1u, oresat-rcl:.0603-B-NOSILK
- removed C6: TBD, rcl_custom:.0402-B-NOSILK
- removed D1, D2: GREEN, SparkFun-LED:LED-0603
- removed Q1: DMP2240UDM, Q-MOSFET-PCH-dual-SOT23-6:SOT23-6
- removed Q2, Q3, Q4: MOSFET-PCH-SOT23-6, Q-MOSFET-PCH-SOT23-6:SOT23-6
- removed Q5: PMV45EN, Tova:SOT23
- removed R1, R12, R2: 2.7k, rcl_custom:.0402-B-NOSILK
- removed R15, R16, R18, R26, R27, R28, R30, R35: 10k, rcl_custom:.0402-B-NOSILK
- removed R24, R25, R3, R4: 100, rcl_custom:.0402-B-NOSILK
- removed R29: 100m, rcl:R1206
- removed R31, R33: 0, rcl_custom:.0402-B-NOSILK
- removed TP1, TP10, TP11, TP12, TP2, TP3, TP4, TP5, TP6, TP7, TP8, TP9: TEST-POINT, Tova:2MM-TEST-POINT
- removed U1: MAX7310ATE, U-Maxim-MAX7310-I2C-GPIO-expander:QFN65P400X400X80-17T210
- removed U2: MAX4211CETE, U-Maxim-MAX4211-power-monitor:QFN65P400X400X80-17T210
- removed U5: MCP1703A, v-reg:SOT23
- added C13, C19, C25: 100n, rcl_custom:.0402-B-NOSILK
- added C14, C20, C26, R108, R109, R110, R111, R112, R113, R114, R115, R116, R117, R118, R119, R128, R130, R132, R133, R143, R144, R145, R146, R147, R148, R149, R150, R151, R152, R153, R154, R163, R165, R167, R168, R73, R74, R75, R76, R77, R78, R79, R80, R81, R82, R83, R84, R93, R95, R97, R98: NP, rcl_custom:.0402-B-NOSILK
- added C15, C16, C21, C22, C27, C28: 1u, oresat-rcl:.0603-B-NOSILK
- added C17, C18, C23, C24, C29, C30: TBD, rcl_custom:.0402-B-NOSILK
- added D10, D6, D8: AMBER, SparkFun-LED:LED-0603
- added D5, D7, D9: GREEN, SparkFun-LED:LED-0603
- added Q11, Q12, Q16, Q17, Q21, Q22: MOSFET-PCH-SOT23-6, Q-MOSFET-PCH-SOT23-6:SOT23-6
- added Q13, Q14, Q18, Q19, Q23, Q24: PMV45EN, Tova:SOT23
- added Q15, Q20, Q25: DMP2240UDM, Q-MOSFET-PCH-dual-SOT23-6:SOT23-6
- added R100, R106, R135, R141, R170, R71: 2.7k, rcl_custom:.0402-B-NOSILK
- added R101, R102, R103, R122, R123, R124, R126, R131, R134, R136, R137, R138, R157, R158, R159, R161, R166, R169, R171, R172, R173, R87, R88, R89, R91, R96, R99: 10k, rcl_custom:.0402-B-NOSILK
- added R104, R105, R139, R140, R174, R175: 47k, rcl_custom:.0402-B-NOSILK
- added R107, R120, R121, R142, R155, R156, R72, R85, R86: 100, rcl_custom:.0402-B-NOSILK
- added R125, R160, R90: 100m, rcl:R1206
- added R127, R129, R162, R164, R92, R94: 0, rcl_custom:.0402-B-NOSILK
- added TP25, TP26, TP27, TP28, TP29, TP30, TP31, TP32, TP33, TP34, TP35, TP36, TP37, TP38, TP39, TP40, TP41, TP42, TP43, TP44, TP45, TP46, TP47, TP48, TP49, TP50, TP51, TP52, TP53, TP54, TP55, TP56, TP57, TP58, TP59, TP60: TEST-POINT, Tova:2MM-TEST-POINT
- added U$1: CARD-CONNECTOR_B, oresat-ACS_driver_board:30-PIN_FFC-PORT
- added U10, U13: MAX7310ATE, U-Maxim-MAX7310-I2C-GPIO-expander:QFN65P400X400X80-17T210
- added U11, U14, U8: MAX4211CETE, U-Maxim-MAX4211-power-monitor:QFN65P400X400X80-17T210
- added U12, U15, U6, U9: MCP1703A, v-reg:SOT23
- C7: value NP -> 100n
- C8: value TBD -> NP
- D3: value AMBER -> GREEN
- Q6: value PMV45EN -> MOSFET-PCH-SOT23-6; device Tova:SOT23 -> Q-MOSFET-PCH-SOT23-6:SOT23-6
- R36: value NP -> 2.7k
- R37: value NP -> 100
- R38: value 10k -> NP
- R39, R40: value 47k -> NP
- U7: value MCP1703A -> MAX7310ATE; device v-reg:SOT23 -> U-Maxim-MAX7310-I2C-GPIO-expander:QFN65P400X400X80-17T210
- moved R55 79.3 mm to (63.7, 8.70), turned to 0 degrees
- moved C9 77.9 mm to (63.0, 11.3), turned to 180 degrees
- moved Q7 75.4 mm to (68.2, 8.80), turned to 180 degrees
- moved R58 74.8 mm to (65.5, 11.4), turned to 180 degrees
- moved R57 73.7 mm to (65.5, 13.1), turned to 0 degrees
- moved Q8 73.3 mm to (72.1, 8.50), turned to 270 degrees
- moved C10 72.5 mm to (62.1, 17.6), turned to 90 degrees
- moved R59 72.1 mm to (67.4, 13.1), turned to 0 degrees
- moved R46 72.1 mm to (74.8, 7.20), turned to 180 degrees
- moved R53 72.0 mm to (70.7, 10.5), turned to 270 degrees
- moved R47 70.6 mm to (74.8, 9.00), turned to 0 degrees
- moved R60 70.5 mm to (69.3, 13.1), turned to 0 degrees
- moved R42 70.5 mm to (77.4, 7.20), turned to 180 degrees
- moved R49 69.2 mm to (74.8, 10.8), turned to 180 degrees
- moved TP15 69.1 mm to (69.5, 14.6), turned to 270 degrees
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Connections:
- removed net MAG_OUT1_Q1: BJ_Q1.P$10, BJ_Q1.P$11
- removed net MAG_OUT1_Q2: BJ_Q2.P$10, BJ_Q2.P$11
- removed net MAG_OUT2_Q1: BJ_Q1.P$8, BJ_Q1.P$9
- removed net MAG_OUT2_Q2: BJ_Q2.P$8, BJ_Q2.P$9
- removed net N$10: TP2.1, U2.13
- removed net N$11: R63.1, U2.5
- removed net N$12: C7.1, R62.2, R63.2
- removed net N$13: C9.1, Q2.4, R55.2, R61.2, U2.15, U5.3
- removed net N$14: R65.2, TP22.1, U1.12
- removed net N$15: D3.A, R65.1
- removed net N$19: R69.1, R70.1, TP21.1, U1.11
- removed net N$2: D2.A, R2.1
- removed net N$270: D1.A, R1.1
- removed net N$3: R52.1, U1.13
- removed net N$385: R39.1, R40.1, TP5.1, U3.11
- removed net N$398: C4.1, Q3.4, R29.2, R35.2, U4.15, U7.3
- removed net N$5: Q7.1, Q7.2, Q7.5, Q7.6, R55.1, U2.16
- removed net N$573: R12.2, TP10.1, U3.12
- removed net N$575: D4.A, R12.1
- removed net N$579: C6.1, Q1.5, R25.2
- removed net N$580: C6.2, Q1.1, Q1.4, R15.2
- removed net N$581: C8.2, Q1.3, R16.2, R18.1
- removed net N$589: R26.1, U3.13
- removed net N$590: Q4.3, Q5.3, R27.1
- removed net N$593: Q4.1, Q4.2, Q4.5, Q4.6, R29.1, U4.16
- removed net N$596: R31.1, R32.2, TP12.1, U4.10
- removed net N$597: R33.1, R34.2, TP11.1, U4.11
- removed net N$598: R31.2, U4.14
- removed net N$599: R33.2, U4.12, U4.9
- removed net N$6: R57.1, R58.2, TP4.1, U2.10
- removed net N$600: TP6.1, U4.13
- removed net N$603: C2.1, R36.2, R37.2
- removed net N$604: R37.1, U4.5
- removed net N$7: R59.1, R60.2, TP3.1, U2.11
- removed net N$8: R57.2, U2.14
- removed net N$9: R59.2, U2.12, U2.9
- removed net VPD: C1.2, C12.1, C3.2, C8.1, Q1.2, Q10.2, R11.2, R18.2, R20.2, R26.2, R3.2, R38.2, R4.2, R42.2, R46.2, R5.2, R52.2, R64.2, R68.2, R7.2, TP1.1, TP19.1, U1.14, U3.14
- new net !FAULT_Q3: Q19.3, R134.1, TP42.1, U10.7
- new net !FAULT_Q4: Q24.3, R169.1, TP54.1, U13.7
- new net AD0_Q3: R108.1, R109.2, R110.2, R111.1, U10.1
- new net AD0_Q4: R143.1, R144.2, R145.2, R146.1, U13.1
- new net AD1_Q3: R112.1, R113.2, R114.2, R115.1, U10.2
- new net AD1_Q4: R147.1, R148.2, R149.2, R150.1, U13.2
- new net AD2_Q3: R116.1, R117.2, R118.2, R119.1, U10.3
- new net AD2_Q4: R151.1, R152.2, R153.2, R154.1, U13.3
- new net BOOT_Q3: U10.10
- new net BOOT_Q4: U13.10
- new net CB-RESET_Q3: R126.2, TP41.1, U10.5, U11.8
- new net CB-RESET_Q4: R161.2, TP53.1, U13.5, U14.8
- new net CB_CTRL_Q3: Q16.3, Q19.1, R131.1, U11.3, U11.4, U11.6
- new net CB_CTRL_Q4: Q21.3, Q24.1, R166.1, U14.3, U14.4, U14.6
- new net MAX4211-3V3_Q3: C22.1, U11.1, U12.2
- new net MAX4211-3V3_Q4: C28.1, U14.1, U15.2
- new net N$21: D3.A, R36.1
- new net N$22: R52.1, U3.13
- new net N$24: Q7.1, Q7.2, Q7.5, Q7.6, R55.1, U4.16
- new net N$25: R57.1, R58.2, TP15.1, U4.10
- new net N$26: R59.1, R60.2, TP14.1, U4.11
- new net N$27: R57.2, U4.14
- new net N$28: R59.2, U4.12, U4.9
- new net N$29: TP13.1, U4.13
- new net N$30: R63.1, U4.5
- new net N$31: C8.1, R62.2, R63.2
- new net N$32: C9.1, Q6.4, R55.2, R61.2, U4.15, U6.3
- new net N$33: R65.2, TP22.1, U3.12
- new net N$34: D4.A, R65.1
- new net N$38: R69.1, R70.1, TP21.1, U3.11
- new net N$41: D5.A, R71.1
- new net N$42: R87.1, U7.13
- new net N$43: Q12.3, Q13.3, R88.1
- new net N$44: Q12.1, Q12.2, Q12.5, Q12.6, R90.1, U8.16
- new net N$45: R92.1, R93.2, TP27.1, U8.10
- new net N$46: R94.1, R95.2, TP26.1, U8.11
- new net N$47: R92.2, U8.14
- new net N$48: R94.2, U8.12, U8.9
- new net N$49: TP25.1, U8.13
- new net N$50: R98.1, U8.5
- new net N$51: C14.1, R97.2, R98.2
- new net N$52: C15.1, Q11.4, R90.2, R96.2, U8.15, U9.3
- new net N$53: R100.2, TP34.1, U7.12
- new net N$54: D6.A, R100.1
- new net N$55: C17.1, Q15.5, R86.2
- new net N$56: C17.2, Q15.1, Q15.4, R101.2
- new net N$58: C18.2, Q15.3, R102.2, R103.1
- new net N$59: R104.1, R105.1, TP33.1, U7.11
- new net N$61: D7.A, R106.1
- new net N$62: R122.1, U10.13
- new net N$63: Q17.3, Q18.3, R123.1
- new net N$64: Q17.1, Q17.2, Q17.5, Q17.6, R125.1, U11.16
- new net N$65: R127.1, R128.2, TP39.1, U11.10
- new net N$66: R129.1, R130.2, TP38.1, U11.11
- new net N$67: R127.2, U11.14
- new net N$68: R129.2, U11.12, U11.9
- new net N$69: TP37.1, U11.13
- new net N$70: R133.1, U11.5
- new net N$71: C20.1, R132.2, R133.2
- new net N$72: C21.1, Q16.4, R125.2, R131.2, U11.15, U12.3
- new net N$73: R135.2, TP46.1, U10.12
- new net N$74: D8.A, R135.1
- new net N$75: C23.1, Q20.5, R121.2
- new net N$76: C23.2, Q20.1, Q20.4, R136.2
- new net N$77: C24.2, Q20.3, R137.2, R138.1
- new net N$78: R139.1, R140.1, TP45.1, U10.11
- new net N$80: D9.A, R141.1
- new net N$81: R157.1, U13.13
- new net N$82: Q22.3, Q23.3, R158.1
- new net N$83: Q22.1, Q22.2, Q22.5, Q22.6, R160.1, U14.16
- new net N$84: R162.1, R163.2, TP51.1, U14.10
- new net N$85: R164.1, R165.2, TP50.1, U14.11
- new net N$86: R162.2, U14.14
- new net N$87: R164.2, U14.12, U14.9
- new net N$88: TP49.1, U14.13
- new net N$89: R168.1, U14.5
- new net N$90: C26.1, R167.2, R168.2
- new net N$91: C27.1, Q21.4, R160.2, R166.2, U14.15, U15.3
- new net N$92: R170.2, TP58.1, U13.12
- new net N$93: D10.A, R170.1
- new net N$94: C29.1, Q25.5, R156.2
- new net N$95: C29.2, Q25.1, Q25.4, R171.2
- new net N$96: C30.2, Q25.3, R172.2, R173.1
- new net N$97: R174.1, R175.1, TP57.1, U13.11
- new net ON/!OFF_Q3: Q18.1, R124.2, TP40.1, U10.4
- new net ON/!OFF_Q4: Q23.1, R159.2, TP52.1, U13.4
- new net PEN-SCL-FILT_Q3: R109.1, R113.1, R117.1, R120.2, TP47.1, U10.15
- new net PEN-SCL-FILT_Q4: R144.1, R148.1, R152.1, R155.2, TP59.1, U13.15
- new net PEN-SDA-FILT_Q3: Q20.6, R111.2, R115.2, R119.2, R137.1, TP48.1, U10.16
- new net PEN-SDA-FILT_Q4: Q25.6, R146.2, R150.2, R154.2, R172.1, TP60.1, U13.16
- new net SCL_Q3: R140.2, U10.8
- new net SCL_Q4: R175.2, U13.8
- new net SDA_Q3: R139.2, U10.9
- new net SDA_Q4: R174.2, U13.9
- new net VBUSP_Q3: C20.2, Q16.1, Q16.2, Q16.5, Q16.6, R106.2, TP43.1
- new net VBUSP_Q4: C26.2, Q21.1, Q21.2, Q21.5, Q21.6, R141.2, TP55.1
- new net VPD_Q1: C12.1, C7.2, Q10.2, R37.2, R38.2, R42.2, R46.2, R52.2, R64.2, R68.2, TP20.1, U3.14
- new net VPD_Q2: C13.2, C18.1, Q15.2, R103.2, R72.2, R73.2, R77.2, R81.2, R87.2, R99.2, TP32.1, U7.14
- new net VPD_Q3: C19.2, C24.1, Q20.2, R107.2, R108.2, R112.2, R116.2, R122.2, R134.2, R138.2, TP44.1, U10.14
- new net VPD_Q4: C25.2, C30.1, Q25.2, R142.2, R143.2, R147.2, R151.2, R157.2, R169.2, R173.2, TP56.1, U13.14
- net !FAULT_Q1: now also Q9.3, R64.1, TP18.1; no longer Q6.3, R38.1, TP8.1
- net !FAULT_Q2: now also Q14.3, R99.1, TP30.1, U7.7; no longer Q9.3, R64.1, TP16.1, U1.7
- net AD0_Q1: now also R38.1, R39.2, R40.2, R41.1; no longer R5.1, R6.2, R8.2, R9.1
- net AD0_Q2: now also R73.1, R74.2, R75.2, R76.1, U7.1; no longer R10.2, R17.2, R41.1, R7.1, U1.1
- net AD1_Q1: now also R42.1, R43.2, R44.2, R45.1; no longer R11.1, R13.2, R14.2, R19.1
- net AD1_Q2: now also R77.1, R78.2, R79.2, R80.1, U7.2; no longer R42.1, R43.2, R44.2, R45.1, U1.2
- net AD2_Q1: now also R46.1, R47.2, R48.2, R49.1; no longer R20.1, R21.2, R22.2, R23.1
- net AD2_Q2: now also R81.1, R82.2, R83.2, R84.1, U7.3; no longer R46.1, R47.2, R48.2, R49.1, U1.3
- net BOOT_Q2: now also U7.10; no longer U1.10
- net CAN2_H: no longer BJ_Q1.P$6, BJ_Q1.P$7, BJ_Q2.P$6, BJ_Q2.P$7
- net CAN2_L: no longer BJ_Q1.P$4, BJ_Q1.P$5, BJ_Q2.P$4, BJ_Q2.P$5
- net CB-RESET_Q1: now also R56.2, TP17.1; no longer R30.2, TP14.1
- net CB-RESET_Q2: now also R91.2, TP29.1, U7.5, U8.8; no longer R56.2, TP15.1, U1.5, U2.8
- net CB_CTRL_Q1: now also Q6.3, Q9.1, R61.1; no longer Q3.3, Q6.1, R35.1
- net CB_CTRL_Q2: now also Q11.3, Q14.1, R96.1, U8.3, U8.4, U8.6; no longer Q2.3, Q9.1, R61.1, U2.3, U2.4, U2.6
- net GND: now also C13.1, C15.2, C16.2, C19.1, C21.2, C22.2, C25.1, C27.2, C28.2, C7.1, D10.C, D5.C, D6.C, D7.C, D8.C, D9.C, Q13.2, Q14.2, Q18.2, Q19.2, Q23.2, Q24.2, R101.1, R110.1, R114.1, R118.1, R124.1, R126.1, R128.1, R130.1, R132.1, R136.1, R145.1, R149.1, R153.1, R159.1, R161.1, R163.1, R165.1, R167.1, R171.1, R40.1, R75.1, R79.1, R83.1, R89.1, R91.1, R93.1, R95.1, R97.1, U10.6, U10.EPAD, U11.7, U11.EPAD, U12.1, U13.6, U13.EPAD, U14.7, U14.EPAD, U15.1, U6.1, U7.6, U7.EPAD, U8.7, U8.EPAD, U9.1; no longer BJ_Q1.P$12, BJ_Q1.P$13, BJ_Q1.P$14, BJ_Q1.P$15, BJ_Q1.P$16, BJ_Q2.P$12, BJ_Q2.P$13, BJ_Q2.P$14, BJ_Q2.P$15, BJ_Q2.P$16, C1.1, C3.1, C4.2, C5.2, D1.C, D2.C, Q5.2, Q6.2, R14.1, R15.1, R17.1, R22.1, R28.1, R30.1, R32.1, R34.1, R36.1, R8.1, U1.6, U1.EPAD, U2.7, U2.EPAD, U5.1, U7.1
- net MAX4211-3V3_Q1: now also C10.1, U6.2; no longer C5.1, U7.2
- net MAX4211-3V3_Q2: now also C16.1, U8.1, U9.2; no longer C10.1, U2.1, U5.2
- net ON/!OFF_Q1: now also Q8.1, R54.2, TP16.1; no longer Q5.1, R28.2, TP13.1
- net ON/!OFF_Q2: now also Q13.1, R89.2, TP28.1, U7.4; no longer Q8.1, R54.2, TP7.1, U1.4
- net OPD_PWR: now also R107.1, R142.1, R37.1, R72.1; no longer R3.1, R4.1
- net OPD_SCL: now also R120.1, R155.1, R85.1; no longer R24.1
- net OPD_SDA: now also R121.1, R156.1, R86.1; no longer R25.1
- net PEN-SCL-FILT_Q1: now also R39.1, R43.1, R47.1, R50.2, TP23.1; no longer R13.1, R21.1, R24.2, R6.1, TP18.1
- net PEN-SCL-FILT_Q2: now also R74.1, R78.1, R82.1, R85.2, TP35.1, U7.15; no longer R10.1, R43.1, R47.1, R50.2, TP23.1, U1.15
- net PEN-SDA-FILT_Q1: now also Q10.6, R41.2, R45.2, R49.2, R67.1, TP24.1; no longer Q1.6, R16.1, R19.2, R23.2, R9.2, TP20.1
- net PEN-SDA-FILT_Q2: now also Q15.6, R102.1, R76.2, R80.2, R84.2, TP36.1, U7.16; no longer Q10.6, R41.2, R45.2, R49.2, R67.1, TP24.1, U1.16
- net SCL_Q1: now also R70.2; no longer R40.2
- net SCL_Q2: now also R105.2, U7.8; no longer R70.2, U1.8
- net SDA_Q1: now also R69.2; no longer R39.2
- net SDA_Q2: now also R104.2, U7.9; no longer R69.2, U1.9
- net VBUS: now also Q12.4, Q17.4, Q22.4, R123.2, R158.2, R88.2; no longer Q4.4, R27.2
- net VBUSP_Q1: now also C8.2, Q6.1, Q6.2, Q6.5, Q6.6, R36.2, TP19.1; no longer BJ_Q1.P$1, BJ_Q1.P$2, BJ_Q1.P$3, C2.2, Q3.1, Q3.2, Q3.5, Q3.6, R1.2, TP9.1
- net VBUSP_Q2: now also C14.2, Q11.1, Q11.2, Q11.5, Q11.6, R71.2, TP31.1; no longer BJ_Q2.P$1, BJ_Q2.P$2, BJ_Q2.P$3, C7.2, Q2.1, Q2.2, Q2.5, Q2.6, R2.2, TP17.1
Routing:
- net VPD: track 85.7 -> 0.00 mm, vias 11 -> 0
- net VPD_Q3: track 0.00 -> 44.7 mm, vias 0 -> 4
- net VPD_Q4: track 0.00 -> 44.7 mm, vias 0 -> 4
- net VPD_Q1: track 0.00 -> 35.8 mm, vias 0 -> 4
- net VPD_Q2: track 0.00 -> 34.8 mm, vias 0 -> 4
- net PEN-SDA-FILT_Q3: track 0.00 -> 30.1 mm, vias 0 -> 4
- net PEN-SDA-FILT_Q4: track 0.00 -> 30.1 mm, vias 0 -> 4
- net PEN-SCL-FILT_Q4: track 0.00 -> 19.6 mm, vias 0 -> 4
- net PEN-SCL-FILT_Q3: track 0.00 -> 19.6 mm, vias 0 -> 4
- net N$398: track 18.6 -> 0.00 mm, vias 2 -> 0
- net CB_CTRL_Q1: track 30.8 -> 13.5 mm, vias 3 -> 2
- net N$52: track 0.00 -> 17.1 mm
- net N$91: track 0.00 -> 17.1 mm
- net N$72: track 0.00 -> 17.1 mm
- net N$32: track 0.00 -> 17.1 mm
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- added copper zone on layer 16, net N$24
- added copper zone on layer 16, net N$44
- added copper zone on layer 16, net N$64
- added copper zone on layer 16, net N$83
- added copper zone on layer 16, net VBUSP_Q3
- added copper zone on layer 16, net VBUSP_Q4
- removed copper zone on layer 16, net N$398
- removed copper zone on layer 16, net N$5
- removed copper zone on layer 16, net N$593

Commit message: oresat card measurements
Parts:
- added U$3, U$4, U$5: CARD-CONNECTOR_C, oresat-ACS_driver_board:30-PIN_FFC-PORT
- moved R160 35.9 mm to (46.2, 7.50), turned to 270 degrees
- moved R142 33.7 mm to (47.3, 25.5), turned to 0 degrees
- moved R143 33.1 mm to (47.7, 23.8), turned to 90 degrees
- moved C27 33.0 mm to (43.6, 6.80), turned to 90 degrees
- moved R147 31.9 mm to (47.7, 21.2), turned to 90 degrees
- moved R151 31.4 mm to (47.7, 18.6), turned to 90 degrees
- moved R155 31.2 mm to (45.7, 26.0), turned to 270 degrees
- moved Q22 31.1 mm to (46.1, 12.0), turned to 90 degrees
- moved R144 29.8 mm to (45.9, 23.8), turned to 270 degrees
- moved R163 29.5 mm to (43.5, 9.30), turned to 90 degrees
- moved U15 29.3 mm to (40.8, 6.80), turned to 270 degrees
- moved Q23 29.3 mm to (46.4, 15.9), turned to 180 degrees
- moved R148 28.3 mm to (45.9, 21.2), turned to 270 degrees
- moved R152 27.8 mm to (45.9, 18.6), turned to 270 degrees
- moved C28 27.3 mm to (37.3, 5.90), turned to 0 degrees
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Connections:
- new net MAG1_Q1: U$1.P$25, U$1.P$26
- new net MAG1_Q2: U$3.P$5, U$3.P$6
- new net MAG1_Q3: U$4.P$5, U$4.P$6
- new net MAG1_Q4: U$5.P$5, U$5.P$6
- new net MAG2_Q1: U$1.P$28, U$1.P$29
- new net MAG2_Q2: U$3.P$2, U$3.P$3
- new net MAG2_Q3: U$4.P$2, U$4.P$3
- new net MAG2_Q4: U$5.P$2, U$5.P$3
- net BOOT_Q1: now also U$1.P$22, U$1.P$23
- net BOOT_Q2: now also U$3.P$8, U$3.P$9
- net BOOT_Q3: now also U$4.P$8, U$4.P$9
- net BOOT_Q4: now also U$5.P$8, U$5.P$9
- net CAN2_H: now also U$1.P$13, U$1.P$14, U$3.P$17, U$3.P$18, U$4.P$17, U$4.P$18, U$5.P$17, U$5.P$18
- net CAN2_L: now also U$1.P$10, U$1.P$11, U$3.P$20, U$3.P$21, U$4.P$20, U$4.P$21, U$5.P$20, U$5.P$21
- net GND: now also U$1.P$1, U$1.P$12, U$1.P$15, U$1.P$18, U$1.P$21, U$1.P$24, U$1.P$27, U$1.P$30, U$1.P$31, U$1.P$32, U$1.P$9, U$3.P$1, U$3.P$10, U$3.P$13, U$3.P$16, U$3.P$19, U$3.P$22, U$3.P$30, U$3.P$31, U$3.P$32, U$3.P$4, U$3.P$7, U$4.P$1, U$4.P$10, U$4.P$13, U$4.P$16, U$4.P$19, U$4.P$22, U$4.P$30, U$4.P$31, U$4.P$32, U$4.P$4, U$4.P$7, U$5.P$1, U$5.P$10, U$5.P$13, U$5.P$16, U$5.P$19, U$5.P$22, U$5.P$30, U$5.P$31, U$5.P$32, U$5.P$4, U$5.P$7
- net SCL_Q1: now also U$1.P$16, U$1.P$17
- net SCL_Q2: now also U$3.P$14, U$3.P$15
- net SCL_Q3: now also U$4.P$14, U$4.P$15
- net SCL_Q4: now also U$5.P$14, U$5.P$15
- net SDA_Q1: now also U$1.P$19, U$1.P$20
- net SDA_Q2: now also U$3.P$11, U$3.P$12
- net SDA_Q3: now also U$4.P$11, U$4.P$12
- net SDA_Q4: now also U$5.P$11, U$5.P$12
- net VBUSP_Q1: now also U$1.P$2, U$1.P$3, U$1.P$4, U$1.P$5, U$1.P$6, U$1.P$7, U$1.P$8
- net VBUSP_Q2: now also U$3.P$23, U$3.P$24, U$3.P$25, U$3.P$26, U$3.P$27, U$3.P$28, U$3.P$29
- net VBUSP_Q3: now also U$4.P$23, U$4.P$24, U$4.P$25, U$4.P$26, U$4.P$27, U$4.P$28, U$4.P$29
- net VBUSP_Q4: now also U$5.P$23, U$5.P$24, U$5.P$25, U$5.P$26, U$5.P$27, U$5.P$28, U$5.P$29

Commit message: ;a
Parts:
- moved R37 28.1 mm to (53.6, 7.30), turned to 180 degrees
- moved R50 27.1 mm to (55.2, 6.80), turned to 90 degrees
- moved R38 26.9 mm to (53.2, 9.00), turned to 270 degrees
- moved R51 25.2 mm to (62.2, 4.50), turned to 180 degrees
- moved R39 25.0 mm to (55.0, 9.00), turned to 90 degrees
- moved R42 24.6 mm to (53.2, 11.6), turned to 270 degrees
- moved C11 23.8 mm to (62.2, 5.50), turned to 0 degrees
- moved R41 23.3 mm to (56.8, 9.00), turned to 270 degrees
- moved R46 22.7 mm to (53.2, 14.2), turned to 270 degrees
- moved R43 22.6 mm to (55.0, 11.6), turned to 90 degrees
- moved Q10 22.1 mm to (66.6, 5.90), turned to 180 degrees
- moved R40 21.7 mm to (58.6, 9.00), turned to 90 degrees
- moved R66 21.2 mm to (64.0, 6.90), turned to 90 degrees
- moved TP24 21.2 mm to (60.0, 8.50), turned to 0 degrees
- moved R67 20.7 mm to (69.4, 7.00), turned to 90 degrees
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
Commit message: card update
Parts:
- U$1: value CARD-CONNECTOR_B -> CARD-FLEX_CONNCARD-FLEX_CONN; device oresat-ACS_driver_board:30-PIN_FFC-PORT -> oresat-ACS_driver_board:10-8_STAGGERED-PAD_CARD_CONN
- U$3, U$4, U$5: value CARD-CONNECTOR_C -> CARD-FLEX_CONNCARD-FLEX_CONN; device oresat-ACS_driver_board:30-PIN_FFC-PORT -> oresat-ACS_driver_board:10-8_STAGGERED-PAD_CARD_CONN
- moved U$5 28.9 mm to (38.9, 40.9), flipped to the top, turned to 225 degrees
- moved U$1 23.4 mm to (60.6, 59.2), flipped to the top
- moved U$3 18.1 mm to (61.0, 41.0), flipped to the top, turned to 315 degrees
- moved U$4 2.31 mm to (38.7, 59.3), flipped to the top, turned to 135 degrees
Connections:
- net BOOT_Q1: now also U$3.BOOT1, U$3.BOOT2; no longer U$1.P$22, U$1.P$23
- net BOOT_Q2: now also U$1.BOOT1, U$1.BOOT2; no longer U$3.P$8, U$3.P$9
- net BOOT_Q3: now also U$4.BOOT1, U$4.BOOT2; no longer U$4.P$8, U$4.P$9
- net BOOT_Q4: now also U$5.BOOT1, U$5.BOOT2; no longer U$5.P$8, U$5.P$9
- net CAN2_H: now also U$1.CAN_H1, U$1.CAN_H2, U$3.CAN_H1, U$3.CAN_H2, U$4.CAN_H1, U$4.CAN_H2, U$5.CAN_H1, U$5.CAN_H2; no longer U$1.P$13, U$1.P$14, U$3.P$17, U$3.P$18, U$4.P$17, U$4.P$18, U$5.P$17, U$5.P$18
- net CAN2_L: now also U$1.CAN_L1, U$1.CAN_L2, U$3.CAN_L1, U$3.CAN_L2, U$4.CAN_L1, U$4.CAN_L2, U$5.CAN_L1, U$5.CAN_L2; no longer U$1.P$10, U$1.P$11, U$3.P$20, U$3.P$21, U$4.P$20, U$4.P$21, U$5.P$20, U$5.P$21
- net GND: now also U$1.GND1, U$1.GND10, U$1.GND11, U$1.GND12, U$1.GND13, U$1.GND14, U$1.GND2, U$1.GND3, U$1.GND4, U$1.GND5, U$1.GND6, U$1.GND7, U$1.GND8, U$1.GND9, U$3.GND1, U$3.GND10, U$3.GND11, U$3.GND12, U$3.GND13, U$3.GND14, U$3.GND2, U$3.GND3, U$3.GND4, U$3.GND5, U$3.GND6, U$3.GND7, U$3.GND8, U$3.GND9, U$4.GND1, U$4.GND10, U$4.GND11, U$4.GND12, U$4.GND13, U$4.GND14, U$4.GND2, U$4.GND3, U$4.GND4, U$4.GND5, U$4.GND6, U$4.GND7, U$4.GND8, U$4.GND9, U$5.GND1, U$5.GND10, U$5.GND11, U$5.GND12, U$5.GND13, U$5.GND14, U$5.GND2, U$5.GND3, U$5.GND4, U$5.GND5, U$5.GND6, U$5.GND7, U$5.GND8, U$5.GND9; no longer U$1.P$1, U$1.P$12, U$1.P$15, U$1.P$18, U$1.P$21, U$1.P$24, U$1.P$27, U$1.P$30, U$1.P$31, U$1.P$32, U$1.P$9, U$3.P$1, U$3.P$10, U$3.P$13, U$3.P$16, U$3.P$19, U$3.P$22, U$3.P$30, U$3.P$31, U$3.P$32, U$3.P$4, U$3.P$7, U$4.P$1, U$4.P$10, U$4.P$13, U$4.P$16, U$4.P$19, U$4.P$22, U$4.P$30, U$4.P$31, U$4.P$32, U$4.P$4, U$4.P$7, U$5.P$1, U$5.P$10, U$5.P$13, U$5.P$16, U$5.P$19, U$5.P$22, U$5.P$30, U$5.P$31, U$5.P$32, U$5.P$4, U$5.P$7
- net MAG1_Q1: now also U$3.MAG11, U$3.MAG12; no longer U$1.P$25, U$1.P$26
- net MAG1_Q2: now also U$1.MAG11, U$1.MAG12; no longer U$3.P$5, U$3.P$6
- net MAG1_Q3: now also U$4.MAG11, U$4.MAG12; no longer U$4.P$5, U$4.P$6
- net MAG1_Q4: now also U$5.MAG11, U$5.MAG12; no longer U$5.P$5, U$5.P$6
- net MAG2_Q1: now also U$3.MAG21, U$3.MAG22; no longer U$1.P$28, U$1.P$29
- net MAG2_Q2: now also U$1.MAG21, U$1.MAG22; no longer U$3.P$2, U$3.P$3
- net MAG2_Q3: now also U$4.MAG21, U$4.MAG22; no longer U$4.P$2, U$4.P$3
- net MAG2_Q4: now also U$5.MAG21, U$5.MAG22; no longer U$5.P$2, U$5.P$3
- net SCL_Q1: now also U$3.SCL1, U$3.SCL2; no longer U$1.P$16, U$1.P$17
- net SCL_Q2: now also U$1.SCL1, U$1.SCL2; no longer U$3.P$14, U$3.P$15
- net SCL_Q3: now also U$4.SCL1, U$4.SCL2; no longer U$4.P$14, U$4.P$15
- net SCL_Q4: now also U$5.SCL1, U$5.SCL2; no longer U$5.P$14, U$5.P$15
- net SDA_Q1: now also U$3.SDA1, U$3.SDA2; no longer U$1.P$19, U$1.P$20
- net SDA_Q2: now also U$1.SDA1, U$1.SDA2; no longer U$3.P$11, U$3.P$12
- net SDA_Q3: now also U$4.SDA1, U$4.SDA2; no longer U$4.P$11, U$4.P$12
- net SDA_Q4: now also U$5.SDA1, U$5.SDA2; no longer U$5.P$11, U$5.P$12
- net VBUSP_Q1: now also U$3.VCC1, U$3.VCC2, U$3.VCC3, U$3.VCC4, U$3.VCC5, U$3.VCC6; no longer U$1.P$2, U$1.P$3, U$1.P$4, U$1.P$5, U$1.P$6, U$1.P$7, U$1.P$8
- net VBUSP_Q2: now also U$1.VCC1, U$1.VCC2, U$1.VCC3, U$1.VCC4, U$1.VCC5, U$1.VCC6; no longer U$3.P$23, U$3.P$24, U$3.P$25, U$3.P$26, U$3.P$27, U$3.P$28, U$3.P$29
- net VBUSP_Q3: now also U$4.VCC1, U$4.VCC2, U$4.VCC3, U$4.VCC4, U$4.VCC5, U$4.VCC6; no longer U$4.P$23, U$4.P$24, U$4.P$25, U$4.P$26, U$4.P$27, U$4.P$28, U$4.P$29
- net VBUSP_Q4: now also U$5.VCC1, U$5.VCC2, U$5.VCC3, U$5.VCC4, U$5.VCC5, U$5.VCC6; no longer U$5.P$23, U$5.P$24, U$5.P$25, U$5.P$26, U$5.P$27, U$5.P$28, U$5.P$29

Commit message: connector update
Parts:
- U$1, U$3, U$4, U$5: value CARD-FLEX_CONNCARD-FLEX_CONN -> MEZZANINE_1; device oresat-ACS_driver_board:10-8_STAGGERED-PAD_CARD_CONN -> oresat-ACS_driver_board:MEZZANINE_1
- moved U$4 10.9 mm to (40.3, 48.5), turned to 45 degrees
- moved U$5 10.6 mm to (49.4, 42.2), turned to 135 degrees
- moved U$3 10.4 mm to (59.5, 51.3), turned to 45 degrees
- moved U$1 10.4 mm to (50.4, 57.6), turned to 315 degrees
Connections:
- net BOOT_Q1: now also U$3.P$22, U$3.P$9; no longer U$3.BOOT1, U$3.BOOT2
- net BOOT_Q2: now also U$1.P$22, U$1.P$9; no longer U$1.BOOT1, U$1.BOOT2
- net BOOT_Q3: now also U$4.P$22, U$4.P$9; no longer U$4.BOOT1, U$4.BOOT2
- net BOOT_Q4: now also U$5.P$22, U$5.P$9; no longer U$5.BOOT1, U$5.BOOT2
- net CAN2_H: now also U$1.P$25, U$1.P$6, U$3.P$25, U$3.P$6, U$4.P$25, U$4.P$6, U$5.P$25, U$5.P$6; no longer U$1.CAN_H1, U$1.CAN_H2, U$3.CAN_H1, U$3.CAN_H2, U$4.CAN_H1, U$4.CAN_H2, U$5.CAN_H1, U$5.CAN_H2
- net CAN2_L: now also U$1.P$26, U$1.P$5, U$3.P$26, U$3.P$5, U$4.P$26, U$4.P$5, U$5.P$26, U$5.P$5; no longer U$1.CAN_L1, U$1.CAN_L2, U$3.CAN_L1, U$3.CAN_L2, U$4.CAN_L1, U$4.CAN_L2, U$5.CAN_L1, U$5.CAN_L2
- net GND: now also U$1.P$1, U$1.P$14, U$1.P$15, U$1.P$16, U$1.P$17, U$1.P$2, U$1.P$29, U$1.P$30, U$3.P$1, U$3.P$14, U$3.P$15, U$3.P$16, U$3.P$17, U$3.P$2, U$3.P$29, U$3.P$30, U$4.P$1, U$4.P$14, U$4.P$15, U$4.P$16, U$4.P$17, U$4.P$2, U$4.P$29, U$4.P$30, U$5.P$1, U$5.P$14, U$5.P$15, U$5.P$16, U$5.P$17, U$5.P$2, U$5.P$29, U$5.P$30; no longer U$1.GND1, U$1.GND10, U$1.GND11, U$1.GND12, U$1.GND13, U$1.GND14, U$1.GND2, U$1.GND3, U$1.GND4, U$1.GND5, U$1.GND6, U$1.GND7, U$1.GND8, U$1.GND9, U$3.GND1, U$3.GND10, U$3.GND11, U$3.GND12, U$3.GND13, U$3.GND14, U$3.GND2, U$3.GND3, U$3.GND4, U$3.GND5, U$3.GND6, U$3.GND7, U$3.GND8, U$3.GND9, U$4.GND1, U$4.GND10, U$4.GND11, U$4.GND12, U$4.GND13, U$4.GND14, U$4.GND2, U$4.GND3, U$4.GND4, U$4.GND5, U$4.GND6, U$4.GND7, U$4.GND8, U$4.GND9, U$5.GND1, U$5.GND10, U$5.GND11, U$5.GND12, U$5.GND13, U$5.GND14, U$5.GND2, U$5.GND3, U$5.GND4, U$5.GND5, U$5.GND6, U$5.GND7, U$5.GND8, U$5.GND9
- net MAG1_Q1: now also U$3.P$10, U$3.P$21; no longer U$3.MAG11, U$3.MAG12
- net MAG1_Q2: now also U$1.P$10, U$1.P$21; no longer U$1.MAG11, U$1.MAG12
- net MAG1_Q3: now also U$4.P$10, U$4.P$21; no longer U$4.MAG11, U$4.MAG12
- net MAG1_Q4: now also U$5.P$10, U$5.P$21; no longer U$5.MAG11, U$5.MAG12
- net MAG2_Q1: now also U$3.P$11, U$3.P$20; no longer U$3.MAG21, U$3.MAG22
- net MAG2_Q2: now also U$1.P$11, U$1.P$20; no longer U$1.MAG21, U$1.MAG22
- net MAG2_Q3: now also U$4.P$11, U$4.P$20; no longer U$4.MAG21, U$4.MAG22
- net MAG2_Q4: now also U$5.P$11, U$5.P$20; no longer U$5.MAG21, U$5.MAG22
- net SCL_Q1: now also U$3.P$24, U$3.P$7; no longer U$3.SCL1, U$3.SCL2
- net SCL_Q2: now also U$1.P$24, U$1.P$7; no longer U$1.SCL1, U$1.SCL2
- net SCL_Q3: now also U$4.P$24, U$4.P$7; no longer U$4.SCL1, U$4.SCL2
- net SCL_Q4: now also U$5.P$24, U$5.P$7; no longer U$5.SCL1, U$5.SCL2
- net SDA_Q1: now also U$3.P$23, U$3.P$8; no longer U$3.SDA1, U$3.SDA2
- net SDA_Q2: now also U$1.P$23, U$1.P$8; no longer U$1.SDA1, U$1.SDA2
- net SDA_Q3: now also U$4.P$23, U$4.P$8; no longer U$4.SDA1, U$4.SDA2
- net SDA_Q4: now also U$5.P$23, U$5.P$8; no longer U$5.SDA1, U$5.SDA2
- net VBUSP_Q1: now also U$3.P$12, U$3.P$13, U$3.P$18, U$3.P$19, U$3.P$27, U$3.P$28, U$3.P$3, U$3.P$4; no longer U$3.VCC1, U$3.VCC2, U$3.VCC3, U$3.VCC4, U$3.VCC5, U$3.VCC6
- net VBUSP_Q2: now also U$1.P$12, U$1.P$13, U$1.P$18, U$1.P$19, U$1.P$27, U$1.P$28, U$1.P$3, U$1.P$4; no longer U$1.VCC1, U$1.VCC2, U$1.VCC3, U$1.VCC4, U$1.VCC5, U$1.VCC6
- net VBUSP_Q3: now also U$4.P$12, U$4.P$13, U$4.P$18, U$4.P$19, U$4.P$27, U$4.P$28, U$4.P$3, U$4.P$4; no longer U$4.VCC1, U$4.VCC2, U$4.VCC3, U$4.VCC4, U$4.VCC5, U$4.VCC6
- net VBUSP_Q4: now also U$5.P$12, U$5.P$13, U$5.P$18, U$5.P$19, U$5.P$27, U$5.P$28, U$5.P$3, U$5.P$4; no longer U$5.VCC1, U$5.VCC2, U$5.VCC3, U$5.VCC4, U$5.VCC5, U$5.VCC6
