File: eaglecad/connector_cable_rev1.brd (EAGLE design)
At the start: 40 x 13.2 mm, 2 parts

Commit message: minor modifications
Other:
- board size 40 x 13.2 mm -> 40 x 13.1 mm
Changed lines of the file:
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@@
 <?xml version="1.0" encoding="utf-8"?>
 <!DOCTYPE eagle SYSTEM "eagle.dtd">
-<eagle version="9.3.0">
+<eagle version="9.4.2">
 <drawing>
 <settings>
-<setting alwaysvectorfont="yes"/>
+<setting alwaysvectorfont="no"/>
 <setting verticaltext="up"/>
 </settings>
@@
 <board>
 <plain>
-<wire x1="0" y1="4" x2="1" y2="3" width="0.01" layer="20" curve="90"/>
-<wire x1="1" y1="3" x2="5.5" y2="1.5" width="0.01" layer="20" curve="-36.869898"/>
-<wire x1="5.5" y1="1.5" x2="10" y2="0" width="0.01" layer="20" curve="36.869883"/>
-<wire x1="10" y1="0" x2="39" y2="0" width="0.01" layer="20"/>
-<wire x1="39" y1="0" x2="40" y2="1" width="0.01" layer="20" curve="90"/>
-<wire x1="40" y1="1" x2="40" y2="9" width="0.01" layer="20"/>
-<wire x1="40" y1="9" x2="39" y2="10" width="0.01" layer="20" curve="90"/>
-<wire x1="39" y1="10" x2="13" y2="10" width="0.01" layer="20"/>
-<wire x1="13" y1="10" x2="9.2" y2="11.6" width="0.01" layer="20" curve="-45.667308"/>
-<wire x1="9.2" y1="11.6" x2="5.4" y2="13.2" width="0.01" layer="20" curve="45.667308"/>
-<wire x1="5.4" y1="13.2" x2="1" y2="13.2" width="0.01" layer="20"/>
-<wire x1="1" y1="13.2" x2="0" y2="12.2" width="0.01" layer="20" curve="90"/>
-<wire x1="0" y1="12.2" x2="0" y2="4" width="0.01" layer="20"/>
 <polygon width="0.1" layer="30">
 <vertex x="23.3" y="8.6"/>
@@
 <vertex x="40" y="1.6"/>
 </polygon>
+<wire x1="1" y1="3.1" x2="1.364465625" y2="3.1" width="0.001" layer="20"/>
+<wire x1="1.364465625" y1="3.1" x2="3.132234375" y2="2.367765625" width="0.001" layer="20" curve="-45.000051"/>
+<wire x1="3.132234375" y1="2.367765625" x2="4.767765625" y2="0.732234375" width="0.001" layer="20"/>
+<wire x1="4.767765625" y1="0.732234375" x2="6.535534375" y2="0" width="0.001" layer="20" curve="45.000072"/>
+<wire x1="6.535534375" y1="0" x2="39" y2="0" width="0.001" layer="20"/>
+<wire x1="39" y1="0" x2="40" y2="1" width="0.001" layer="20" curve="90"/>
+<wire x1="40" y1="1" x2="40" y2="9" width="0.001" layer="20"/>
+<wire x1="40" y1="9" x2="39" y2="10" width="0.001" layer="20" curve="90"/>
+<wire x1="39" y1="10" x2="11.535534375" y2="10" width="0.001" layer="20"/>
+<wire x1="11.535534375" y1="10" x2="9.767765625" y2="10.732234375" width="0.001" layer="20" curve="-45.000051"/>
+<wire x1="9.767765625" y1="10.732234375" x2="8.132234375" y2="12.367765625" width="0.001" layer="20"/>
+<wire x1="8.132234375" y1="12.367765625" x2="6.364465625" y2="13.1" width="0.001" layer="20" curve="45.000072"/>
+<wire x1="6.364465625" y1="13.1" x2="1" y2="13.1" width="0.001" layer="20"/>
+<wire x1="1" y1="13.1" x2="0" y2="12.1" width="0.001" layer="20" curve="90"/>
+<wire x1="0" y1="12.1" x2="0" y2="4.1" width="0.001" layer="20"/>
+<wire x1="0" y1="4.1" x2="1" y2="3.1" width="0.001" layer="20" curve="90"/>
 </plain>
 <attributes>
@@
 <via x="19.1" y="2.5" extent="1-16" drill="0.254"/>
 <wire x1="6.9" y1="5.6" x2="10" y2="2.5" width="0.1524" layer="1"/>
-<wire x1="29.25" y1="7.5" x2="29.25" y2="7" width="0" layer="19" extent="16-16"/>
-<wire x1="23.75" y1="7" x2="23.75" y2="7.5" width="0" layer="19" extent="16-16"/>
-<wire x1="6.9" y1="6.1" x2="10" y2="7" width="0" layer="19" extent="16-16"/>
-<wire x1="23.75" y1="2.5" x2="23.75" y2="3" width="0" layer="19" extent="16-16"/>
-<wire x1="29.25" y1="3" x2="29.25" y2="7" width="0" layer="19" extent="16-16"/>
-<wire x1="29.25" y1="2.5" x2="29.25" y2="3" width="0" layer="19" extent="16-16"/>
 <polygon width="0.1" layer="16" thermals="no">
 <vertex x="23.3" y="7.1"/>
@@
 <vertex x="40" y="2.6"/>
 </polygon>
-<wire x1="20.7" y1="3" x2="23.75" y2="3" width="0" layer="19"/>
-<wire x1="23.75" y1="2.5" x2="19.1" y2="2.5" width="0" layer="19"/>
-<wire x1="21.5" y1="7" x2="23.75" y2="7" width="0" layer="19"/>
-<wire x1="19.1" y1="7.5" x2="23.75" y2="7.5" width="0" layer="19"/>
+<wire x1="23.75" y1="3" x2="23.75" y2="2.5" width="0" layer="19" extent="16-16"/>
+<wire x1="10" y1="7" x2="6.9" y2="6.1" width="0" layer="19" extent="16-16"/>
+<wire x1="23.75" y1="7.5" x2="23.75" y2="7" width="0" layer="19" extent="16-16"/>
 </signal>
 <signal name="CAN_L">
@@
 <via x="22.3" y="3.5" extent="1-16" drill="0.254"/>
 <wire x1="6.9" y1="6.6" x2="10" y2="3.5" width="0.1524" layer="1"/>
-<wire x1="23.75" y1="3.5" x2="29.25" y2="3.5" width="0" layer="19" extent="16-16"/>
 <polygon width="0.1" layer="16" thermals="no">
 <vertex x="23.3" y="3.6"/>
@@
 <vertex x="40" y="3.6"/>
 </polygon>
-<wire x1="22.3" y1="3.5" x2="23.75" y2="3.5" width="0" layer="19"/>
 </signal>
 <signal name="CAN_H">
@@
 <via x="19.9" y="4" extent="1-16" drill="0.254"/>
 <wire x1="6.9" y1="7.1" x2="10" y2="4" width="0.1524" layer="1"/>
-<wire x1="23.75" y1="4" x2="29.25" y2="4" width="0" layer="19" extent="16-16"/>
 <polygon width="0.1" layer="16" thermals="no">
 <vertex x="23.3" y="4.1"/>
@@
 <vertex x="40" y="4.1"/>
 </polygon>
-<wire x1="19.9" y1="4" x2="23.75" y2="4" width="0" layer="19"/>
 </signal>
 <signal name="SCL">
@@
 <via x="21.5" y="4.5" extent="1-16" drill="0.254"/>
 <wire x1="6.9" y1="7.6" x2="10" y2="4.5" width="0.1524" layer="1"/>
-<wire x1="23.75" y1="4.5" x2="29.25" y2="4.5" width="0" layer="19" extent="16-16"/>
 <polygon width="0.1" layer="16" thermals="no">
 <vertex x="23.3" y="4.6"/>
@@
 <vertex x="40" y="4.6"/>
 </polygon>
-<wire x1="21.5" y1="4.5" x2="23.75" y2="4.5" width="0" layer="19"/>
 </signal>
 <signal name="SDA">
@@
 <via x="19.1" y="5" extent="1-16" drill="0.254"/>
 <wire x1="6.9" y1="8.1" x2="10" y2="5" width="0.1524" layer="1"/>
-<wire x1="23.75" y1="5" x2="29.25" y2="5" width="0" layer="19" extent="16-16"/>
 <polygon width="0.1" layer="16" thermals="no">
 <vertex x="23.3" y="5.1"/>
@@
 <vertex x="40" y="5.1"/>
 </polygon>
-<wire x1="19.1" y1="5" x2="23.75" y2="5" width="0" layer="19"/>
 </signal>
 <signal name="BOOT">
@@
 <via x="20.7" y="5.5" extent="1-16" drill="0.254"/>
 <wire x1="6.9" y1="8.6" x2="10" y2="5.5" width="0.1524" layer="1"/>
-<wire x1="23.75" y1="5.5" x2="29.25" y2="5.5" width="0" layer="19" extent="16-16"/>
 <polygon width="0.1" layer="16" thermals="no">
 <vertex x="23.3" y="5.6"/>
@@
 <vertex x="40" y="5.6"/>
 </polygon>
-<wire x1="20.7" y1="5.5" x2="23.75" y2="5.5" width="0" layer="19"/>
 </signal>
 <signal name="MAG1">
@@
 <via x="22.3" y="6" extent="1-16" drill="0.254"/>
 <wire x1="6.9" y1="9.1" x2="10" y2="6" width="0.1524" layer="1"/>
-<wire x1="23.75" y1="6" x2="29.25" y2="6" width="0" layer="19" extent="16-16"/>
 <polygon width="0.1" layer="16" thermals="no">
 <vertex x="23.3" y="6.1"/>
@@
 <vertex x="40" y="6.1"/>
 </polygon>
-<wire x1="23.75" y1="6" x2="22.3" y2="6" width="0" layer="19"/>
 </signal>
 <signal name="MAG2">
@@
 <via x="19.9" y="6.5" extent="1-16" drill="0.254"/>
 <wire x1="6.9" y1="9.6" x2="10" y2="6.5" width="0.1524" layer="1"/>
-<wire x1="23.75" y1="6.5" x2="29.25" y2="6.5" width="0" layer="19" extent="16-16"/>
 <polygon width="0.1" layer="16" thermals="no">
 <vertex x="23.3" y="6.6"/>
@@
 <vertex x="40" y="6.6"/>
 </polygon>
-<wire x1="19.9" y1="6.5" x2="23.75" y2="6.5" width="0" layer="19"/>
 </signal>
 <signal name="GND">
@@
 <wire x1="6.9" y1="5.1" x2="10" y2="8" width="0" layer="19" extent="16-16"/>
 <wire x1="23.75" y1="1.5" x2="23.75" y2="2" width="0" layer="19" extent="16-16"/>
-<wire x1="19.9" y1="1.5" x2="23.75" y2="1.5" width="0" layer="19"/>
-<wire x1="21.5" y1="2" x2="23.75" y2="2" width="0" layer="19"/>
-<wire x1="20.7" y1="8" x2="23.75" y2="8" width="0" layer="19"/>
-<wire x1="22.3" y1="8.5" x2="23.75" y2="8.5" width="0" layer="19"/>
 </signal>
 </signals>
