File: eaglecad/controller_rev4.3_flat.brd (EAGLE design)
At the start: 129 parts, among them J2 J-SAMTEC-TFM-120-X1-XXX-D-RA, U100 STM32L452XX_QFPN48, U101 TCAN330, U200 TPS63070, U300 STSPIN230, U301 TSV991ILT, U302 AS5047P, U400 STSPIN250, U401 TSV991ILT, X101 ABM10-16MHz

Commit message: Board Flattened ready for review
Parts:
- removed JP301: (no value), pinhead-2:1X03M
- removed LED7: AMBER, led:CHIPLED_0603
- removed LED8: GREEN, led:CHIPLED_0603
- added J301, J302: (no value), pinhead:2X03
- added LED3, LED4: BLUE, led:CHIPLED_0603
- added LED301: CLX6E-FKC, D-Cree-CLX6E-RGB-LED:CLX6E-FKC
- added R7: 380, rcl_custom:.0402-B-NOSILK
- added R8: 400, rcl_custom:.0402-B-NOSILK
- added R9: 320, rcl_custom:.0402-B-NOSILK
- LED1: value BLUE -> AMBER
- LED2: value BLUE -> GREEN
- moved SWD1 37.0 mm to (34.7, 81.0)
- moved R1 35.9 mm to (14.3, 71.1)
- moved R2 35.9 mm to (16.8, 71.1)
- moved LED1 24.3 mm to (14.0, 72.3), turned to 90 degrees
- moved LED2 23.8 mm to (17.1, 72.3), turned to 270 degrees
- moved LED6 23.6 mm to (52.9, 85.6)
- moved LED5 18.5 mm to (50.3, 85.6)
- moved R305 16.6 mm to (49.3, 39.7)
- moved R306 16.6 mm to (51.3, 39.7)
- moved C201 16.4 mm to (29.0, 48.5)
- moved X101 16.0 mm to (41.4, 64.2)
- moved C101 16.0 mm to (39.0, 62.5)
- moved C104 16.0 mm to (39.6, 64.4)
- moved C305 16.0 mm to (40.7, 44.0)
- moved R302 16.0 mm to (40.7, 45.0)
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Connections:
- removed net V_BATT: J2.21, J2.22, J2.23, J2.24, J2.25, J2.26
- new net N$10: J301.1, J301.2
- new net N$11: J302.2, LED301.P$6
- new net N$12: J302.4, LED301.P$5
- new net N$13: J302.6, LED301.P$4
- new net N$14: LED301.P$1, R7.2
- new net N$15: LED301.P$2, R8.2
- new net N$16: LED301.P$3, R9.2
- new net N$4: J301.5, J301.6
- new net N$9: J301.3, J301.4
- net 3.3V: now also LED2.A; no longer LED8.A
- net DEBUG_1: now also LED3.A; no longer LED6.A
- net DEBUG_2: now also LED4.A; no longer LED5.A
- net DEBUG_3: now also LED5.A; no longer LED1.A
- net DEBUG_4: now also LED6.A; no longer LED2.A
- net GND: now also R7.1, R8.1, R9.1
- net N$1: now also LED5.C; no longer LED1.C
- net N$2: now also LED6.C; no longer LED2.C
- net N$5: now also LED4.C; no longer LED5.C
- net N$6: now also LED3.C; no longer LED6.C
- net N$7: now also LED1.C; no longer LED7.C
- net N$8: now also LED2.C; no longer LED8.C
- net U: now also J302.1; no longer JP301.1
- net V: now also J302.3; no longer JP301.2
- net VBUS: now also J2.21, J2.22, J2.23, J2.24, J2.25, J2.26, LED1.A; no longer LED7.A
- net W: now also J302.5; no longer JP301.3
Routing:
- net GND: track 47.4 -> 71.2 mm, vias 16 -> 200
- net NRST: track 39.8 -> 22.1 mm
- net SWDIO: track 47.6 -> 32.3 mm
- net SWCLK: track 44.7 -> 29.8 mm
- net VBUS: track 8.88 -> 20.9 mm, vias 1 -> 25
- net W: track 0.00 -> 11.5 mm
- net OUT1: track 26.6 -> 38.1 mm, vias 2 -> 3
- net 3.3V: track 32.1 -> 42.6 mm, vias 6 -> 20
- net U: track 0.00 -> 7.56 mm, vias 0 -> 1
- net V: track 0.00 -> 7.04 mm
- net TPS-L5: track 0.00 -> 6.53 mm, vias 0 -> 7
- net TPS-L6: track 0.00 -> 6.50 mm, vias 0 -> 7
- net OUT2: track 23.9 -> 30.4 mm, vias 2 -> 3
- net N$13: track 0.00 -> 5.90 mm
- net UART_RX: track 32.0 -> 37.7 mm
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- added copper zone on layer 15, net 3.3V
- added copper zone on layer 16, net 3.3V
- added copper zone on layer 1, net GND
- added copper zone on layer 16, net GND
- added copper zone on layer 15, net VBUS
- added copper zone on layer 16, net VBUS
Other:
- board outline added: 66 x 88 mm
- board text added: "ACS TestBench Rev 4.3_flat OreSat Eric Ruhl"
- board text removed: "ACS Driver OreSat Rev 4.3_flat Eric Ruhl"

Commit message: Flat ready for review for real this time
Parts:
- renumbered TP29 to 3.3V_C, TP30 to 3.3V_A, TP31 to 3.3V_B
Changed lines of the file:
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@@
 <attribute name="NAME" x="34.666" y="56.5" size="0.635" layer="26" font="vector" ratio="20" rot="MR0"/>
 </element>
-<element name="TP29" library="oresat-misc" package="1X01" value="TEST-POINT-LARGE" x="51.666" y="52.5" smashed="yes" rot="R90">
+<element name="3.3V_C" library="oresat-misc" package="1X01" value="TEST-POINT-LARGE" x="51.666" y="52.5" smashed="yes" rot="R90">
 <attribute name="BOM" value="EXCLUDE" x="51.666" y="52.5" size="1.778" layer="27" rot="R90" display="off"/>
 <attribute name="NAME" x="53.166" y="52.83" size="0.635" layer="26" font="vector" ratio="20" rot="MR180"/>
 </element>
-<element name="TP30" library="oresat-misc" package="1X01" value="TEST-POINT-LARGE" x="35.666" y="62" smashed="yes" rot="R90">
+<element name="3.3V_A" library="oresat-misc" package="1X01" value="TEST-POINT-LARGE" x="35.666" y="62" smashed="yes" rot="R90">
 <attribute name="BOM" value="EXCLUDE" x="35.666" y="62" size="1.778" layer="27" rot="R90" display="off"/>
 <attribute name="NAME" x="34.666" y="61.8" size="0.635" layer="26" font="vector" ratio="20" rot="MR0"/>
 </element>
-<element name="TP31" library="oresat-misc" package="1X01" value="TEST-POINT-LARGE" x="45.666" y="66.5" smashed="yes" rot="R90">
+<element name="3.3V_B" library="oresat-misc" package="1X01" value="TEST-POINT-LARGE" x="45.666" y="66.5" smashed="yes" rot="R90">
 <attribute name="BOM" value="EXCLUDE" x="45.666" y="66.5" size="1.778" layer="27" rot="R90" display="off"/>
 <attribute name="NAME" x="45.466" y="67.5" size="0.635" layer="26" font="vector" ratio="20" rot="MR90"/>
@@
 <contactref element="C310" pad="1"/>
 <contactref element="C107" pad="1"/>
-<contactref element="TP29" pad="1"/>
-<contactref element="TP30" pad="1"/>
-<contactref element="TP31" pad="1"/>
+<contactref element="3.3V_C" pad="1"/>
+<contactref element="3.3V_A" pad="1"/>
+<contactref element="3.3V_B" pad="1"/>
 <contactref element="SWD1" pad="VTREF"/>
 <contactref element="LED2" pad="A"/>
@@
 <wire x1="17.063" y1="40" x2="19.613" y2="42.55" width="0.26" layer="16"/>
 <wire x1="13" y1="39.92" x2="11.22" y2="41.7" width="0.26" layer="16"/>
-<wire x1="9.479" y1="51.181" x2="9.479" y2="51.71969375" width="0.26" layer="16"/>
-<wire x1="9.479" y1="51.71969375" x2="8.89869375" y2="52.3" width="0.26" layer="16"/>
-<wire x1="8.89869375" y1="52.3" x2="7.466" y2="52.3" width="0.26" layer="16"/>
+<wire x1="9.488290625" y1="51.130403125" x2="8.31869375" y2="52.3" width="0.26" layer="16"/>
+<wire x1="8.31869375" y1="52.3" x2="7.466" y2="52.3" width="0.26" layer="16"/>
 <wire x1="13" y1="39.92" x2="13.08" y2="40" width="0.26" layer="16"/>
 <wire x1="13.08" y1="40" x2="17.063" y2="40" width="0.26" layer="16"/>
-<wire x1="11.22" y1="41.7" x2="9.479" y2="51.181" width="0.26" layer="16"/>
+<wire x1="11.22" y1="41.7" x2="9.488290625" y2="51.130403125" width="0.26" layer="16"/>
 </signal>
 <signal name="SWDIO">
@@
 <wire x1="17.38" y1="37.38" x2="13" y2="37.38" width="0.26" layer="16"/>
 <wire x1="13" y1="37.38" x2="11.2" y2="39.18" width="0.26" layer="16"/>
-<wire x1="9.07" y1="51.5313875" x2="9.07" y2="50.97" width="0.26" layer="16"/>
-<wire x1="9.07" y1="51.5313875" x2="8.8013875" y2="51.8" width="0.26" layer="16"/>
-<wire x1="7.466" y1="51.8" x2="8.8013875" y2="51.8" width="0.26" layer="16"/>
+<wire x1="9.07" y1="50.9713875" x2="9.07" y2="50.97" width="0.26" layer="16"/>
+<wire x1="9.07" y1="50.9713875" x2="8.2413875" y2="51.8" width="0.26" layer="16"/>
+<wire x1="7.466" y1="51.8" x2="8.2413875" y2="51.8" width="0.26" layer="16"/>
 <wire x1="11.2" y1="39.18" x2="9.07" y2="50.97" width="0.26" layer="16"/>
 </signal>
@@
 <wire x1="16.02" y1="50" x2="13.08" y2="50" width="0.52" layer="16"/>
 <wire x1="13.08" y1="50" x2="13" y2="50.08" width="0.26" layer="16"/>
-<wire x1="11.04" y1="52.42" x2="11.04" y2="52.04" width="0.26" layer="16"/>
-<wire x1="13" y1="50.08" x2="11.04" y2="52.04" width="0.26" layer="16"/>
-<wire x1="11.04" y1="52.42" x2="9.16" y2="54.3" width="0.26" layer="16"/>
-<wire x1="9.16" y1="54.3" x2="7.466" y2="54.3" width="0.26" layer="16"/>
-<wire x1="13" y1="50.08" x2="11.04" y2="52.04" width="0.26" layer="1"/>
-<wire x1="11.04" y1="52.04" x2="11.04" y2="52.42" width="0.26" layer="1"/>
-<wire x1="11.04" y1="52.42" x2="9.16" y2="54.3" width="0.26" layer="1"/>
+<wire x1="13" y1="50.08" x2="8.78" y2="54.3" width="0.26" layer="16"/>
+<wire x1="8.78" y1="54.3" x2="7.466" y2="54.3" width="0.26" layer="16"/>
+<wire x1="13" y1="50.08" x2="8.78" y2="54.3" width="0.26" layer="1"/>
 <via x="5.82" y="54.3" extent="1-16" drill="0.254"/>
 <wire x1="5.82" y1="54.3" x2="3.466" y2="54.3" width="0.26" layer="16"/>
-<wire x1="9.16" y1="54.3" x2="5.82" y2="54.3" width="0.26" layer="1"/>
+<wire x1="8.78" y1="54.3" x2="5.82" y2="54.3" width="0.26" layer="1"/>
 </signal>
 <signal name="OUT2">
@@
 <via x="39.266" y="59.1" extent="1-16" drill="0.26"/>
 <contactref element="JP3" pad="6"/>
-<wire x1="13" y1="47.54" x2="11.15420625" y2="49.38579375" width="0.26" layer="16"/>
-<wire x1="10.646190625" y1="51.623809375" x2="10.65" y2="51.62" width="0.26" layer="16"/>
-<wire x1="10.65" y1="51.62" x2="10.65" y2="52.26" width="0.26" layer="16"/>
-<wire x1="10.65" y1="52.26" x2="9.11" y2="53.8" width="0.26" layer="16"/>
-<wire x1="9.11" y1="53.8" x2="7.466" y2="53.8" width="0.26" layer="16"/>
+<wire x1="13" y1="47.54" x2="11.18714375" y2="49.35285625" width="0.26" layer="16"/>
+<wire x1="10.65" y1="51.719190625" x2="10.65" y2="51.72" width="0.26" layer="16"/>
+<wire x1="10.65" y1="51.72" x2="8.57" y2="53.8" width="0.26" layer="16"/>
+<wire x1="8.57" y1="53.8" x2="7.466" y2="53.8" width="0.26" layer="16"/>
 <wire x1="39.266" y1="59.1" x2="37.97545" y2="57.80945" width="0.26" layer="1"/>
 <wire x1="37.97545" y1="57.80945" x2="37.97545" y2="54.6647125" width="0.26" layer="1"/>
@@
 <wire x1="25" y1="53" x2="19.54" y2="47.54" width="0.26" layer="1"/>
 <wire x1="7.466" y1="53.8" x2="3.466" y2="53.8" width="0.26" layer="16"/>
-<wire x1="11.15420625" y1="49.38579375" x2="10.646190625" y2="51.623809375" width="0.26" layer="16"/>
+<wire x1="11.18714375" y1="49.35285625" x2="10.65" y2="51.719190625" width="0.26" layer="16"/>
 </signal>
 <signal name="B_IN+">
@@
 <contactref element="JP3" pad="4"/>
 <wire x1="13" y1="42.46" x2="11.23" y2="44.23" width="0.26" layer="16"/>
-<wire x1="9.866" y1="51.394" x2="9.866" y2="51.91" width="0.26" layer="16"/>
-<wire x1="9.866" y1="51.91" x2="8.976" y2="52.8" width="0.26" layer="16"/>
-<wire x1="8.976" y1="52.8" x2="7.466" y2="52.8" width="0.26" layer="16"/>
+<wire x1="9.876346875" y1="51.339653125" x2="8.416" y2="52.8" width="0.26" layer="16"/>
+<wire x1="8.416" y1="52.8" x2="7.466" y2="52.8" width="0.26" layer="16"/>
 <wire x1="50.166" y1="55.5" x2="47.6108125" y2="52.9448125" width="0.26" layer="1"/>
 <wire x1="37.49211875" y1="52.9448125" x2="36.77330625" y2="52.226" width="0.26" layer="1"/>
@@
 <wire x1="25.3206125" y1="52.226" x2="15.5546125" y2="42.46" width="0.26" layer="1"/>
 <wire x1="3.466" y1="52.8" x2="7.466" y2="52.8" width="0.26" layer="16"/>
-<wire x1="11.23" y1="44.23" x2="9.866" y2="51.394" width="0.26" layer="16"/>
+<wire x1="11.23" y1="44.23" x2="9.876346875" y2="51.339653125" width="0.26" layer="16"/>
 </signal>
 <signal name="I2C_SDA">
@@
 <contactref element="JP3" pad="5"/>
 <wire x1="13" y1="45" x2="11.17" y2="46.83" width="0.26" layer="16"/>
-<wire x1="10.253" y1="51.6139125" x2="10.253" y2="52.08969375" width="0.26" layer="16"/>
-<wire x1="9.04269375" y1="53.3" x2="7.466" y2="53.3" width="0.26" layer="16"/>
-<wire x1="10.253" y1="52.08969375" x2="9.04269375" y2="53.3" width="0.26" layer="16"/>
+<wire x1="8.49269375" y1="53.3" x2="7.466" y2="53.3" width="0.26" layer="16"/>
+<wire x1="10.2706" y1="51.52209375" x2="8.49269375" y2="53.3" width="0.26" layer="16"/>
 <wire x1="51.666" y1="54.5" x2="51.666" y2="55.2747375" width="0.26" layer="1"/>
 <wire x1="51.666" y1="55.2747375" x2="50.5512875" y2="56.38945" width="0.26" layer="1"/>
@@
 <wire x1="25.16030625" y1="52.613" x2="17.54730625" y2="45" width="0.26" layer="1"/>
 <wire x1="3.466" y1="53.3" x2="7.466" y2="53.3" width="0.26" layer="16"/>
-<wire x1="11.17" y1="46.83" x2="10.253" y2="51.6139125" width="0.26" layer="16"/>
+<wire x1="10.2706" y1="51.52209375" x2="11.17" y2="46.83" width="0.26" layer="16"/>
 </signal>
 <signal name="ADDR_0">

Commit message: flat board ready for second round of inspection
Parts:
- removed C204: 100n, rcl_custom:.0402-B-NOSILK
- removed C205: 10u, oresat-rcl:.0603-B-NOSILK
- removed C206, C207: 22u, oresat-rcl:.0805-B-NOSILK
- removed EN, FB2, VSEL: TEST-POINT-LARGE, oresat-misc:1X01
- removed LED5, LED6: BLUE, led:CHIPLED_0603
- removed R203: 10k, rcl_custom:.0402-B-NOSILK
- removed R204: 470k, rcl_custom:.0402-B-NOSILK
- removed R205: 150k, rcl_custom:.0402-B-NOSILK
- removed R5, R6: 100, oresat-rcl:.0402-B-NOSILK
- removed U200: TPS63070, ic-pwr-tps63070x:TPS63070X
- added 3.3V, SYNC, VBUSP: TEST-POINT-LARGE-SQUARE, oresat-misc:1X01
- added R104: 10k, rcl_custom:.0402-B-NOSILK
- added R105, R106: 4.7k, rcl_custom:.0402-B-NOSILK
- added U201: TPS62111RSA, U-TI-TPS6211x-SPS-buck:S-PVQFN-16
- C201: value 22u -> 10u
- C202: value 22u -> 1u; device oresat-rcl:.0805-B-NOSILK -> oresat-rcl:.0603-C-NOSILK
- C203: value 10u -> 22u; device oresat-rcl:.0603-B-NOSILK -> oresat-rcl:.0805-B-NOSILK
- JP1: device pinhead:1X04 -> pinhead:1X02
- JP2: device pinhead:2X04 -> pinhead:2X02
- L201: value 1.5 uH -> 6.8u; device L-Coilcraft-XFL4020:L-COILCRAFT-XFL4020 -> L-ECS-MPI4040:ECS-MPI4040
- PG: value TEST-POINT-LARGE -> TEST-POINT-LARGE-SQUARE
- R201, R202: device rcl_custom:.0402-B-NOSILK -> oresat-rcl:.0603-C-NOSILK
- moved LED2 32.4 mm to (15.3, 39.9), turned to 0 degrees
- moved R2 31.0 mm to (14.1, 40.2), turned to 90 degrees
- moved LED1 29.4 mm to (15.3, 43.0), turned to 180 degrees
- moved R1 28.3 mm to (14.1, 42.7), turned to 270 degrees
- moved JP2 21.7 mm to (52.5, 97.3), flipped to the top, turned to 0 degrees
- moved R412 21.5 mm to (18.0, 85.0), turned to 90 degrees
- moved J1 20.2 mm to (18.4, 97.5), turned to 180 degrees
- moved R411 18.9 mm to (21.0, 85.0), turned to 90 degrees
- moved R307 18.0 mm to (54.6, 65.3)
- moved R413 17.7 mm to (40.4, 84.8)
- moved R410 17.7 mm to (23.6, 84.6), turned to 90 degrees
- moved R414 17.6 mm to (37.5, 83.7), turned to 90 degrees
- moved C411 17.0 mm to (33.4, 84.8)
- moved C408 17.0 mm to (33.4, 86.2)
- moved C409 17.0 mm to (30.9, 87.7)
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Connections:
- removed net CAN_SHDN: U101.5
- removed net DEBUG_3: JP1.3, JP2.1, LED5.A
- removed net DEBUG_4: JP1.4, JP2.5, LED6.A
- removed net FB2: FB2.1, U200.6
- removed net N$11: J302.2, LED301.P$6
- removed net N$13: J302.6, LED301.P$4
- removed net N$2 (its old number): LED6.C, R6.2
- removed net PG: PG.1, U200.2
- removed net TPS-EN2: EN.1, R201.1, R202.2, U200.1, U200.14
- removed net TPS-FB2: R204.1, R205.2, U200.5
- removed net TPS-L5: L201.1, U200.11
- removed net TPS-L6: L201.2, U200.9
- removed net TPS-VAUX2: C204.1, U200.3
- removed net TPS-VSEL2: R203.2, U200.15, VSEL.1
- removed net VBUS: C201.1, C202.1, C203.1, C301.1, C302.1, C303.1, C401.1, C402.1, C403.1, J1.P$4, J2.21, J2.22, J2.23, J2.24, J2.25, J2.26, JP3.1, LED1.A, R201.2, U$2.P$12, U$2.P$13, U$2.P$18, U$2.P$19, U$2.P$27, U$2.P$28, U$2.P$3, U$2.P$4, U200.12-13, U300.6, U400.6
- new net N$3: J302.6, LED301.P$6
- new net TPS62111-PG2: PG.1, U201.13
- new net TPS62111-SYNC2: R201.1, R202.2, SYNC.1, U201.5
- new net TPS62111_SW1: L201.1, U201.14, U201.15
- new net UART_RX1: J1.P$3, R104.1
- new net VBUSP: C201.1, C202.1, C301.1, C302.1, C303.1, C401.1, C402.1, C403.1, J1.P$4, J2.21, J2.22, J2.23, J2.24, J2.25, J2.26, JP3.1, LED1.A, R201.2, U$2.P$12, U$2.P$13, U$2.P$18, U$2.P$19, U$2.P$27, U$2.P$28, U$2.P$3, U$2.P$4, U201.2, U201.3, U201.4, U201.8, U300.6, U400.6, VBUSP.1
- net 3.3V: now also 3.3V.1, C203.1, L201.2, R105.2, R106.2, U201.10; no longer C205.1, C206.1, C207.1, R204.2, U200.7-8
- net ADDR_0: now also JP2.1; no longer JP2.2, JP2.4
- net ADDR_1: now also JP2.3; no longer JP2.6, JP2.8
- net DEBUG_1: now also LED4.A, U100.18; no longer LED3.A, U100.17
- net DEBUG_2: now also LED3.A, U100.17; no longer LED4.A, U100.18
- net GND: now also JP2.2, JP2.4, U201.1, U201.11, U201.12, U201.16, U201.6, U201.7, U201.9, U201.PAD; no longer C204.2, C205.2, C206.2, C207.2, JP2.3, JP2.7, R203.1, R205.1, R5.1, R6.1, U200.10, U200.4
- net I2C_SCL: now also R105.1
- net I2C_SDA: now also R106.1
- net N$1: now also J302.2, LED301.P$4; no longer LED5.C, R5.2
- net UART_RX: now also R104.2; no longer J1.P$3
Routing:
- net VBUSP: track 0.00 -> 24.1 mm, vias 0 -> 24
- net VBUS: track 20.9 -> 0.00 mm, vias 25 -> 0
- net SPI1_MISO: track 66.9 -> 81.9 mm
- net SPI1_CS: track 74.2 -> 89.2 mm
- net SPI1_SCK: track 70.6 -> 85.6 mm
- net UART_RX1: track 0.00 -> 11.7 mm
- net UART_TX: track 35.7 -> 46.7 mm
- net DEBUG_4: track 10.1 -> 0.00 mm
- net TPS-EN2: track 9.62 -> 0.00 mm
- net U: track 7.56 -> 16.9 mm, vias 1 -> 0
- net GND: track 71.2 -> 80.3 mm, vias 200 -> 220
- net I2C_SCL: track 63.0 -> 71.5 mm
- net DEBUG_3: track 7.87 -> 0.00 mm
- net 3.3V: track 42.6 -> 50.3 mm
- net I2C_SDA: track 65.3 -> 72.3 mm
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- added copper zone on layer 2, net 3.3V
- added copper zone on layer 15, net GND
- added copper zone on layer 16, net TPS62111_SW1
- added copper zone on layer 16, net VBUSP
- added copper zone on layer 2, net VBUSP
- removed copper zone on layer 15, net 3.3V
- removed copper zone on layer 2, net GND
- removed copper zone on layer 16, net TPS-L5
- removed copper zone on layer 16, net TPS-L6
- removed copper zone on layer 15, net VBUS
- removed copper zone on layer 16, net VBUS
Other:
- board size 66 x 88 mm -> 66 x 103 mm
- board text added: "3.3V"
- board text added: "VBUSP"
- board text removed: "DEBUG_3"
- board text removed: "DEBUG_4"
