File: eaglecad/controller_rev4.3_flat.sch (EAGLE design)
At the start: 134 parts, among them J2 J-SAMTEC-TFM-120-X1-XXX-D-RA, U100 STM32L452XX_QFPN48, U101 TCAN330, U200 TPS63070, U300 STSPIN230, U301 TSV991ILT, U302 AS5047P, U400 STSPIN250, U401 TSV991ILT, X101 ABM10-16MHz

Commit message: flat board ready for second round of inspection
Parts:
- removed C204: 100n, rcl_custom:C-EU0402-B-NOSILK
- removed C205: 10u, oresat-rcl:C-EU0603-B-NOSILK
- removed C206, C207: 22u, oresat-rcl:C-EU0805-B-NOSILK
- removed EN, FB2, VSEL: TEST-POINT-LARGE, oresat-misc:TEST-POINT-LARGE
- removed LED5, LED6: BLUE, led:LEDCHIPLED_0603
- removed R203: 10k, rcl_custom:R-US_0402-B-NOSILK
- removed R204: 470k, rcl_custom:R-US_0402-B-NOSILK
- removed R205: 150k, rcl_custom:R-US_0402-B-NOSILK
- removed R5, R6: 100, oresat-rcl:R-US_0402-B-NOSILK
- removed U200: TPS63070, ic-pwr-tps63070x:TPS63070X
- added 3.3V, SYNC, VBUSP: TEST-POINT-LARGE-SQUARE, oresat-misc:TEST-POINT-LARGE-SQUARE
- added R104: 10k, rcl_custom:R-US_0402-B-NOSILK
- added R105, R106: 4.7k, rcl_custom:R-US_0402-B-NOSILK
- added U201: TPS62111RSA, U-TI-TPS6211x-SPS-buck:TPS6211X
- C201: value 22u -> 10u; DIS (none) -> Digi-Key; DPN (none) -> 1276-6472-1-ND; MFR (none) -> Samsung; MPN (none) -> CL21B106KOQNNNG
- C202: value 22u -> 1u; device oresat-rcl:C-EU0805-B-NOSILK -> oresat-rcl:C-EU0603-C-NOSILK; DIS (none) -> Digi-Key; DPN (none) -> 311-1444-1-ND; MFR (none) -> Yageo; MPN (none) -> CC0603KRX5R7BB105
- C203: value 10u -> 22u; device oresat-rcl:C-EU0603-B-NOSILK -> oresat-rcl:C-EU0805-B-NOSILK; DPN 1276-1001-1-ND -> 490-9959-1-ND; MFR Samsung -> Murata; MPN CL05B104KO5NNNC -> GRM21BD71A226ME44L
- JP1: device pinhead:PINHD-1X4 -> pinhead:PINHD-1X2
- JP2: device pinhead:PINHD-2X4 -> pinhead:PINHD-2X2
- L201: value 1.5 uH -> 6.8u; device L-Coilcraft-XFL4020:L-COILCRAFT-XFL4020 -> L-ECS-MPI4040:L-ECS-MPI4040; DIS Mouser -> Digi-Key; DPN 994-XFL4020-152MEB -> XC2337CT-ND; MFR Coilcraft -> ECS; MPN XFL4020-152ME -> ECS-MPI4040R4-6R8-R
- PG: value TEST-POINT-LARGE -> TEST-POINT-LARGE-SQUARE; device oresat-misc:TEST-POINT-LARGE -> oresat-misc:TEST-POINT-LARGE-SQUARE
- R201: device rcl_custom:R-US_0402-B-NOSILK -> oresat-rcl:R-US_0603-C-NOSILK; DPN 1276-4275-1-ND -> RNCP0603FTD10K0CT-ND; MFR Samsung -> Stackpole; MPN RC1005F6653CS -> RNCP0603FTD10K0
- R202: device rcl_custom:R-US_0402-B-NOSILK -> oresat-rcl:R-US_0603-C-NOSILK
Connections:
- removed net CAN_SHDN: U101.SHDN
- removed net DEBUG_3: JP1.3, JP2.1, LED5.A
- removed net DEBUG_4: JP1.4, JP2.5, LED6.A
- removed net FB2: FB2.TP, U200.FB2
- removed net N$11: J302.2, LED301.BA
- removed net N$13: J302.6, LED301.RA
- removed net N$2 (its old number): LED6.C, R6.2
- removed net PG: PG.TP, U200.PG
- removed net TPS-EN2: EN.TP, R201.1, R202.2, U200.EN, U200.PS/SYNC
- removed net TPS-FB2: R204.1, R205.2, U200.FB
- removed net TPS-L5: L201.1, U200.L1
- removed net TPS-L6: L201.2, U200.L2
- removed net TPS-VAUX2: C204.1, U200.VAUX
- removed net TPS-VSEL2: R203.2, U200.VSEL, VSEL.TP
- removed net VBUS: C201.1, C202.1, C203.1, C301.1, C302.1, C303.1, C401.1, C402.1, C403.1, J1.VCC, J2.21, J2.22, J2.23, J2.24, J2.25, J2.26, JP3.1, LED1.A, R201.2, U$2.VCC, U200.VIN, U300.VS, U400.VS
- new net N$3: J302.6, LED301.BA
- new net TPS62111-PG2: PG.1, U201.PG
- new net TPS62111-SYNC2: R201.1, R202.2, SYNC.1, U201.SYNC
- new net TPS62111_SW1: L201.1, U201.SW
- new net UART_RX1: J1.RXI, R104.1
- new net VBUSP: C201.1, C202.1, C301.1, C302.1, C303.1, C401.1, C402.1, C403.1, J1.VCC, J2.21, J2.22, J2.23, J2.24, J2.25, J2.26, JP3.1, LED1.A, R201.2, U$2.VCC, U201.EN, U201.VIN, U300.VS, U400.VS, VBUSP.1
- net 3.3V: now also 3.3V.1, C203.1, L201.2, R105.2, R106.2, U201.FB; no longer C205.1, C206.1, C207.1, R204.2, U200.VOUT
- net ADDR_0: now also JP2.1; no longer JP2.2, JP2.4
- net ADDR_1: now also JP2.3; no longer JP2.6, JP2.8
- net DEBUG_1: now also LED4.A, U100.PB0; no longer LED3.A, U100.PA7
- net DEBUG_2: now also LED3.A, U100.PA7; no longer LED4.A, U100.PB0
- net GND: now also JP2.2, JP2.4, U201.GND, U201.LBI, U201.LBO; no longer C204.2, C205.2, C206.2, C207.2, JP2.3, JP2.7, R203.1, R205.1, R5.1, R6.1, U200.GND, U200.PGND
- net I2C_SCL: now also R105.1
- net I2C_SDA: now also R106.1
- net N$1: now also J302.2, LED301.RA; no longer LED5.C, R5.2
- net UART_RX: now also R104.2; no longer J1.RXI
Other:
- note added: "ECS-MPI4040R4-6R8-R"
- note added: "TO MEZZANINE"
- note removed: "0603"
- note removed: "TO ORESAT CARD CONNECTION"
- moved on the sheet: C107, C201, C202, C203, DEBUG_1, DEBUG_2, J1, L201, LED2, LED3, LED301, LED4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

Commit message: BOM
Parts:
- removed U$2: MEZZANINE_1, oresat-ACS_driver_board:MEZZANINE_1
- removed U100: STM32L452XX_QFPN48, oresat-ACS_driver_board:STM32L452XX_QFPN48
- added J3: MEZZANINE_PLUG, J-Molex-05xxxx030x-30pin-mezzanine-connector-M+F:MEZZANINE_PLUG
- added U$1: STM32L452CEU3, U-ST-STML453CEU3-uC:STM32L452CEU3
- J2: DESCRIPTION (none) -> 90 degree 40 pos conn header; DIST (none) -> Digi-Key; DIST_PN (none) -> SAM10145-ND; GENERIC (none) -> N; MFG (none) -> Samtec Inc.; MFG_PN (none) -> TFM-120-01-L-D-RA; P-NP (none) -> P
- JP2: DESCRIPTION (none) -> 2x2 .1 inch pin header; DIST (none) -> Digi-Key; DIST_PN (none) -> 952-1772-ND; GENERIC (none) -> Y; MFG (none) -> Harwin Inc.; MFG_PN (none) -> M20-9760246; P-NP (none) -> P
- U300: device oresat-ACS_driver_board:STSPIN230 -> U-ST-STSPIN2x0-motor-drivers:STSPIN230
- U301, U401: device oresat-ACS_driver_board:TSV991ILT -> U-ST-TSV991ILT-op-amp:TSV991ILT
- U302: device U-AMS-AS5047P-encoder:AS5047P -> U-AMS-AS5047P-ATSM-BLDC-encoder:AS5047P
- U400: device oresat-ACS_driver_board:STSPIN250 -> U-ST-STSPIN2x0-motor-drivers:STSPIN250
Connections:
- net 3.3V: now also U$1.VBAT, U$1.VDD, U$1.VDDA; no longer U100.VBAT, U100.VDD, U100.VDDA
- net ADDR_0: now also U$1.PB1; no longer U100.PB1
- net ADDR_1: now also U$1.PB2; no longer U100.PB2
- net BLDC_CURR_FDB: now also U$1.PA1; no longer U100.PA1
- net BLDC_EN: now also U$1.PA12; no longer U100.PA12
- net BLDC_FAULT: now also U$1.PA11; no longer U100.PA11
- net BLDC_INUH: now also U$1.PB13; no longer U100.PB13
- net BLDC_INUL: now also U$1.PA8; no longer U100.PA8
- net BLDC_INVH: now also U$1.PB14; no longer U100.PB14
- net BLDC_INVL: now also U$1.PA9; no longer U100.PA9
- net BLDC_INWH: now also U$1.PB15; no longer U100.PB15
- net BLDC_INWL: now also U$1.PA10; no longer U100.PA10
- net BLDC_STBY: now also U$1.PB12; no longer U100.PB12
- net BOOT: now also J3.BOOT, U$1.PH3-BOOT0; no longer U$2.BOOT, U100.PH3-BOOT0
- net CAN_H: now also J3.CAN_H; no longer U$2.CAN_H
- net CAN_L: now also J3.CAN_L; no longer U$2.CAN_L
- net CAN_RX: now also U$1.PB5; no longer U100.PB5
- net CAN_SILENT: now also U$1.PB4; no longer U100.PB4
- net CAN_TX: now also U$1.PB6; no longer U100.PB6
- net CLK1: now also U$1.PH0-OSC_IN; no longer U100.PH0-OSC_IN
- net CLK2: now also U$1.PH1-OSC_OUT; no longer U100.PH1-OSC_OUT
- net DEBUG_1: now also U$1.PB0; no longer U100.PB0
- net DEBUG_2: now also U$1.PA7; no longer U100.PA7
- net GND: now also J3.GND, U$1.VDDUSB, U$1.VSS, U$1.VSSA; no longer U$2.GND, U100.VDDUSB, U100.VSS, U100.VSSA
- net I2C_SCL: now also J3.I2C_SCL, U$1.PB10; no longer U$2.I2C_SCL, U100.PB10
- net I2C_SDA: now also J3.I2C_SDA, U$1.PB11; no longer U$2.I2C_SDA, U100.PB11
- net MAG_CURR_FDB: now also U$1.PA0; no longer U100.PA0
- net MAG_DIR: now also U$1.PB3; no longer U100.PB3
- net MAG_EN: now also U$1.PB9; no longer U100.PB9
- net MAG_FAULT: now also U$1.PB8; no longer U100.PB8
- net MAG_PWM: now also U$1.PA15; no longer U100.PA15
- net MAG_STBY: now also U$1.PB7; no longer U100.PB7
- net NRST: now also U$1.NRST; no longer U100.NRST
- net OUT1: now also J3.MAG_1; no longer U$2.MAG_1
- net OUT2: now also J3.MAG_2; no longer U$2.MAG_2
- net SPI1_CS: now also U$1.PA4; no longer U100.PA4
- net SPI1_MISO: now also U$1.PA6; no longer U100.PA6
- net SPI1_SCK: now also U$1.PA5; no longer U100.PA5
- net SWCLK: now also U$1.PA14; no longer U100.PA14
- net SWDIO: now also U$1.PA13; no longer U100.PA13
- net UART_RX: now also U$1.PA3; no longer U100.PA3
- net UART_TX: now also U$1.PA2; no longer U100.PA2
- net VBUSP: now also J3.VCC; no longer U$2.VCC
Other:
- note added: "4.3f"
- note added: "Note on Op Amp Circuit: First stack of resistors offsets the shunt voltage by 0.78V it also reduces measured voltage difference by 25% Op Amp feedback doubles the voltage from the positive input terminal Voltage offset from shunt is 1.56V Shunt Delta gain is 1.5"
- note added: "Note: R305 and R306 are 0805 resistors"
- note added: "Put into formulaic terms where i: Current from SenseVW/SenseU (mA) Shunt equation: S(i) mV=.34 (mV/mA) * i + 0.4 mV Output Equation: O(i) mV=.52 (mV/mA) * i + 1560 mV Gain and Offset: O(i) mV = 1.5 * S(i) mV + 1560 mV"
- note removed: "4.2"
