File: eaglecad/archived/controller_rev3.1-test.sch (EAGLE design)
At the start: 79 parts, among them CON502 CARD CONN, U100 STM32L452XX_QFPN48, U101 TCAN330, U200 TPS63070, U300 STSPIN230, U301 TSV991ILT, U302 AS5047P, U400 STSPIN250, U401 TSV991ILT, X101 ABM10-16MHz

Commit message: order update
Parts:
- removed C501: DEBUG_CON, oresat-ACS_driver_board:DEBUG_CON
- removed CON502: CARD CONN, oresat-ACS_driver_board:LOW-PROFILE_CONNECTOR(TAB)
- removed R304: 680, rcl_custom:R-US_0402-B-NOSILK
- removed R305, R306, R411, R412: 0.68, oresat-rcl:R-US_0805-B-NOSILK
- removed R307: 2.2k, rcl_custom:R-US_0402-B-NOSILK
- removed R404: 330, rcl_custom:R-US_0402-B-NOSILK
- removed TP2, TP3: TPTP06R, testpad:TPTP06R
- added 3.3V, EN, FB2, PG, VSEL: TPTP15SQ, testpad:TPTP15SQ
- added C106: 100n, rcl_custom:C-EU0402-B-NOSILK
- added J1: 1.27MM-SWD-CONNECTOR, J-CNC-3220-10-0100-00-ARM-SWD-port:1.27MM-SWD-CONNECTOR
- added JP1, JP102, JP302, JP401: (no value), pinhead:PINHD-1X2
- added JP103: (no value), SparkFun-Connectors:6_PIN_SERIAL_TARGETSILK
- added R206: 150k, rcl_custom:R-US_0402-B-NOSILK
- added R207: NP, rcl_custom:R-US_0402-B-NOSILK
- added R310, R311, R415, R416: 0.68, oresat-rcl:R-US_0805-B-NOSILK
- added R312, R313, R417, R418: 2.2k, rcl_custom:R-US_0402-B-NOSILK
- added R314, R419: 0, rcl_custom:R-US_0402-B-NOSILK
- added R315: 10k, rcl_custom:R-US_0402-B-NOSILK
- C103: value 10n -> 100n
- C104: value 10p -> 20p
- C105: value 100n -> 20p; DPN 1276-1001-1-ND -> 1276-6601-1-ND; MPN CL05B104KO5NNNC -> CL05C200JB51PNC
- C306: value 4.7u -> 680p; device oresat-rcl:C-EU0603-B-NOSILK -> rcl_custom:C-EU0402-B-NOSILK
- C307, C408: value 100n -> 680p
- C308: value 680p -> 100n
- C309, C410: value 680p -> 4.7u; device rcl_custom:C-EU0402-B-NOSILK -> oresat-rcl:C-EU0603-B-NOSILK
- C406: value 2.2n -> 22n
- C407: value 22n -> 2.2n
- C409: value 4.7u -> 100n; device oresat-rcl:C-EU0603-B-NOSILK -> rcl_custom:C-EU0402-B-NOSILK
- R201: value 10k -> 0; device rcl_custom:R-US_0402-B-NOSILK -> rcl_custom:R-US_0805-B-NOSILK; DPN 1276-4275-1-ND -> RHM0.0ARCT-ND; MFR Samsung -> Rohm; MPN RC1005F6653CS -> MCR10EZPJ000
- R202: value NP -> 10k
- R203: value 10k -> NP
- R204: value 470k -> 10k
- R205: value 150k -> 470k
- R303: value 2.2k -> 0; device rcl_custom:R-US_0402-B-NOSILK -> oresat-rcl:R-US_0805-B-NOSILK; DIS Digi-Key -> (none); DPN 1276-4275-1-ND -> (none); MFR Samsung -> (none); MPN RC1005F6653CS -> (none)
- R309: value 10k -> 680
- R403: value 330 -> 0; device rcl_custom:R-US_0402-B-NOSILK -> oresat-rcl:R-US_0805-B-NOSILK; DIS Digi-Key -> (none); DPN 1276-4275-1-ND -> (none); MFR Samsung -> (none); MPN RC1005F6653CS -> (none)
- R405: value 100k -> 330
- R406: value 18k -> 330
- R409: value 2.2k -> 100k
- R410: value 680 -> 18k
- R414: value 2.2k -> 680
- U100: value STM32L452XX_QFPN48 -> STM32F042K6; device oresat-ACS_driver_board:STM32L452XX_QFPN48 -> STM32F042K:STM32F042K6; DIS (none) -> Digi-Key; DPN (none) -> STM32F042K6T7-ND; MFR (none) -> STMicroelectronics; MPN (none) -> STM32F042K6T7
- U200: DIS Digi-Key -> (none); DPN 296-44874-1-ND -> (none); MFR TI -> (none); MPN TPS63070 -> (none)
- U300: device oresat-ACS_driver_board:STSPIN230 -> U-ST-STSPIN230-BLDC-controller:STSPIN230
- U301, U401: device oresat-ACS_driver_board:TSV991ILT -> TSV991ILT:TSV991ILT
- U400: device oresat-ACS_driver_board:STSPIN250 -> U-ST-STSPIN250-Brushed-DC-controller:STSPIN250
- X101: value ABM10-16MHz -> 16MHZ-2.5x2mm
Connections:
- net SPI1_SCK renamed PA5/SPI1_SCK
- net TPS-L5 renamed TPS-L1
- net TPS-L6 renamed TPS-L2
- net TPS-VAUX2 renamed TPS-VAUX
- removed net BLDC_CURR_FDB: C309.1, R307.2, U100.PA1, U301.OUT
- removed net BLDC_EN: R302.2, U100.PA12
- removed net BLDC_FAULT: C305.1, R302.1, U100.PA11, U300.EN/FAULT
- removed net BLDC_INUH: U100.PB13, U300.INUH
- removed net BLDC_INUL: U100.PA8, U300.INUL
- removed net BLDC_INVH: U100.PB14, U300.INVH
- removed net BLDC_INVL: U100.PA9, U300.INVL
- removed net BLDC_INWH: U100.PB15, U300.INWH
- removed net BLDC_INWL: U100.PA10, U300.INWL
- removed net BLDC_STBY: C304.1, R301.2, TP2.TP, U100.PB12, U300.STBY/RESET
- removed net B_IN+: C308.1, R303.1, R304.2, U301.IN+
- removed net B_IN-: C309.2, R307.1, R308.2, U301.IN-
- removed net CAN_SILENT: U100.PB4, U101.S
- removed net CLK1: C104.1, U100.PH0-OSC_IN, X101.2
- removed net CLK2: C104.2, U100.PH1-OSC_OUT, X101.1
- removed net DEBUG_1: C501.3, U100.PB2
- removed net DEBUG_2: C501.4, U100.PB1
- removed net MAG_CURR_FDB: C411.1, R413.2, U100.PA0, U401.OUT
- removed net MAG_DIR: R403.2, U100.PB3
- removed net MAG_EN: R402.2, U100.PB9
- removed net MAG_FAULT: C405.1, R402.1, U100.PB8, U400.EN/FAULT
- removed net MAG_PWM: R404.2, U100.PA15
- removed net MAG_STBY: C404.1, R401.2, TP3.TP, U100.PB7, U400.STBY/RESET
- removed net M_IN+: C410.1, R409.1, R410.2, U401.IN+
- removed net M_IN-: C411.2, R413.1, R414.2, U401.IN-
- removed net M_PH: R403.1, U400.PH
- removed net M_PWM: R404.1, U400.PWM
- removed net NRST: C501.7, U100.NRST
- removed net SPI1_CS: U100.PA4, U302.CSN
- removed net SPI1_MISO: U100.PA6, U302.MISO
- removed net TOFF1: C407.1, R407.2
- removed net TPS-EN2: R201.1, R202.2, U200.EN, U200.PS/SYNC
- removed net TPS-FB2: R204.1, R205.2, U200.FB
- removed net TPS-VSEL2: R203.2, U200.VSEL
- removed net UART_RX: C501.5, U100.PA3
- removed net UART_TX: C501.6, U100.PA2
- removed net VBUS: C201.1, C202.1, C203.1, C301.1, C302.1, C303.1, C401.1, C402.1, C403.1, C501.1, CON502.1, R201.2, U200.VIN, U300.VS, U400.VS
- new net BLDC-I-IN+: C306.1, R308.1, R309.2, U301.IN+
- new net BLDC-I-IN-: C307.1, R312.1, R313.2, U301.IN-
- new net BLDC-I-OUT: C307.2, R313.1, R314.2, U301.OUT
- new net CRYSTALIN: C105.1, U100.PF0-OSC_IN, X101.1
- new net CRYSTALOUT: C104.1, U100.PF1-OSC_OUT, X101.2
- new net MAG-I-IN+: C408.1, R413.1, R414.2, U401.IN+
- new net MAG-I-IN-: C411.1, R417.1, R418.2, U401.IN-
- new net MAG-I-OUT: C411.2, R418.1, R419.2, U401.OUT
- new net N$2: C406.2, R407.2
- new net N$3: R406.1, U400.PWM
- new net N$5: R405.1, U400.PH
- new net N$7: C301.1, C302.1, C303.1, R303.1, U300.VS
- new net N$8: C401.1, C402.1, C403.1, R403.1, U400.VS
- new net NRESET: J1.!RESET, U100.NRST
- new net PA0/CURR_FDB_MAG: R419.1, U100.PA0
- new net PA1/CURR_FDB_BLDC: R314.1, U100.PA1
- new net PA10/INWH: U100.PA10, U300.INWH
- new net PA15/CAN_SILENT: U100.PA15, U101.S
- new net PA2/USART2_TX: JP103.TXO, U100.PA2
- new net PA3/USART2_RX: JP103.RXI, U100.PA3
- new net PA4/FAULT_BLDC: C305.2, R302.1, U100.PA4, U300.EN/FAULT
- new net PA6/SPI1_NSS: U100.PA6, U302.CSN
- new net PA7/INUL: U100.PA7, U300.INUL
- new net PA8/INUH/PWM_MAG: R406.2, U100.PA8, U300.INUH
- new net PA9/INVH/DIR_MAG: R405.2, U100.PA9, U300.INVH
- new net PB0/INVL: U100.PB0, U300.INVL
- new net PB1/INWL: U100.PB1, U300.INWL
- new net PB3/EN_MAG: R402.2, U100.PB3
- new net PB4/SPI1_MISO: U100.PB4, U302.MISO
- new net PB5: U100.PB5
- new net PB6/EN_BLDC: R302.2, U100.PB6
- new net PB7/FAULT_MAG: C405.2, R402.1, U100.PB7, U400.EN/FAULT
- new net QUAD_A: JP302.1, U302.A
- new net QUAD_B: JP302.2, U302.B
- new net STBY/RESET_BLDC: C304.2, R301.1, U300.STBY/RESET
- new net STBY/RESET_MAG: C404.2, R401.1, U400.STBY/RESET
- new net TPS-EN: EN.TP, R202.1, R203.2, U200.EN, U200.PS/SYNC
- new net TPS-FB: R205.1, R206.2, U200.FB
- new net TPS-PG: PG.TP, R207.1, U200.PG
- new net TPS-VIN: C201.1, C202.1, C203.1, R201.1, R202.2, U200.VIN
- new net TSP-FB2: FB2.TP, U200.FB2
- new net TSP-VSEL: R204.2, U200.VSEL, VSEL.TP
- new net V_BATT: JP1.1, JP103.VCC, R201.2, R303.2, R403.2
- net 250_REF: now also C407.2, R409.2, R410.1; no longer C406.1, R405.2, R406.1
- net 3.3V: now also 3.3V.TP, C101.2, C102.2, C103.2, C106.2, C308.2, C309.1, C310.2, C410.1, J1.VTREF, R205.2, R207.2, R301.2, R308.2, R315.1, R401.2, R409.1, R413.2, U100.VDDIO2; no longer C101.1, C102.1, C103.1, C105.1, C306.1, C307.1, C310.1, C408.1, C501.2, R204.2, R301.1, R303.2, R309.1, R401.1, R405.1, R409.2, U100.VBAT
- net AS5047_MOSI: now also R315.2; no longer R309.2
- net BOOT: now also U100.PB8-BOOT0; no longer U100.PH3-BOOT0
- net CAN_H: now also JP102.1; no longer CON502.3
- net CAN_L: now also JP102.2; no longer CON502.2
- net CAN_RX: now also U100.PA11; no longer U100.PB5
- net CAN_TX: now also U100.PA12; no longer U100.PB6
- net GND: now also C101.1, C102.1, C103.1, C104.2, C106.1, C304.1, C305.1, C308.1, C309.2, C310.1, C404.1, C405.1, C406.1, C407.1, J1.GND, J1.GND@2, JP1.2, JP103.GND, R204.1, R206.1, R310.1, R311.1, R312.2, R410.2, R415.2, R416.2, R417.2; no longer C101.2, C102.2, C103.2, C304.2, C305.2, C307.2, C308.2, C310.2, C404.2, C405.2, C406.2, C407.2, C501.10, CON502.6, R202.1, R205.1, R305.1, R306.1, R308.1, R406.2, R411.2, R412.2, R414.1, U100.VDDUSB, U100.VSSA
- net OUT1: now also JP401.1; no longer CON502.5
- net OUT2: now also JP401.2; no longer CON502.4
- net SENSE_BLDC: now also R309.1, R310.2, R311.2; no longer R304.1, R305.2, R306.2
- net SENSE_MAG: now also R414.1, R415.1, R416.1; no longer R410.1, R411.1, R412.1
- net SWCLK: now also J1.SWDCLK/TCK, U100.PA14-SWCLK; no longer C501.9, U100.PA14
- net SWDIO: now also J1.SWDIO/TMS, U100.PA13-SWDIO; no longer C501.8, U100.PA13
Other:
- note added: "3"
- note added: "All caps are ceramic 10% X5R >= 16V Vwv unless marked"
- note added: "All resistors 0402 +/- 1% unless marked"
- note added: "CAN_SHDN and CAN_LSTN pins have internal pull-down resistors. If CAN_SHDN is pulled high it shuts the IC off. If CAN_LSTN is pulled high it puts the IC intro receive-only mode. Leave CAN_SHDN disconnected."
- note added: "Change to 3 pin for final rev"
- note added: "Current feedback to STM32."
- note added: "NP FOR FLIGHT"
- note added: "NRST pull-up built in"
- note added: "Place on breakoff"
- note added: "Quadrature output leads for motor spec test case"
- note added: "STM32 Current Feedback"
- note added: "TBD: CONNECTOR TO ORESAT ACS CARD"
- note added: "TO MAGNETORQUER"
- note removed: "4.1"
- note removed: "ASC BOARD CONNECTORS"
- note removed: "CON501"
- note removed: "CONNECTION TO ACS DRIVER PROG. ADDAPTER"
- note removed: "CONNECTION TO STANDARD ORESAT CARD"
- note removed: "DEBUG CONN"
- note removed: "PROGRAM ADDAPTER"
- note removed: "TO ORESAT CARD CONNECTION"
- moved on the sheet: BOOT, C101, C102, C103, C104, C105, C201, C202, C203, C204, C205, C206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
