File: rev-6/rev6.0_flat_powerstage/LEDs.kicad_sch (KiCad schematic)
At the start: 34 parts

Commit message: Rev 6 pre design review
Parts:
- removed C100, C101, C102, C88, C89, C90, C91, C92, C93, C94, C95, C96, C97, C98, C99: 100n, Capacitor_SMD:C_0603_1608Metric, symbol Device:C_Small
- removed C86, C87: 22u, Capacitor_SMD:C_0805_2012Metric, symbol Device:C_Small
- removed D10, D11, D12, D13, D14, D15, D16, D17, D18, D19, D20, D21, D7, D8, D9: APA102-2020, LED_SMD:LED-APA102-2020, symbol LED:APA102-2020
- removed R53, R54: 220, Resistor_SMD:R_0603_1608Metric, symbol Device:R_Small_US
Other:
- note removed: "Essential Motor Underglow LEDs"
