File: oresat-rw-board-rev7/control-stage/control-stage.kicad_sch (KiCad schematic)
At the start: 68 parts, among them J1 MEZZ, J2 10132797-021100LF, J3 10132797-021100LF, J4 10132797-021100LF, J5 Hirose_FH12-10S-0.5SH, Q1 TPN4R712MD,L1Q, U1 ADP7156ACPZ, U2 TLV62569DRL, U3 STM32G474RBTx, U5 TCAN330, Y1 Crystal_GND24

Commit message: Move rev-7 to oresat-acs-board-rev7
Parts:
- removed J5: Hirose_FH12-10S-0.5SH, Connector_FFC-FPC:Hirose_FH12-10S-0.5SH_1x10-1MP_P0.50mm_Horizontal, symbol Connector_Generic_MountingPin:Conn_01x10_MountingPin
- removed R19: THJP0603ABT1, Resistor_SMD:R_0603_1608Metric, symbol Device:R_Small_US
- added C21, C30, C31, C33: 22u, Capacitor_SMD:C_0603_1608Metric, symbol Device:C_Small
- added C60, C61: 1u, Capacitor_SMD:C_0402_1005Metric, symbol Device:C_Small
- added J6: J-TE-Debug-2-1734592-0, rev-7-footprints:J-TE_2-1734592-0, symbol rev-7-symbols:J-TE-Debug-2-1734592-0
- added J7: PROBE, Connector_PinHeader_1.27mm:PinHeader_2x05_P1.27mm_Horizontal, symbol Connector_Generic:Conn_02x05_Odd_Even
- added TP1, TP2, TP3, TP4, TP5, TP6: TestPoint_Alt, TestPoint:TestPoint_THTPad_1.0x1.0mm_Drill0.5mm, symbol Connector:TestPoint_Alt
- C11, C9: value 20p -> 18p
- H1: footprint rev-7-footprints:top-board-def -> rev-7-footprints:top-board-def-rev7.1
- R1: value 100k -> 100k/1%
- R11, R12, R13, R14, R15, R16, R17, R18: value THJP0603ABT1 -> THJP1206ABT1; footprint Resistor_SMD:R_0603_1608Metric -> Resistor_SMD:R_1206_3216Metric
- U3: value STM32G474RBTx -> STM32G474RET3
- Y1: P/N ECS-160-12-37BQ-CTN-TR -> LFXTAL071255REEL
Connections:
- net +3V3: now also Q1.1 (S), R1.2, C21.2, C30.2, C31.2, C33.2, J6.11 (VTARGET), TP6.1
- net +5V: now also J2.10 (Pin_10), J2.11 (Pin_11), J2.12 (Pin_12), J2.9 (Pin_9), J6.1 (VBUSP), J6.2 (VBUSP); no longer Q1.1 (S), R1.1
- net BOOT0: now also J6.17 (DEBUG-0)
- net CAN_RX: now also U3.34 (PB12); no longer U3.58 (PB5)
- net CAN_TX: now also U3.35 (PB13); no longer U3.59 (PB6)
- net DEBUG_RX: now also U3.60 (PB7), J6.12 (CARD-RX), J7.4 (Pin_4); no longer U3.53 (PC11)
- net DEBUG_SWCLK: now also J6.15 (SWCLK), TP4.1
- net DEBUG_SWDIO: now also J6.14 (SWDIO), TP3.1
- net DEBUG_SWO: now also J6.16 (SWO), TP1.1
- net DEBUG_TX: now also U3.59 (PB6), J6.13 (CARD-TX), J7.2 (Pin_2); no longer U3.52 (PC10)
- net GND: now also C21.1, C30.1, C31.1, C33.1, C60.1, C61.1, J6.3 (GND), J6.6 (GND), J6.9 (GND), J6.PAD1 (PAD), J6.PAD2 (PAD), J7.9 (Pin_9), TP2.1; no longer J3.10 (Pin_10), J3.11 (Pin_11)
- net NRST: now also J6.10 (NRST), TP5.1
- net SPI_MISO: now also U3.53 (PC11); no longer U3.20 (PA6)
- net SPI_MOSI: now also U3.54 (PC12); no longer U3.21 (PA7)
- net SPI_SCK: now also U3.52 (PC10); no longer U3.19 (PA5)
- net SPI_nCS: now also U3.51 (PA15); no longer U3.18 (PA4)
- net THERM_A: now also C60.2
- net THERM_B: now also C61.2
- net UART_RX: now also U3.17 (PA3), J6.19 (DEBUG-2); no longer U3.23 (PC5)
- net UART_TX: now also U3.14 (PA2), J6.18 (DEBUG-1); no longer U3.22 (PC4)
- net 5V_FILT: now reaches C10.1, C22.1, C7.1, C8.1, FB1.2, U1.10 (VIN), U1.5 (EN), U1.9 (VIN)
- net DEBUG3: now reaches U3.55 (PD2)
- net DEBUG3: now also J7.7 (Pin_7)
- net DEBUG2: now reaches U3.57 (PB4)
- net DEBUG2: now also J7.5 (Pin_5)
- net DEBUG0: now reaches U3.62 (PB9)
- net DEBUG0: now also J7.1 (Pin_1)
- removed net +5V_SW: J2.10 (Pin_10), J2.11 (Pin_11), J2.12 (Pin_12), J2.9 (Pin_9), Q1.3 (D)
- removed net SW_5V: Q1.2 (G), R1.2, U3.60 (PB7)
- new net +3V3_SW: J3.10 (Pin_10), J3.11 (Pin_11), Q1.3 (D)
- new net DEBUG1: J7.3 (Pin_3), U3.58 (PB5)
- new net SCOPE0: J7.10 (Pin_10), U3.18 (PA4)
- new net SCOPE1: J7.8 (Pin_8), U3.19 (PA5)
- new net SCOPE2: J7.6 (Pin_6), U3.20 (PA6)
- new net SW_3V3: Q1.2 (G), R1.1, U3.22 (PC4)
- no-connect marks 20 -> 18
Other:
- note added: "Encoder power switch"
- note added: "Fake trace connector"
- note added: "It's easier to power cycle the encoder than it is to clear errors between program resets"
- note added: "Mezz plug to ADCS card"
- note added: "Notes: - Weird sense line pins is b/c using ADC fast channels - HRTIM B/E/F has best pinout - SCOPE0-3 and DEBUG0-3 are DAC and GPIO respectively - GND and GNDA are the same, but returns are managed on different layers"
- note added: "OreSat FFC Debug Connector"
- note added: "Star at B2B connector"
- note added: "Test points for high speed SWO"
- note added: "no term needed"
- note added: "pinout verified ok"
- note added: "super precision, super expensive"
- note added: "verify ok"
- note added: "wheeeeeee"
- note removed: "5V tolerant"
- note removed: "BOM"
- note removed: "Inverter board +5V switch"
- note removed: "Star at mezz"
- note removed: "Swap with MEMS?"
- note removed: "Thermal jumper"
- note removed: "check if 5V tolerant"
- moved on the sheet: C10, C15, C16, C17, C22, C25, C26, C28, C38, C4, C7, C8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
