File: oresat-rw-board-rev7/power-stage/power-stage.kicad_sch (KiCad schematic)
At the start: 142 parts, among them J1 10132797-021100LF, J2 10132797-021100LF, J3 10132797-021100LF, J4 Motor, Q1 LMG5200, Q2 LMG5200, Q3 LMG5200, U1 AS5047P, U2 INA240A1PW, U3 INA240A1PW, U4 INA240A1PW

Commit message: Move rev-7 to oresat-acs-board-rev7
Parts:
- removed C60, C61: 1u, Capacitor_SMD:C_0402_1005Metric, symbol Device:C_Small
- removed R34, R39, R41, R49, R52, R53, R54, R56, R58, R65, R66: THJP0603ABT1, Resistor_SMD:R_0603_1608Metric, symbol Device:R_Small_US
- removed U1: AS5047P, Package_SO:TSSOP-14_4.4x5mm_P0.65mm, symbol Sensor_Magnetic:AS5047D
- removed U2, U3, U4: INA240A1PW, Package_SO:TSSOP-8_4.4x3mm_P0.65mm, symbol Amplifier_Current:INA240A1PW
- added C44, C45, C46, C57, C58, C59: 4.7u, Capacitor_SMD:C_0805_2012Metric, symbol Device:C_Small
- added J10, J5, J6, J7, J8, J9: PAD, Connector_Wire:SolderWirePad_1x01_SMD_1x2mm, symbol Connector_Generic:Conn_01x01
- added R68, R69: THJP0603ABT1, Resistor_SMD:R_0603_1608Metric, symbol Device:R_Small_US
- added U2, U3, U4: INA241, Package_TO_SOT_SMD:SOT-23-8, symbol rev-7-symbols:INA241
- added U5: MA732, Package_DFN_QFN:QFN-16-1EP_3x3mm_P0.5mm_EP1.75x1.75mm, symbol Sensor_Magnetic:MA730
- C1: value 1u -> 47u; footprint Capacitor_SMD:C_0402_1005Metric -> Capacitor_SMD:C_1210_3225Metric
- C2: value 100n -> 4.7u; footprint Capacitor_SMD:C_0402_1005Metric -> Capacitor_SMD:C_0805_2012Metric; MPN (none) -> GCM21BC7YA475KE36L
- C35, C36: value 47u -> 4.7u; footprint Capacitor_SMD:C_1210_3225Metric -> Capacitor_SMD:C_0805_2012Metric; MPN (none) -> GCM21BC7YA475KE36L; P/N GRM32EC81C476ME15L -> (none)
- C37, C56: value 22u -> 4.7u; MPN (none) -> GCM21BC7YA475KE36L; P/N GRT21BR61E226ME13L -> (none)
- H1: footprint rev-7-footprints:board-def -> rev-7-footprints:board-def-rev7.3
- R13, R14, R15: value 9m -> 10m; footprint rev-7-footprints:KRL3216 -> Resistor_SMD:R_Shunt_Vishay_WSK2512_6332Metric_T1.19mm; P/N KRL3216T4A-M-R009-F-T1 -> WSK2512R0100DEA
- R35, R44, R47, R61: value THJP0603ABT1 -> THJP1206ABT1; footprint Resistor_SMD:R_0603_1608Metric -> Resistor_SMD:R_1206_3216Metric
Connections:
- net +3V3A: now also U2.6 (V+), U3.6 (V+), U4.6 (V+)
- net +5V: no longer C3.1, C4.1
- net CHASSIS: now also R44.1, R47.1, R68.1, R69.1; no longer R44.2, R60.2
- net GND: now also R44.2, J10.1 (Pin_1), R68.2, R69.2, U2.2 (GND), U2.3 (REF2), U2.4 (GND), U3.2 (GND), U3.3 (REF2), U3.4 (GND), U4.2 (GND), U4.3 (REF2), U4.4 (GND), U5.10 (TEST), U5.15 (SSCK), U5.17 (PAD), U5.8 (GND); no longer C2.2, J2.10 (Pin_10), J2.11 (Pin_11)
- net IA_SNS: now also U4.5
- net IB_SNS: now also U3.5
- net IC_SNS: now also U2.5
- net PGND: now also C2.2, R60.2, C44.2, C45.2, C46.2, C57.2, C58.2, C59.2
- net PHA_RAW: no longer R44.1
- net PHB: no longer R47.1
- net SPI_MISO: now also J8.1 (Pin_1), U5.7 (MISO)
- net SPI_MOSI: now also J5.1 (Pin_1), U5.4 (MOSI)
- net SPI_SCK: now also J6.1 (Pin_1), U5.12 (SCLK)
- net SPI_nCS: now also J7.1 (Pin_1), U5.5 (~{CS})
- net VBUS: now also C2.1, C44.1, C45.1, C46.1, C57.1, C58.1, C59.1
- net PHA_FLT_H: now reaches C15.1, Q2.4 (HI), R6.2
- net +3V3_SW: now reaches C1.1
- net +3V3_SW: now also C3.1, C4.1, J2.10 (Pin_10), J2.11 (Pin_11), J9.1 (Pin_1), U5.13 (VDD); no longer C2.1
- net PHA_FLT_L: now reaches C12.1, Q2.5 (LI), R7.2
- net INAC_P: now reaches C32.2, R16.2
- net INAC_P: now also U2.8 (+)
- net INAC_N: now reaches C32.1, R10.1
- net INAC_N: now also U2.1 (-)
- net INAC_REF: now reaches C41.1, R19.1
- net INAC_REF: now also U2.7 (REF1)
- net PHA_VCC: now reaches C18.1, C9.1, Q2.6 (VCC), R2.2
- net INAB_REF: now reaches C43.1, R21.1
- net INAB_REF: now also U3.7 (REF1)
- net INAB_N: now reaches C34.1, R12.1
- net INAB_N: now also U3.1 (-)
- net SNSB_N: now reaches R12.2, R14.2
- net PHC_FLT_L: now reaches C11.1, Q1.5 (LI), R5.2
- net PHB_VCC: now reaches C10.1, C19.1, Q3.6 (VCC), R3.2
- net PHC_VCC: now reaches C17.1, C8.1, Q1.6 (VCC), R1.2
- net INAB_P: now reaches C34.2, R18.2
- net INAB_P: now also U3.8 (+)
- net SNSC_N: now reaches R10.2, R15.2
- net PHB_FLT_H: now reaches C16.1, Q3.4 (HI), R8.2
- net INAA_N: now reaches C33.1, R11.1
- net INAA_N: now also U4.1 (-)
- net INAA_P: now reaches C33.2, R17.2
- net INAA_P: now also U4.8 (+)
- net PHB_FLT_L: now reaches C13.1, Q3.5 (LI), R9.2
- net PHC_FLT_H: now reaches C14.1, Q1.4 (HI), R4.2
- net INAA_REF: now reaches C42.1, R20.1
- net INAA_REF: now also U4.7 (REF1)
- net SNSC_P: now reaches R15.3, R16.1
- net SNSB_P: now reaches R14.3, R18.1
- net SNSA_N: now reaches R11.2, R13.2
- net SNSA_P: now reaches R13.3, R17.1
- no-connect marks 4 -> 7
Other:
- note added: "100k @ 25C"
- note added: "18uF ea"
- note added: "6uF local"
- note added: "Bottom-side decouple/bulk"
- note added: "Switched 3v3 power for encoder from control board"
- note added: "~100uF total mlcc"
- note added: "~2uF ea"
- note added: "~3uF ea"
- moved on the sheet: R35, R40, R43, R46, R51, R55, R57, R59, R60, R61, R62, R63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
