File: oresat-rw-card/oresat-mag-card-sch-magnetorquers.kicad_sch (KiCad schematic)
At the start: 88 parts, among them Q16 DMP2240UDM, Q17 PMV45EN, Q18 DMP3050LVT-7, Q19 DMP3050LVT-7, Q20 PMV45EN, U19 MAX7310, U20 MIC842LYC5, U21 MIC842LYC5, U22 TS5A21366DCUR, U23 MAX4211FETE, U24 TPS62111RSA

Commit message: Pushed because Andrew told me to
Parts:
- removed C39: 10u, oresat-passives:0805-B-NOSILK, symbol Device:C_Small
- removed C40: 1u, oresat-passives:c_0603-SMALL, symbol Device:C_Small
- removed C43: 22u, oresat-passives:0805-B-NOSILK, symbol Device:C_Small
- removed D11: GREEN, oresat-acs-card:LED-0603, symbol Device:LED
- removed L4: 6.8u, oresat-acs-card:ECS-MPI4040, symbol Device:L
- removed R164, R175: 10k, Resistor_SMD:R_0603_1608Metric, symbol Device:R_Small_US
- removed R165: DNP, Resistor_SMD:R_0603_1608Metric, symbol Device:R_Small_US
- removed TP66, TP70, TP71: Test-Point, oresat-misc:TestPoint-0.75mm-th, symbol oresat-misc:Test-Point-0.75mm-th
- removed U24: TPS62111RSA, Package_DFN_QFN:Texas_RSA_VQFN-16-1EP_4x4mm_P0.65mm_EP2.7x2.7mm, symbol oresat-ics:TPS6211X
Other:
- note removed: "0805"
- note removed: "3.3V Card Switching Supply"
- company: Edward Tsoi -> Portland State Aerospace Society
- title: OreSat ADCS Card -> OreSat Reaction Wheel Card
