File: oresat-rw-card/oresat-mag-card-sch-power.kicad_sch (KiCad schematic)
At the start: 88 parts, among them Q1 DMP2240UDM, Q2 PMV45EN, Q3 DMP3050LVT-7, Q4 DMP3050LVT-7, Q9 PMV45EN, U1 MAX7310, U18 MAX4211FETE, U2 MIC842LYC5, U3 MIC842LYC5, U5 TS5A21366DCUR, U6 TPS62111RSA

Commit message: Pushed because Andrew told me to
Parts:
- removed C10: 22u, oresat-passives:0805-B-NOSILK, symbol Device:C_Small
- removed C8: 10u, oresat-passives:0805-B-NOSILK, symbol Device:C_Small
- removed C9: 1u, oresat-passives:c_0603-SMALL, symbol Device:C_Small
- removed D3: GREEN, oresat-acs-card:LED-0603, symbol Device:LED
- removed L1: 6.8u, oresat-acs-card:ECS-MPI4040, symbol Device:L
- removed R39, R42: 10k, Resistor_SMD:R_0603_1608Metric, symbol Device:R_Small_US
- removed R40: DNP, Resistor_SMD:R_0603_1608Metric, symbol Device:R_Small_US
- removed TP16, TP18, TP19: Test-Point, oresat-misc:TestPoint-0.75mm-th, symbol oresat-misc:Test-Point-0.75mm-th
- removed U6: TPS62111RSA, Package_DFN_QFN:Texas_RSA_VQFN-16-1EP_4x4mm_P0.65mm_EP2.7x2.7mm, symbol oresat-ics:TPS6211X
Other:
- note removed: "0805"
- note removed: "3.3V Card Switching Supply"
- company: Edward Tsoi -> Portland State Aerospace Society
- title: OreSat ADCS Card -> OreSat Reaction Wheel Card

Commit message: Start moving towards hiearchical RW card, just did Q1
Connections:
- net BOOT_CONFIG renamed BOOTCFG-Q1
- net SW_COM1 renamed RW-UART-TX-Q1
- net SW_COM2 renamed RW-UART-RX-Q1
- net VBUSP renamed VBUSP-Q1
Other:
- note removed: "To MCXN digitally configued boot pin"
- moved on the sheet: R23
Changed lines of the file:
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@@
 		)
 	)
-	(text "To MCXN digitally configued boot pin\n"
-		(exclude_from_sim no)
-		(at 202.438 271.018 0)
-		(effects
-			(font
-				(size 1.778 1.5113)
-			)
-			(justify left bottom)
-		)
-	)
 	(text "Address selection for Card\n(See MAX7310 datasheet)"
 		(exclude_from_sim no)
@@
 	(wire
 		(pts
-			(xy 194.31 215.9) (xy 215.9 215.9)
+			(xy 194.31 215.9) (xy 220.98 215.9)
 		)
 		(stroke
@@
 	(wire
 		(pts
-			(xy 200.66 210.82) (xy 200.66 273.05)
-		)
-		(stroke
-			(width 0)
-			(type default)
-		)
-	)
-	(wire
-		(pts
 			(xy 436.88 119.38) (xy 436.88 121.92)
 		)
@@
 	(wire
 		(pts
-			(xy 215.9 226.06) (xy 220.98 226.06)
-		)
-		(stroke
-			(width 0)
-			(type default)
-		)
-	)
-	(wire
-		(pts
 			(xy 128.27 165.1) (xy 128.27 168.91)
 		)
@@
 	(wire
 		(pts
-			(xy 471.17 114.3) (xy 471.17 115.57)
+			(xy 471.17 110.49) (xy 471.17 115.57)
 		)
 		(stroke
@@
 	(wire
 		(pts
-			(xy 215.9 215.9) (xy 215.9 226.06)
+			(xy 220.98 215.9) (xy 220.98 226.06)
 		)
 		(stroke
@@
 	(wire
 		(pts
-			(xy 220.98 238.76) (xy 220.98 243.84)
+			(xy 220.98 233.68) (xy 220.98 236.22)
 		)
 		(stroke
@@
 	(wire
 		(pts
-			(xy 181.61 210.82) (xy 200.66 210.82)
+			(xy 181.61 210.82) (xy 199.39 210.82)
 		)
 		(stroke
@@
 	(wire
 		(pts
-			(xy 220.98 226.06) (xy 220.98 233.68)
+			(xy 220.98 226.06) (xy 220.98 228.6)
 		)
 		(stroke
@@
 	(wire
 		(pts
-			(xy 200.66 273.05) (xy 212.09 273.05)
-		)
-		(stroke
-			(width 0)
-			(type default)
-		)
-	)
-	(wire
-		(pts
 			(xy 361.95 170.18) (xy 361.95 175.26)
 		)
@@
 		)
 	)
-	(hierarchical_label "SW_COM1"
-		(shape input)
+	(hierarchical_label "RW-UART-TX-Q1"
+		(shape output)
 		(at 252.73 233.68 180)
 		(effects
@@
 		)
 	)
-	(hierarchical_label "SW_COM2"
+	(hierarchical_label "VBUSP-Q1"
 		(shape output)
+		(at 471.17 110.49 90)
+		(effects
+			(font
+				(size 1.27 1.27)
+			)
+			(justify left)
+		)
+	)
+	(hierarchical_label "RW-UART-RX-Q1"
+		(shape input)
 		(at 252.73 236.22 180)
 		(effects
@@
 		)
 	)
-	(hierarchical_label "BOOT_CONFIG"
+	(hierarchical_label "BOOTCFG-Q1"
 		(shape output)
-		(at 212.09 273.05 0)
+		(at 199.39 210.82 0)
 		(effects
 			(font
@@
 		(lib_name "GND_1")
 		(lib_id "power:GND")
-		(at 220.98 243.84 0)
+		(at 220.98 236.22 0)
 		(unit 1)
 		(exclude_from_sim no)
@@
 		(fields_autoplaced yes)
 		(property "Reference" "#GND09"
-			(at 220.98 250.19 0)
+			(at 220.98 242.57 0)
 			(effects
 				(font
@@
 		)
 		(property "Value" "GND"
-			(at 220.98 248.92 0)
+			(at 220.98 241.3 0)
 			(effects
 				(font
@@
 		)
 		(property "Footprint" ""
-			(at 220.98 243.84 0)
+			(at 220.98 236.22 0)
 			(effects
 				(font
@@
 		)
 		(property "Datasheet" ""
-			(at 220.98 243.84 0)
+			(at 220.98 236.22 0)
 			(effects
 				(font
@@
 		)
 		(property "Description" "Power symbol creates a global label with name \"GND\" , ground"
-			(at 220.98 243.84 0)
+			(at 220.98 236.22 0)
 			(effects
 				(font
@@
 	)
 	(symbol
-		(lib_id "power:VCC")
-		(at 471.17 114.3 0)
-		(unit 1)
-		(exclude_from_sim no)
-		(in_bom yes)
-		(on_board yes)
-		(dnp no)
-		(fields_autoplaced yes)
-		(property "Reference" "#VBUSP06"
-			(at 471.17 118.11 0)
-			(effects
-				(font
-					(size 1.27 1.27)
-				)
-				(hide yes)
-			)
-		)
-		(property "Value" "VBUSP"
-			(at 471.17 109.22 0)
-			(effects
-				(font
-					(size 1.27 1.27)
-				)
-			)
-		)
-		(property "Footprint" ""
-			(at 471.17 114.3 0)
-			(effects
-				(font
-					(size 1.27 1.27)
-				)
-				(hide yes)
-			)
-		)
-		(property "Datasheet" ""
-			(at 471.17 114.3 0)
-			(effects
-				(font
-					(size 1.27 1.27)
-				)
-				(hide yes)
-			)
-		)
-		(property "Description" "Power symbol creates a global label with name \"VCC\""
-			(at 471.17 114.3 0)
-			(effects
-				(font
-					(size 1.27 1.27)
-				)
-				(hide yes)
-			)
-		)
-		(pin "1"
-		)
-		(instances
-			(project "oresat-mag-card"
-				(path "/c58960d9-4cac-4036-ad2e-1aef26946dae/2e7c06c0-a412-4c3a-b490-9aec08573322"
-					(reference "#VBUSP06")
-					(unit 1)
-				)
-			)
-		)
-	)
-	(symbol
 		(lib_id "oresat-misc:Test-Point-0.75mm-th")
 		(at 367.03 149.86 0)
@@
 	(symbol
 		(lib_id "Device:R_Small_US")
-		(at 220.98 236.22 0)
+		(at 220.98 231.14 0)
 		(mirror x)
 		(unit 1)
@@
 		(dnp no)
 		(property "Reference" "R23"
-			(at 221.742 240.792 0)
+			(at 221.742 235.712 0)
 			(effects
 				(font
@@
 		)
 		(property "Value" "10k"
-			(at 221.742 238.76 0)
+			(at 221.742 233.68 0)
 			(effects
 				(font
@@
 		)
 		(property "Footprint" "Resistor_SMD:R_0603_1608Metric"
-			(at 220.98 236.22 0)
+			(at 220.98 231.14 0)
 			(effects
 				(font
@@
 		)
 		(property "Datasheet" "~"
-			(at 220.98 236.22 0)
+			(at 220.98 231.14 0)
 			(effects
 				(font
@@
 		)
 		(property "Description" ""
-			(at 220.98 236.22 0)
+			(at 220.98 231.14 0)
 			(effects
 				(font
@@
 		)
 		(property "DIST" ""
-			(at 220.98 236.22 0)
+			(at 220.98 231.14 0)
 			(effects
 				(font
