File: oresat-rw-card/oresat-rw-card.kicad_pcb (KiCad board)
At the start: 4 copper layers, 99.8 x 94.6 mm, 242 parts, among them J1 J-SAMTEC-TFM-120-01-L-D-RA, J2 SM14B-SHLS-TF, Q1 DMP2240UDM, Q10 PMV45EN, Q11 DMP2240UDM, Q12 PMV45EN, Q13 DMP3050LVT-7, Q14 DMP3050LVT-7, Q15 PMV45EN, Q16 DMP2240UDM, Q17 PMV45EN, Q18 DMP3050LVT-7, Q19 DMP3050LVT-7, Q2 PMV45EN, Q20 PMV45EN, Q3 DMP3050LVT-7, Q4 DMP3050LVT-7, Q5 DMP2240UDM, Q6 PMV45EN, Q7 DMP3050LVT-7, Q8 DMP3050LVT-7, Q9 PMV45EN, U1 MAX7310, U10 MAX4211FETE, U11 TPS62111RSA, U12 MAX7310, U13 MIC842LYC5, U14 MIC842LYC5, U15 TS5A21366DCUR, U16 MAX4211FETE, U17 TPS62111RSA, U18 MAX4211FETE, U19 MAX7310, U2 MIC842LYC5, U20 MIC842LYC5, U21 MIC842LYC5, U22 TS5A21366DCUR, U23 MAX4211FETE, U24 TPS62111RSA, U3 MIC842LYC5, U4 MAX7310, U5 TS5A21366DCUR, U6 TPS62111RSA, U7 MIC842LYC5, U8 MIC842LYC5, U9 TS5A21366DCUR

Commit message: RW card needs scrutiny
Parts:
- removed D11, D3, D5, D8: GREEN, oresat-acs-card:LED-0603
- removed L1, L2, L3, L4: 6.8u, oresat-acs-card:ECS-MPI4040
- removed R120, R131, R164, R175, R39, R42, R76, R87: 10k, Resistor_SMD:R_0603_1608Metric
- removed R121, R165, R40, R77: DNP, Resistor_SMD:R_0603_1608Metric
- removed U11, U17, U24, U6: TPS62111RSA, Package_DFN_QFN:Texas_RSA_VQFN-16-1EP_4x4mm_P0.65mm_EP2.7x2.7mm
- moved D6 245.9 mm to (308.1, -87.3)
- moved Q6 245.9 mm to (333.0, -45.0)
- moved Q8 245.9 mm to (336.3, -109.4)
- moved R43 245.9 mm to (312.5, -64.9)
- moved R44 245.9 mm to (312.5, -62.4)
- moved R45 245.9 mm to (312.5, -59.9)
- moved R46 245.9 mm to (312.5, -57.3)
- moved R47 245.9 mm to (286.6, -64.5)
- moved R48 245.9 mm to (254.7, -77.9)
- moved R51 245.9 mm to (263.4, -77.8)
- moved R52 245.9 mm to (312.5, -47.3)
- moved R53 245.9 mm to (289.1, -71.0)
- moved R54 245.9 mm to (316.5, -64.9)
- moved R55 245.9 mm to (316.5, -62.4)
- moved R56 245.9 mm to (316.5, -59.9)
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Connections:
- net /Card Power Domain 2/AD0 renamed /RW Power Domain Q2/AD0
- net /Card Power Domain 2/AD1 renamed /RW Power Domain Q2/AD1
- net /Card Power Domain 2/AD2 renamed /RW Power Domain Q2/AD2
- net /Card Power Domain 2/CB-RESET renamed /RW Power Domain Q2/CB-RESET
- net /Card Power Domain 2/CB_CTRL renamed /RW Power Domain Q2/CB_CTRL
- net /Card Power Domain 2/ON/~{OFF} renamed /RW Power Domain Q2/ON/~{OFF}
- net /Card Power Domain 2/PEN-SCL-FILT renamed /RW Power Domain Q2/PEN-SCL-FILT
- net /Card Power Domain 2/PEN-SDA-FILT renamed /RW Power Domain Q2/PEN-SDA-FILT
- net /Card Power Domain 2/SW_COM1 renamed /RW Power Domain Q2/RW-UART-TX-Q2
- net /Card Power Domain 2/SW_COM2 renamed /RW Power Domain Q2/RW-UART-RX-Q2
- net /Card Power Domain 2/UART_EN renamed /RW Power Domain Q2/UART_EN
- net /Card Power Domain 2/~{FAULT} renamed /RW Power Domain Q2/~{FAULT}
- net /Card Power Domain 3/AD0 renamed /RW Power Domain Q3/AD0
- net /Card Power Domain 3/AD1 renamed /RW Power Domain Q3/AD1
- net /Card Power Domain 3/AD2 renamed /RW Power Domain Q3/AD2
- net /Card Power Domain 3/BOOT_CONFIG renamed /RW Power Domain Q3/BOOT_CONFIG-Q3
- net /Card Power Domain 3/C3-UART-RX renamed /RW Power Domain Q3/C3-UART-RX
- net /Card Power Domain 3/C3-UART-TX renamed /RW Power Domain Q3/C3-UART-TX
- net /Card Power Domain 3/CB-RESET renamed /RW Power Domain Q3/CB-RESET
- net /Card Power Domain 3/CB_CTRL renamed /RW Power Domain Q3/CB_CTRL
- net /Card Power Domain 3/ON/~{OFF} renamed /RW Power Domain Q3/ON/~{OFF}
- net /Card Power Domain 3/OPD_PWR renamed /RW Power Domain Q3/OPD_PWR
- net /Card Power Domain 3/OPD_SCL renamed /RW Power Domain Q3/OPD_SCL
- net /Card Power Domain 3/OPD_SDA renamed /RW Power Domain Q3/OPD_SDA
- net /Card Power Domain 3/PEN-SCL-FILT renamed /RW Power Domain Q3/PEN-SCL-FILT
- net /Card Power Domain 3/PEN-SDA-FILT renamed /RW Power Domain Q3/PEN-SDA-FILT
- net /Card Power Domain 3/SW_COM1 renamed /RW Power Domain Q3/RW-UART-TX-Q3
- net /Card Power Domain 3/SW_COM2 renamed /RW Power Domain Q3/RW-UART-RX-Q3
- net /Card Power Domain 3/UART_EN renamed /RW Power Domain Q3/UART_EN
- net /Card Power Domain 3/~{FAULT} renamed /RW Power Domain Q3/~{FAULT}
- net /Card Power Domain 4/AD0 renamed /RW Power Domain Q4/AD0
- net /Card Power Domain 4/AD1 renamed /RW Power Domain Q4/AD1
- net /Card Power Domain 4/AD2 renamed /RW Power Domain Q4/AD2
- net /Card Power Domain 4/BOOT_CONFIG renamed /RW Power Domain Q4/BOOT_CONFIG-Q4
- net /Card Power Domain 4/C3-UART-RX renamed /RW Power Domain Q4/C3-UART-RX
- net /Card Power Domain 4/C3-UART-TX renamed /RW Power Domain Q4/C3-UART-TX
- net /Card Power Domain 4/CB-RESET renamed /RW Power Domain Q4/CB-RESET
- net /Card Power Domain 4/CB_CTRL renamed /RW Power Domain Q4/CB_CTRL
- net /Card Power Domain 4/ON/~{OFF} renamed /RW Power Domain Q4/ON/~{OFF}
- net /Card Power Domain 4/OPD_PWR renamed /RW Power Domain Q4/OPD_PWR
- net /Card Power Domain 4/OPD_SCL renamed /RW Power Domain Q4/OPD_SCL
- net /Card Power Domain 4/OPD_SDA renamed /RW Power Domain Q4/OPD_SDA
- net /Card Power Domain 4/PEN-SCL-FILT renamed /RW Power Domain Q4/PEN-SCL-FILT
- net /Card Power Domain 4/PEN-SDA-FILT renamed /RW Power Domain Q4/PEN-SDA-FILT
- net /Card Power Domain 4/SW_COM1 renamed /RW Power Domain Q4/RW-UART-TX-Q4
- net /Card Power Domain 4/SW_COM2 renamed /RW Power Domain Q4/RW-UART-RX-Q4
- net /Card Power Domain 4/UART_EN renamed /RW Power Domain Q4/UART_EN
- net /Card Power Domain 4/~{FAULT} renamed /RW Power Domain Q4/~{FAULT}
- net /Card Power Domain/AD0 renamed /RW Power Domain Q1/AD0
- net /Card Power Domain/AD1 renamed /RW Power Domain Q1/AD1
- net /Card Power Domain/AD2 renamed /RW Power Domain Q1/AD2
- net /Card Power Domain/CB-RESET renamed /RW Power Domain Q1/CB-RESET
- net /Card Power Domain/CB_CTRL renamed /RW Power Domain Q1/CB_CTRL
- net /Card Power Domain/ON/~{OFF} renamed /RW Power Domain Q1/ON/~{OFF}
- net /Card Power Domain/PEN-SCL-FILT renamed /RW Power Domain Q1/PEN-SCL-FILT
- net /Card Power Domain/PEN-SDA-FILT renamed /RW Power Domain Q1/PEN-SDA-FILT
- net /Card Power Domain/UART_EN renamed /RW Power Domain Q1/UART_EN
- net /Card Power Domain/~{FAULT} renamed /RW Power Domain Q1/~{FAULT}
- J1 pad 1: /MAG_SDA -> unconnected-(J1-Pad1)
- J1 pad 11: /OPD_SDA -> /RW Power Domain Q1/OPD_SDA
- J1 pad 12: /OPD_SDA -> /RW Power Domain Q1/OPD_SDA
- J1 pad 13: /OPD_SCL -> /RW Power Domain Q1/OPD_SCL
- J1 pad 14: /OPD_SCL -> /RW Power Domain Q1/OPD_SCL
- J1 pad 15: /OPD_PWR -> /RW Power Domain Q1/OPD_PWR
- J1 pad 16: /OPD_PWR -> /RW Power Domain Q1/OPD_PWR
- J1 pad 2: /MAG_SDA -> unconnected-(J1-Pad2)
- J1 pad 3: /MAG_SCL -> unconnected-(J1-Pad3)
- J1 pad 4: /MAG_SCL -> unconnected-(J1-Pad4)
- J1 pad 5: MAG_PWR -> unconnected-(J1-Pad5)
- J1 pad 6: MAG_PWR -> unconnected-(J1-Pad6)
- Q14 pad 1: VBUSP -> VBUSP-Q3
- Q14 pad 2: VBUSP -> VBUSP-Q3
- Q14 pad 5: VBUSP -> VBUSP-Q3
- Q14 pad 6: VBUSP -> VBUSP-Q3
- Q19 pad 1: VBUSP -> VBUSP-Q4
- Q19 pad 2: VBUSP -> VBUSP-Q4
- Q19 pad 5: VBUSP -> VBUSP-Q4
- Q19 pad 6: VBUSP -> VBUSP-Q4
- Q4 pad 1: VBUSP -> /RW Power Domain Q1/VBUSP-Q1
- Q4 pad 2: VBUSP -> /RW Power Domain Q1/VBUSP-Q1
- Q4 pad 5: VBUSP -> /RW Power Domain Q1/VBUSP-Q1
- Q4 pad 6: VBUSP -> /RW Power Domain Q1/VBUSP-Q1
- Q8 pad 1: VBUSP -> VBUSP-Q2
- Q8 pad 2: VBUSP -> VBUSP-Q2
- Q8 pad 5: VBUSP -> VBUSP-Q2
- Q8 pad 6: VBUSP -> VBUSP-Q2
- R1 pad 1: VPD -> VPD-Q1
- R1 pad 2: /OPD_PWR -> /RW Power Domain Q1/OPD_PWR
- R13 pad 1: VPD -> VPD-Q1
- R130 pad 2: VPD -> VPD-Q3
- R132 pad 2: VBUSP -> VBUSP-Q3
- R174 pad 2: VPD -> VPD-Q4
- R176 pad 2: VBUSP -> VBUSP-Q4
- R18 pad 2: VPD -> VPD-Q1
- R21 pad 2: VPD -> VPD-Q1
- R22 pad 2: VPD -> VPD-Q1
- R3 pad 1: VPD -> VPD-Q1
- R38 pad 2: VPD -> VPD-Q1
- R41 pad 2: VBUSP -> /RW Power Domain Q1/VBUSP-Q1
- R43 pad 2: /Card Power Domain 2/OPD_PWR -> /RW Power Domain Q1/OPD_PWR
- R48 pad 2: /Card Power Domain 2/OPD_SCL -> /RW Power Domain Q1/OPD_SCL
- R51 pad 2: /Card Power Domain 2/OPD_SDA -> /RW Power Domain Q1/OPD_SDA
- R6 pad 2: /OPD_SCL -> /RW Power Domain Q1/OPD_SCL
- R7 pad 2: /OPD_SDA -> /RW Power Domain Q1/OPD_SDA
- R71 pad 1: /Card Power Domain 2/C3-UART-RX -> /C3-UART-RX
- R72 pad 1: /Card Power Domain 2/C3-UART-TX -> /C3-UART-TX
- R86 pad 2: VPD -> VPD-Q2
- R88 pad 2: VBUSP -> VBUSP-Q2
- R9 pad 1: VPD -> VPD-Q1
- U1 pad 10: /Card Power Domain 2/BOOT_CONFIG -> /RW Power Domain Q1/BOOT_CONFIG
- U1 pad 14: VPD -> VPD-Q1
- U2 pad 5: VPD -> VPD-Q1
- U3 pad 5: VPD -> VPD-Q1
- U4 pad 10: /Card Power Domain 2/BOOT_CONFIG -> /RW Power Domain Q2/BOOT_CONFIG-Q2
- U5 pad 2: /Card Power Domain/SW_COM1 -> /RW Power Domain Q1/RW-UART-TX-Q1
- U5 pad 6: /Card Power Domain/SW_COM2 -> /RW Power Domain Q1/RW-UART-RX-Q1
Routing:
- net /RW Power Domain Q1/UART_EN: track 0.00 -> 40.8 mm, vias 0 -> 2
- net /RW Power Domain Q1/ON/~{OFF}: track 0.00 -> 38.1 mm
- net /RW Power Domain Q1/PEN-SCL-FILT: track 0.00 -> 37.5 mm, vias 0 -> 4
- net VPD-Q1: track 0.00 -> 37.0 mm, vias 0 -> 3
- net /RW Power Domain Q1/CB_CTRL: track 0.00 -> 32.9 mm, vias 0 -> 3
- net /RW Power Domain Q1/PEN-SDA-FILT: track 0.00 -> 26.2 mm, vias 0 -> 2
- net /RW Power Domain Q1/AD2: track 0.00 -> 24.5 mm
- net Net-(Q4-S): track 0.00 -> 18.5 mm, vias 0 -> 2
- net /RW Power Domain Q1/CB-RESET: track 0.00 -> 16.9 mm, vias 0 -> 2
- net Net-(U3-OUT): track 0.00 -> 16.8 mm, vias 0 -> 2
- net /RW Power Domain Q1/AD1: track 0.00 -> 14.6 mm
- net Net-(Q1B-G): track 0.00 -> 10.0 mm
- net Net-(Q2-D): track 0.00 -> 9.86 mm, vias 0 -> 2
- net /RW Power Domain Q1/AD0: track 0.00 -> 8.85 mm
- net Net-(U18-CIN2+): track 0.00 -> 8.13 mm, vias 0 -> 2
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- added copper zone on F.Cu, net Net-(U18-RS+)

Commit message: Schematic Done + Board outline set
Fixed heirarchical labels, cleaned up ERCs, board is ready for layout
Parts:
- removed J2: SM14B-SHLS-TF, oresat-connectors:J-JST-SM14BSHLSTF
- added C11: 1u, Capacitor_SMD:C_0201_0603Metric, F.Cu at (214.7, 53.8)
- added C12: 1u, Capacitor_SMD:C_0201_0603Metric, F.Cu at (243.6, -26.5)
- added C13: 100n, Capacitor_SMD:C_0201_0603Metric, F.Cu at (61.6, 141.0)
- added C14: 1u, Capacitor_SMD:C_0201_0603Metric, F.Cu at (128.8, 177.8)
- added C15: 100n, Capacitor_SMD:C_0201_0603Metric, F.Cu at (128.8, 179.6)
- added C16: 1u, Capacitor_SMD:C_0201_0603Metric, F.Cu at (128.8, 181.3)
- added C19: 10n, Capacitor_SMD:C_0201_0603Metric, F.Cu at (128.8, 183.1)
- added C2: 1u, Capacitor_SMD:C_0201_0603Metric, F.Cu at (174.2, 123.7)
- added C20: 470n, Capacitor_SMD:C_0201_0603Metric, F.Cu at (296.7, -49.8)
- added C22: 1u, Capacitor_SMD:C_0201_0603Metric, F.Cu at (68.4, 60.1)
- added C23: 1u, Capacitor_SMD:C_0201_0603Metric, F.Cu at (124.4, 174.3)
- added C24: 100n, Capacitor_SMD:C_0201_0603Metric, F.Cu at (124.4, 176.1)
- added C25: 1u, Capacitor_SMD:C_0201_0603Metric, F.Cu at (38.6, 55.7)
- added C26: 100n, Capacitor_SMD:C_0201_0603Metric, F.Cu at (124.4, 179.6)
- added C27: 1u, Capacitor_SMD:C_0201_0603Metric, F.Cu at (124.4, 181.3)
- added C3: 1u, Capacitor_SMD:C_0201_0603Metric, F.Cu at (168.1, 129.9)
- added C30: 10n, Capacitor_SMD:C_0201_0603Metric, F.Cu at (124.4, 183.1)
- added C31: 470n, Capacitor_SMD:C_0201_0603Metric, F.Cu at (71.1, 34.2)
- added C33: 1u, Capacitor_SMD:C_0201_0603Metric, F.Cu at (61.9, 162.0)
- added C34: 1u, Capacitor_SMD:C_0201_0603Metric, F.Cu at (59.2, 158.4)
- added C35: 100n, Capacitor_SMD:C_0201_0603Metric, F.Cu at (52.1, 126.6)
- added C36: 1u, Capacitor_SMD:C_0201_0603Metric, F.Cu at (133.3, 177.8)
- added C37: 100n, Capacitor_SMD:C_0201_0603Metric, F.Cu at (133.3, 179.6)
- added C38: 1u, Capacitor_SMD:C_0201_0603Metric, F.Cu at (133.3, 181.3)
- added C4: 100n, Capacitor_SMD:C_0201_0603Metric, F.Cu at (139.0, 123.4)
- added C41: 10n, Capacitor_SMD:C_0201_0603Metric, F.Cu at (133.3, 183.1)
- added C42: 470n, Capacitor_SMD:C_0201_0603Metric, F.Cu at (133.3, 184.8)
- added C5: 100n, Capacitor_SMD:C_0201_0603Metric, F.Cu at (120.0, 177.8)
- added C6: 1u, Capacitor_SMD:C_0201_0603Metric, F.Cu at (120.0, 179.6)
- added C68: 10n, Capacitor_SMD:C_0201_0603Metric, F.Cu at (126.0, 141.9)
- added C69: 470n, Capacitor_SMD:C_0201_0603Metric, F.Cu at (133.2, 127.4)
- added C7: 1u, Capacitor_SMD:C_0201_0603Metric, F.Cu at (120.0, 181.3)
- added J3: 0555600307, oresat-connectors:J-Molex-555600307, F.Cu at (48.1, 83.5)
- added J4: 0555600307, oresat-connectors:J-Molex-555600307, F.Cu at (48.1, 89.5)
- added J5: 0555600307, oresat-connectors:J-Molex-555600307, F.Cu at (36.6, 95.2)
- added J6: 0555600307, oresat-connectors:J-Molex-555600307, F.Cu at (48.1, 101.5)
- added R129: 10k, oresat-passives:0603-C-NOSILK, F.Cu at (55.9, 100.8)
- added R173: 10k, oresat-passives:0603-C-NOSILK, F.Cu at (70.5, 100.8)
- added R50: 10k, oresat-passives:0603-C-NOSILK, F.Cu at (55.9, 89.1)
- added R85: 10k, oresat-passives:0603-C-NOSILK, F.Cu at (70.5, 89.1)
- added TP10: Test-Point, oresat-misc:TestPoint-0.75mm-th, F.Cu at (60.6, 86.8)
- added TP11: Test-Point, oresat-misc:TestPoint-0.75mm-th, F.Cu at (63.1, 81.8)
- added TP12: Test-Point, oresat-misc:TestPoint-0.75mm-th, F.Cu at (63.1, 84.3)
- added TP13: Test-Point, oresat-misc:TestPoint-0.75mm-th, F.Cu at (63.1, 86.8)
- added TP14: Test-Point, oresat-misc:TestPoint-0.75mm-th, F.Cu at (65.7, 81.8)
- added TP15: Test-Point, oresat-misc:TestPoint-0.75mm-th, F.Cu at (65.7, 84.3)
- added TP17: Test-Point, oresat-misc:TestPoint-0.75mm-th, F.Cu at (65.7, 86.8)
- added TP2: Test-Point, oresat-misc:TestPoint-0.75mm-th, F.Cu at (55.6, 81.8)
- added TP20: Test-Point, oresat-misc:TestPoint-0.75mm-th, F.Cu at (70.2, 81.8)
- added TP21: Test-Point, oresat-misc:TestPoint-0.75mm-th, F.Cu at (70.2, 84.3)
- added TP22: Test-Point, oresat-misc:TestPoint-0.75mm-th, F.Cu at (70.2, 86.8)
- added TP23: Test-Point, oresat-misc:TestPoint-0.75mm-th, F.Cu at (72.7, 81.8)
- added TP24: Test-Point, oresat-misc:TestPoint-0.75mm-th, F.Cu at (72.7, 84.3)
- added TP25: Test-Point, oresat-misc:TestPoint-0.75mm-th, F.Cu at (72.7, 86.8)
- added TP26: Test-Point, oresat-misc:TestPoint-0.75mm-th, F.Cu at (75.2, 81.8)
- added TP27: Test-Point, oresat-misc:TestPoint-0.75mm-th, F.Cu at (75.2, 84.3)
- added TP28: Test-Point, oresat-misc:TestPoint-0.75mm-th, F.Cu at (75.2, 86.8)
- added TP29: Test-Point, oresat-misc:TestPoint-0.75mm-th, F.Cu at (77.8, 81.8)
- added TP3: Test-Point, oresat-misc:TestPoint-0.75mm-th, F.Cu at (55.6, 84.3)
- added TP31: Test-Point, oresat-misc:TestPoint-0.75mm-th, F.Cu at (77.8, 84.3)
- added TP32: Test-Point, oresat-misc:TestPoint-0.75mm-th, F.Cu at (77.8, 86.8)
- added TP33: Test-Point, oresat-misc:TestPoint-0.75mm-th, F.Cu at (80.3, 81.8)
- added TP36: Test-Point, oresat-misc:TestPoint-0.75mm-th, F.Cu at (80.3, 84.3)
- added TP37: Test-Point, oresat-misc:TestPoint-0.75mm-th, F.Cu at (80.3, 86.8)
- added TP38: Test-Point, oresat-misc:TestPoint-0.75mm-th, F.Cu at (55.6, 93.4)
- added TP39: Test-Point, oresat-misc:TestPoint-0.75mm-th, F.Cu at (55.6, 96.0)
- added TP4: Test-Point, oresat-misc:TestPoint-0.75mm-th, F.Cu at (55.6, 86.8)
- added TP40: Test-Point, oresat-misc:TestPoint-0.75mm-th, F.Cu at (55.6, 98.5)
- added TP41: Test-Point, oresat-misc:TestPoint-0.75mm-th, F.Cu at (58.1, 93.4)
- added TP42: Test-Point, oresat-misc:TestPoint-0.75mm-th, F.Cu at (58.1, 96.0)
- added TP43: Test-Point, oresat-misc:TestPoint-0.75mm-th, F.Cu at (58.1, 98.5)
- added TP44: Test-Point, oresat-misc:TestPoint-0.75mm-th, F.Cu at (60.6, 93.4)
- added TP45: Test-Point, oresat-misc:TestPoint-0.75mm-th, F.Cu at (60.6, 96.0)
- added TP46: Test-Point, oresat-misc:TestPoint-0.75mm-th, F.Cu at (60.6, 98.5)
- added TP47: Test-Point, oresat-misc:TestPoint-0.75mm-th, F.Cu at (63.1, 93.4)
- added TP49: Test-Point, oresat-misc:TestPoint-0.75mm-th, F.Cu at (63.1, 96.0)
- added TP5: Test-Point, oresat-misc:TestPoint-0.75mm-th, F.Cu at (58.1, 81.8)
- added TP50: Test-Point, oresat-misc:TestPoint-0.75mm-th, F.Cu at (63.1, 98.5)
- added TP51: Test-Point, oresat-misc:TestPoint-0.75mm-th, F.Cu at (65.7, 93.4)
- added TP54: Test-Point, oresat-misc:TestPoint-0.75mm-th, F.Cu at (65.7, 96.0)
- added TP55: Test-Point, oresat-misc:TestPoint-0.75mm-th, F.Cu at (65.7, 98.5)
- added TP56: Test-Point, oresat-misc:TestPoint-0.75mm-th, F.Cu at (70.2, 93.4)
- added TP57: Test-Point, oresat-misc:TestPoint-0.75mm-th, F.Cu at (70.2, 96.0)
- added TP58: Test-Point, oresat-misc:TestPoint-0.75mm-th, F.Cu at (70.2, 98.5)
- added TP59: Test-Point, oresat-misc:TestPoint-0.75mm-th, F.Cu at (72.7, 93.4)
- added TP6: Test-Point, oresat-misc:TestPoint-0.75mm-th, F.Cu at (58.1, 84.3)
- added TP60: Test-Point, oresat-misc:TestPoint-0.75mm-th, F.Cu at (72.7, 96.0)
- added TP61: Test-Point, oresat-misc:TestPoint-0.75mm-th, F.Cu at (72.7, 98.5)
- added TP62: Test-Point, oresat-misc:TestPoint-0.75mm-th, F.Cu at (75.2, 93.4)
- added TP63: Test-Point, oresat-misc:TestPoint-0.75mm-th, F.Cu at (75.2, 96.0)
- added TP64: Test-Point, oresat-misc:TestPoint-0.75mm-th, F.Cu at (75.2, 98.5)
- added TP65: Test-Point, oresat-misc:TestPoint-0.75mm-th, F.Cu at (77.8, 93.4)
- added TP67: Test-Point, oresat-misc:TestPoint-0.75mm-th, F.Cu at (77.8, 96.0)
- added TP68: Test-Point, oresat-misc:TestPoint-0.75mm-th, F.Cu at (77.8, 98.5)
- added TP69: Test-Point, oresat-misc:TestPoint-0.75mm-th, F.Cu at (80.3, 93.4)
- added TP7: Test-Point, oresat-misc:TestPoint-0.75mm-th, F.Cu at (58.1, 86.8)
- added TP72: Test-Point, oresat-misc:TestPoint-0.75mm-th, F.Cu at (80.3, 96.0)
- added TP73: Test-Point, oresat-misc:TestPoint-0.75mm-th, F.Cu at (80.3, 98.5)
- added TP8: Test-Point, oresat-misc:TestPoint-0.75mm-th, F.Cu at (60.6, 81.8)
- added TP9: Test-Point, oresat-misc:TestPoint-0.75mm-th, F.Cu at (60.6, 84.3)
- C1: footprint Capacitor_SMD:C_1206_3216Metric -> Capacitor_SMD:C_0805_2012Metric
- moved Q3 23.3 mm to (142.6, 136.9)
- moved R10 23.3 mm to (147.2, 128.8)
- moved R15 23.3 mm to (150.1, 121.9)
- moved R16 23.3 mm to (151.7, 128.8)
- moved R19 23.3 mm to (165.6, 123.4)
- moved R26 23.3 mm to (137.2, 143.0)
- moved R27 23.3 mm to (159.1, 141.9)
- moved R32 23.3 mm to (153.1, 142.9)
- moved R36 23.3 mm to (154.2, 137.9)
- moved R4 23.3 mm to (142.7, 128.8)
- moved R6 23.3 mm to (150.1, 123.4)
- moved U1 23.3 mm to (157.6, 134.0)
- moved R1 23.3 mm to (160.1, 122.8)
- moved R11 23.3 mm to (148.7, 131.1)
- moved R12 23.3 mm to (150.2, 130.5)
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Connections:
- net VBUSP-Q2 renamed /RW Power Domain Q2/VBUSP-Q2
- net VBUSP-Q3 renamed /RW Power Domain Q3/VBUSP-Q3
- net VBUSP-Q4 renamed /RW Power Domain Q4/VBUSP-Q4
- J1 pad 11: /RW Power Domain Q1/OPD_SDA -> /OPD_SDA
- J1 pad 12: /RW Power Domain Q1/OPD_SDA -> /OPD_SDA
- J1 pad 13: /RW Power Domain Q1/OPD_SCL -> /OPD_SCL
- J1 pad 14: /RW Power Domain Q1/OPD_SCL -> /OPD_SCL
- J1 pad 15: /RW Power Domain Q1/OPD_PWR -> /OPD_PWR
- J1 pad 16: /RW Power Domain Q1/OPD_PWR -> /OPD_PWR
- R1 pad 2: /RW Power Domain Q1/OPD_PWR -> /OPD_PWR
- R115 pad 1: /RW Power Domain Q3/C3-UART-RX -> /C3-UART-RX
- R116 pad 1: /RW Power Domain Q3/C3-UART-TX -> /C3-UART-TX
- R133 pad 2: /RW Power Domain Q4/OPD_PWR -> /OPD_PWR
- R138 pad 2: /RW Power Domain Q4/OPD_SCL -> /OPD_SCL
- R139 pad 2: /RW Power Domain Q4/OPD_SDA -> /OPD_SDA
- R159 pad 1: /RW Power Domain Q4/C3-UART-RX -> /C3-UART-RX
- R160 pad 1: /RW Power Domain Q4/C3-UART-TX -> /C3-UART-TX
- R43 pad 2: /RW Power Domain Q1/OPD_PWR -> /OPD_PWR
- R48 pad 2: /RW Power Domain Q1/OPD_SCL -> /OPD_SCL
- R51 pad 2: /RW Power Domain Q1/OPD_SDA -> /OPD_SDA
- R6 pad 2: /RW Power Domain Q1/OPD_SCL -> /OPD_SCL
- R7 pad 2: /RW Power Domain Q1/OPD_SDA -> /OPD_SDA
- R89 pad 2: /RW Power Domain Q3/OPD_PWR -> /OPD_PWR
- R94 pad 2: /RW Power Domain Q3/OPD_SCL -> /OPD_SCL
- R95 pad 2: /RW Power Domain Q3/OPD_SDA -> /OPD_SDA
- U1 pad 10: /RW Power Domain Q1/BOOT_CONFIG -> /RW Power Domain Q1/BOOTCFG-Q1
- U12 pad 10: /RW Power Domain Q3/BOOT_CONFIG-Q3 -> /RW Power Domain Q3/BOOTCFG-Q3
- U19 pad 10: /RW Power Domain Q4/BOOT_CONFIG-Q4 -> /RW Power Domain Q4/BOOTCFG-Q4
- U4 pad 10: /RW Power Domain Q2/BOOT_CONFIG-Q2 -> /CAN2_L
- U9 pad 6: /RW Power Domain Q2/RW-UART-RX-Q2 -> /CAN2_H
Routing:
- added copper zone on In1.Cu, net GND

Commit message: Lots of work needs to be done still
Parts:
- C11, C12, C13, C14, C15, C16, C19, C2, C20, C22, C23, C24, C25, C26, C27, C3, C30, C31, C33, C34, C35, C36, C37, C38, C4, C41, C42, C5, C6, C68, C69, C7: footprint Capacitor_SMD:C_0201_0603Metric -> Capacitor_SMD:C_0603_1608Metric
- D1, D10, D12, D2, D4, D6, D7, D9: footprint oresat-acs-card:LED-0603 -> LED_SMD:LED_0603_1608Metric_Pad1.05x0.95mm_HandSolder
- moved TP5 116.3 mm to (163.1, 131.9)
- moved TP6 116.0 mm to (163.1, 133.6)
- moved TP7 110.3 mm to (163.1, 120.5)
- moved TP12 108.5 mm to (155.4, 141.4)
- moved TP15 106.3 mm to (157.2, 138.3)
- moved TP13 105.4 mm to (151.4, 144.4)
- moved TP10 105.2 mm to (148.1, 145.3)
- moved TP11 104.4 mm to (150.6, 138.8)
- moved TP14 101.1 mm to (151.2, 135.6)
- moved TP3 99.3 mm to (143.0, 131.3)
- moved TP2 97.6 mm to (139.8, 130.9)
- moved TP4 96.1 mm to (143.1, 126.5)
- moved TP8 95.5 mm to (147.3, 121.9)
- moved R50 90.0 mm to (131.2, 138.5)
- moved C4 87.6 mm to (224.8, 105.9)
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Routing:
- net /RW Power Domain Q1/ON/~{OFF}: track 38.1 -> 62.8 mm, vias 0 -> 1
- net VPD-Q1: track 37.0 -> 45.6 mm, vias 3 -> 4
- net Net-(C7-Pad2): track 1.50 -> 9.56 mm, vias 0 -> 2
- net /RW Power Domain Q1/AD1: track 14.6 -> 22.4 mm
- net /RW Power Domain Q1/AD0: track 8.85 -> 16.5 mm
- net /RW Power Domain Q1/VBUSP-Q1: track 5.84 -> 10.9 mm
- net /RW Power Domain Q1/UART_EN: track 40.8 -> 36.4 mm
- net Net-(U1-IO6): track 0.00 -> 4.18 mm
- net /RW Power Domain Q1/AD2: track 24.5 -> 27.7 mm
- net /RW Power Domain Q1/PEN-SDA-FILT: track 26.2 -> 29.4 mm, vias 2 -> 4
- net Net-(U5-NO1): track 1.85 -> 4.37 mm
- net Net-(U18-CIN1+): track 7.93 -> 10.2 mm
- net /RW Power Domain Q1/PEN-SCL-FILT: track 37.5 -> 39.7 mm, vias 4 -> 5
- net Net-(Q2-D): track 9.86 -> 7.79 mm
- net Net-(U3-OUT): track 16.8 -> 18.8 mm
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
Commit message: Push for design review
Parts:
- added C10: 100n, Capacitor_SMD:C_0603_1608Metric, F.Cu at (99.7, 167.9)
- added C17: 100n, Capacitor_SMD:C_0603_1608Metric, F.Cu at (99.7, 170.4)
- added C18: 100n, Capacitor_SMD:C_0603_1608Metric, F.Cu at (105.7, 159.9)
- added C21: 100n, Capacitor_SMD:C_0603_1608Metric, F.Cu at (105.7, 163.4)
- added C28: 100n, Capacitor_SMD:C_0603_1608Metric, F.Cu at (105.7, 167.9)
- added C29: 100n, Capacitor_SMD:C_0603_1608Metric, F.Cu at (105.7, 170.4)
- added C8: 100n, Capacitor_SMD:C_0603_1608Metric, F.Cu at (99.7, 160.9)
- added C9: 100n, Capacitor_SMD:C_0603_1608Metric, F.Cu at (99.7, 163.4)
- D12, D6, D9: footprint LED_SMD:LED_0603_1608Metric_Pad1.05x0.95mm_HandSolder -> oresat-acs-card:LED-0603
- moved C4 64.3 mm to (164.8, 129.2)
- moved TP13 23.0 mm to (152.2, 121.4)
- moved TP8 19.3 mm to (162.3, 134.1)
- moved Q4 19.3 mm to (143.3, 120.3)
- moved TP11 18.8 mm to (146.3, 120.4)
- moved U18 18.5 mm to (148.6, 123.5), turned to 90 degrees
- moved D2 17.9 mm to (146.6, 145.9), turned to 90 degrees
- moved D1 17.7 mm to (145.0, 145.9), turned to 90 degrees
- moved R31 15.5 mm to (143.0, 123.0)
- moved Q3 15.4 mm to (138.4, 122.5)
- moved R41 14.9 mm to (146.6, 142.7), turned to 90 degrees
- moved R27 14.1 mm to (145.0, 142.7), turned to 90 degrees
- moved TP10 12.4 mm to (136.0, 148.0)
- moved R15 9.63 mm to (146.2, 130.7)
- moved R6 9.63 mm to (146.2, 132.2)
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Routing:
- net /RW Power Domain Q1/CB_CTRL: track 34.3 -> 68.3 mm, vias 3 -> 2
- net Net-(Q4-G): track 5.75 -> 35.8 mm
- net /RW Power Domain Q1/VBUSP-Q1: track 10.9 -> 40.8 mm, vias 0 -> 1
- net Net-(U18-CIN1-): track 3.51 -> 31.9 mm, vias 0 -> 1
- net Net-(U18-IOUT): track 3.54 -> 28.8 mm, vias 0 -> 4
- net /RW Power Domain Q1/CB-RESET: track 18.8 -> 40.7 mm, vias 2 -> 3
- net VBUS: track 4.41 -> 25.9 mm
- net Net-(Q2-D): track 7.79 -> 28.6 mm
- net Net-(U18-CIN2+): track 8.13 -> 28.8 mm
- net Net-(U18-INHIBIT): track 3.80 -> 23.4 mm
- net Net-(U18-CIN1+): track 10.2 -> 29.5 mm, vias 2 -> 1
- net Net-(Q4-S): track 20.2 -> 31.1 mm
- net Net-(U3-OUT): track 18.8 -> 27.7 mm, vias 2 -> 1
- net /RW Power Domain Q1/ON/~{OFF}: track 62.8 -> 54.6 mm, vias 1 -> 2
- net VPD-Q1: track 45.6 -> 51.8 mm, vias 4 -> 8
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- added copper zone on F.Cu, net /RW Power Domain Q1/VBUSP-Q1
- added copper zone on F.Cu, net Net-(Q4-S)
- added copper zone on In2.Cu, net VBUS

Commit message: Push for preservation
Parts:
- moved C9 94.2 mm to (175.5, 107.3), turned to 180 degrees
- moved C8 85.3 mm to (173.2, 117.6), turned to -90 degrees
- moved C6 45.0 mm to (155.5, 170.0)
- moved R31 42.9 mm to (154.8, 164.3), turned to 90 degrees
- moved TP11 41.6 mm to (157.2, 160.6)
- moved TP13 41.6 mm to (163.2, 161.5)
- moved U18 41.6 mm to (159.5, 163.6)
- moved R22 32.3 mm to (175.5, 105.8)
- moved R15 31.6 mm to (170.4, 110.3), turned to 180 degrees
- moved R20 29.7 mm to (173.0, 106.4), turned to 90 degrees
- moved R6 29.1 mm to (167.9, 112.8), turned to 90 degrees
- moved R33 28.7 mm to (166.8, 168.8)
- moved R34 28.7 mm to (165.7, 165.3)
- moved R35 28.7 mm to (168.3, 168.8)
- moved R36 28.7 mm to (168.7, 165.3)
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Routing:
- net /RW Power Domain Q1/CB_CTRL: track 68.3 -> 0.00 mm, vias 2 -> 0
- net /RW Power Domain Q1/ON/~{OFF}: track 54.6 -> 0.00 mm, vias 2 -> 0
- net /RW Power Domain Q1/CB-RESET: track 40.7 -> 0.00 mm, vias 3 -> 0
- net Net-(Q4-G): track 35.8 -> 0.00 mm
- net Net-(U18-CIN1-): track 31.9 -> 0.00 mm, vias 1 -> 0
- net Net-(Q4-S): track 31.1 -> 0.00 mm, vias 2 -> 0
- net Net-(U18-CIN1+): track 29.5 -> 0.00 mm, vias 1 -> 0
- net Net-(U18-IOUT): track 28.8 -> 0.00 mm, vias 4 -> 0
- net Net-(U18-CIN2+): track 28.8 -> 0.00 mm, vias 2 -> 0
- net Net-(Q2-D): track 28.6 -> 0.00 mm, vias 2 -> 0
- net /RW Power Domain Q1/UART_EN: track 30.8 -> 2.57 mm, vias 3 -> 0
- net VPD-Q1: track 51.8 -> 25.6 mm, vias 8 -> 3
- net Net-(U18-INHIBIT): track 23.4 -> 0.00 mm, vias 2 -> 0
- net VBUS: track 25.9 -> 2.69 mm
- net /RW Power Domain Q1/PEN-SCL-FILT: track 35.8 -> 15.3 mm, vias 7 -> 0
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- removed copper zone on F.Cu, net /RW Power Domain Q1/VBUSP-Q1
- removed copper zone on F.Cu, net Net-(Q4-S)

Commit message: Minor changes
Parts:
- moved R3 33.7 mm to (167.7, 122.6), turned to 180 degrees
- moved R5 32.6 mm to (167.7, 124.1), turned to 180 degrees
- moved TP15 32.5 mm to (184.6, 159.2)
- moved Q9 31.6 mm to (187.5, 160.9)
- moved R38 31.6 mm to (187.5, 157.4)
- moved R2 28.3 mm to (164.7, 122.6), turned to 180 degrees
- moved C2 28.2 mm to (158.5, 136.4)
- moved Q1 28.2 mm to (151.5, 133.2)
- moved R19 28.2 mm to (160.1, 136.4)
- moved R21 28.2 mm to (156.1, 138.6)
- moved U3 28.2 mm to (155.9, 129.9)
- moved C8 28.2 mm to (153.8, 138.0)
- moved R14 28.2 mm to (151.0, 135.7)
- moved R20 28.2 mm to (153.6, 126.8)
- moved TP7 28.2 mm to (153.5, 135.7)
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Routing:
- net /RW Power Domain Q1/PEN-SCL-FILT: track 15.3 -> 39.0 mm
- net /RW Power Domain Q1/VBUSP-Q1: track 27.3 -> 3.96 mm
- net /RW Power Domain Q1/PEN-SDA-FILT: track 24.0 -> 44.3 mm, vias 0 -> 3
- net VPD-Q1: track 25.6 -> 45.4 mm, vias 3 -> 7
- net /RW Power Domain Q1/~{FAULT}: track 12.4 -> 1.74 mm
- net Net-(U1-~{RESET}): track 0.00 -> 3.54 mm
- net Net-(U3-OUT): track 9.54 -> 7.23 mm
- net /RW Power Domain Q1/AD0: track 9.82 -> 11.7 mm, vias 0 -> 2
- net /RW Power Domain Q1/AD2: track 9.82 -> 10.6 mm, vias 0 -> 2
- net /RW Power Domain Q1/AD1: track 9.82 -> 9.59 mm, vias 0 -> 2
- added copper zone on F.Cu, net /RW Power Domain Q1/AD0
- added copper zone on F.Cu, net /RW Power Domain Q1/AD1
- added copper zone on F.Cu, net /RW Power Domain Q1/AD2
