File: oresat-rw-card/oresat-rw-card-sch-q3.kicad_sch (KiCad schematic)
At the start: 78 parts, among them Q11 DMP2240UDM, Q12 PMV45EN, Q13 DMP3050LVT-7, Q14 DMP3050LVT-7, Q15 PMV45EN, U12 MAX7310, U13 MIC842LYC5, U14 MIC842LYC5, U15 TS5A21366DCUR, U16 MAX4211FETE

Commit message: Design review on current state of sch/brd
Parts:
- R100, R115, R116, R89, R90, R94, R95, R98: DIS (none) -> DigiKey; DPN (none) -> RMCF0603FT100RCT-ND; MFR (none) -> Stackpole Electronics; MPN (none) -> RMCF0603FT100R
- R102, R103: DIS (none) -> DigiKey; DPN (none) -> RMCF0603FT665KCT-ND; MFR (none) -> Stackpole Electronics; MPN (none) -> RMCF0603FT665K

Commit message: Commit because I was told to
Also fixed a lot of things
Connections:
- net VPD is gone; now on net VPD-Q3: C18.1, C21.1, C24.1, R101.1, R106.2, R109.2, R110.2, R89.1, R91.1, R97.1, TP38.1, U12.14 (V+), U13.5 (VDD), U14.5 (VDD)
Other:
- moved on the sheet: C18, C21, C22, C23, Q11A, Q11B, R102, R103, R107, R108, R109, R110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

Commit message: Schematic and layout polishing and prep for fabrication
Updated schematic symbols, cleaned up schematic pages to be more like protocard, removed uncessessary TPs, updated layout, cleaned up layout routing and some zones, added Makefile and READMEs for fabrication. Only BOM formatting left!
Parts:
- removed TP42, TP43, TP44: Test-Point, oresat-misc:TestPoint-0.75mm-th, symbol oresat-misc:Test-Point-0.75mm-th
- D7, D9: symbol Device:LED -> Device:LED_Small_Filled
- R124: value 0 -> 10k
- R126: value 0 -> 10k; now fitted
- R89: value 100 -> 10; DPN RMCF0603FT100RCT-ND -> (none); MPN RMCF0603FT100R -> (none)
- U15: DIS (none) -> DigiKey; DPN (none) -> 296-24304-1-ND; MFR (none) -> Texas Instruments; MPN (none) -> TS5A21366DCUR
Other:
- note added: "250 ms inhibit on power up"
- note added: "Allows ~ 4.0 A continuous"
- note added: "Circuit breaker switch with ~10 ms soft start"
- note added: "Main Power Switch Vbus = (6.0, 7.2, 8.4) V"
- note added: "ON/~{OFF} signal powers MAX4211 + TS5A Saves quiescent OPD power draw"
- note added: "RW Q3 has OPD Address 0x22"
- note added: "UART switch"
- note removed: "(3.3V)"
- note removed: "Address selection for Card (See MAX7310 datasheet)"
- note removed: "CLEANUP - CHANGE: all VPD to VPD-Qn VBUSP to VBUSP-Qn BOOT_CONFIG to BOOTCFG-Qn SW-COM1 to RW-UART-TX-Qn SW-COM2 to RW-UART-RX-Qn Fit in sheet boundaries"
- note removed: "FIXME - ?A"
- note removed: "Main Power Switch"
- note removed: "OPD Address 0x1A"
- note removed: "To MCXN digitally configued boot pin"
- note removed: "Vbus = (6.0,7.2,8.4)V"
- moved on the sheet: C25, C26, Q12, Q13, R111, R112, R113, R114, R115, R116, R130, R132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

Commit message: Better BOM
Parts:
- C18, C21, C24, C26: DIS (none) -> DigiKey; DPN (none) -> 399-6856-1-ND; MFR (none) -> KEMET; MPN (none) -> C0603C104K5RACAUTO
- C22, C23, C25, C27: DIS (none) -> DigiKey; DPN (none) -> 490-GRT188R71E105KE13DCT-ND; MFR (none) -> Murata Electronics; MPN (none) -> GRT188R71E105KE13D
- C30: DIS (none) -> DigiKey; DPN (none) -> 399-12983-1-ND; MFR (none) -> KEMET; MPN (none) -> C0603C103J5RACAUTO
- C31: DIS (none) -> DigiKey; DPN (none) -> 399-C0603C474K3RACAUTOCT-ND; MFR (none) -> KEMET; MPN (none) -> C0603C474K3RACAUTO
- D7: DIS (none) -> DigiKey; DPN (none) -> 732-150060AS75000CT-ND; MFR (none) -> Wurth; MPN (none) -> 150060AS75000
- D9: DIS (none) -> DigiKey; DPN (none) -> 732-4971-1-ND; MFR (none) -> Wurth; MPN (none) -> 150060GS75000
- Q11, U12: DIS Digi-Key -> DigiKey
- Q12, Q15: DIS Digi-Key -> DigiKey; DPN 1727-2307-1-ND -> 31-DMN3028LQ-7CT-ND; MFR Nexperia -> Diodes Inc.; MPN PMV45EN2R -> DMN3028LQ-7
- Q13, Q14: DIS Digi-Key -> DigiKey; DPN DMP3050LVT-7DICT-ND -> 31-DMP2035UQ-7CT-ND; MPN DMP3050LVT-7 -> DMP2035UQ-7
- R106, R111, R112, R114, R118, R122, R124, R126, R127, R128, R129, R130, R132: DIS (none) -> DigiKey; DPN (none) -> RMCF0603FT10K0CT-ND; MFR (none) -> Stackpole Electronics; MPN (none) -> RMCF0603FT10K0
- R107, R108: DIS (none) -> DigiKey; DPN (none) -> RMCF0603FT330KCT-ND; MFR (none) -> Stackpole Electronics; MPN (none) -> RMCF0603FT330K
- R109, R110: DIS (none) -> DigiKey; DPN (none) -> RMCF0603FT1M00CT-ND; MFR (none) -> Stackpole Electronics; MPN (none) -> RMCF0603FT1M00
- R113: DIS (none) -> DigiKey; DPN (none) -> RMCF0603FT4K70CT-ND; MFR (none) -> Stackpole Electronics; MPN (none) -> RMCF0603FT4K70
- R117: DIS (none) -> DigiKey; DPN (none) -> RMCF0603FT100KCT-ND; MFR (none) -> Stackpole Electronics; MPN (none) -> RMCF0603FT100K
- R119: DIS (none) -> DigiKey; DPN (none) -> 738-CSS0805FT15L0CT-ND; MFR (none) -> Stackpole Electronics; MPN (none) -> CSS0805FT15L0
- R123: DIS (none) -> DigiKey; DPN (none) -> RMCF0603ZT0R00CT-ND; MFR (none) -> Stackpole Electronics; MPN (none) -> RMCF0603ZT0R00
- R89: DPN (none) -> RMCF0603FT10R0CT-ND; MPN (none) -> RMCF0603FT10R0
- U13, U14: DIS (none) -> DigiKey; DPN (none) -> 576-2927-1-ND; MFR (none) -> Microchip; MPN (none) -> MIC842LYC5-TR
- U16: DIS Digi-Key -> DigiKey; MFR Maxim -> Analog Devices

Commit message: Fixed a few small BOM issues, checked everything, ready for fab.
Parts:
- Q11: MPN DMP2240UDM -> DMP2240UDM-7
Changed lines of the file:
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@@
 			)
 		)
-		(property "Datasheet" "~"
+		(property "Datasheet" "https://www.diodes.com/assets/Datasheets/ds31197.pdf"
 			(at 58.42 182.88 0)
 			(effects
@@
 			)
 		)
-		(property "Description" "Dual PMOS transistor, 6 pin package"
+		(property "Description" "Mosfet Array 2 P-Channel (Dual) 20V 2A 600mW Surface Mount SOT-26"
 			(at 58.42 184.15 0)
 			(effects
@@
 			)
 		)
-		(property "MPN" "DMP2240UDM"
+		(property "MPN" "DMP2240UDM-7"
 			(at 58.42 184.15 0)
 			(effects
@@
 			)
 		)
-		(property "Datasheet" "~"
+		(property "Datasheet" "https://www.diodes.com/assets/Datasheets/ds31197.pdf"
 			(at 58.42 227.33 0)
 			(effects
@@
 			)
 		)
-		(property "Description" "Dual PMOS transistor, 6 pin package"
+		(property "Description" "Mosfet Array 2 P-Channel (Dual) 20V 2A 600mW Surface Mount SOT-26"
 			(at 58.42 228.6 0)
 			(effects
@@
 			)
 		)
-		(property "MPN" "DMP2240UDM"
+		(property "MPN" "DMP2240UDM-7"
 			(at 58.42 228.6 0)
 			(effects

Commit message: Sent off for fabrication.
Last sweep of BOM, ground stitching, and inner layer planes. Lots of small tweaks.
Parts:
- Q11: value DMP2240UDM -> DMP2240UDM-7
- Q12, Q15: value PMV45EN -> DMN3028LQ-7
- Q13, Q14: value DMP3050LVT-7 -> DMPH2040UVTQ-7; DPN 31-DMP2035UQ-7CT-ND -> 31-DMPH2040UVTQ-7CT-ND; MFR Diodes Inc -> Diodes Incorporated; MPN DMP2035UQ-7 -> DMPH2040UVTQ-7
Other:
- moved on the sheet: C18, C21, C22, C23, C24, C25, C26, C27, C30, C31, D7, D9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

Commit message: Fix BOM - some packages were wrong size, caught by CM.
Parts:
- R119: DPN 738-CSS0805FT15L0CT-ND -> CSNL1206FT15L0CT-ND; MPN CSS0805FT15L0 -> CSNL1206FT15L0
Changed lines of the file:
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@@
 			)
 		)
-		(property "Datasheet" "https://www.seielect.com/catalog/SEI-CSS_CSSH.PDF"
+		(property "Datasheet" "https://www.seielect.com/catalog/SEI-CSNL.pdf"
 			(at 273.05 39.37 0)
 			(effects
@@
 			)
 		)
-		(property "Description" "15 mOhms ±1% 0.5W, 1/2W Chip Resistor 0805 (2012 Metric) Automotive AEC-Q200, Current Sense Metal Element"
+		(property "Description" "15 mOhms ±1% 1W Chip Resistor 1206 (3216 Metric) Current Sense, Moisture Resistant Metal Element"
 			(at 273.05 39.37 0)
 			(effects
@@
 			)
 		)
-		(property "DPN" "738-CSS0805FT15L0CT-ND"
+		(property "DPN" "CSNL1206FT15L0CT-ND"
 			(at 273.05 39.37 90)
 			(effects
@@
 			)
 		)
-		(property "MPN" "CSS0805FT15L0"
+		(property "MPN" "CSNL1206FT15L0"
 			(at 273.05 39.37 90)
 			(effects
