File: oresat-rw-card/oresat-rw-card-sch-q4.kicad_sch (KiCad schematic)
At the start: 78 parts, among them Q16 DMP2240UDM, Q17 PMV45EN, Q18 DMP3050LVT-7, Q19 DMP3050LVT-7, Q20 PMV45EN, U19 MAX7310, U20 MIC842LYC5, U21 MIC842LYC5, U22 TS5A21366DCUR, U23 MAX4211FETE

Commit message: Design review on current state of sch/brd
Parts:
- R133, R134, R138, R139, R142, R148, R159, R160: DIS (none) -> DigiKey; DPN (none) -> RMCF0603FT100RCT-ND; MFR (none) -> Stackpole Electronics; MPN (none) -> RMCF0603FT100R
- R146, R147: DIS (none) -> DigiKey; DPN (none) -> RMCF0603FT665KCT-ND; MFR (none) -> Stackpole Electronics; MPN (none) -> RMCF0603FT665K

Commit message: Commit because I was told to
Also fixed a lot of things
Connections:
- net VPD is gone; now on net VPD-Q4: C28.1, C29.1, C35.1, R133.1, R135.1, R141.1, R145.1, R150.2, R153.2, R154.2, TP56.1, U19.14 (V+), U20.5 (VDD), U21.5 (VDD)
Other:
- moved on the sheet: C28, C29, C33, C34, Q16A, Q16B, R138, R139, R146, R147, R151, R152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

Commit message: Schematic and layout polishing and prep for fabrication
Updated schematic symbols, cleaned up schematic pages to be more like protocard, removed uncessessary TPs, updated layout, cleaned up layout routing and some zones, added Makefile and READMEs for fabrication. Only BOM formatting left!
Parts:
- removed TP60, TP61, TP62: Test-Point, oresat-misc:TestPoint-0.75mm-th, symbol oresat-misc:Test-Point-0.75mm-th
- D10, D12: symbol Device:LED -> Device:LED_Small_Filled
- R133: value 100 -> 10; DPN RMCF0603FT100RCT-ND -> (none); MPN RMCF0603FT100R -> (none)
- R168: value 0 -> 10k
- R170: value 0 -> 10k; now fitted
- U22: DIS (none) -> DigiKey; DPN (none) -> 296-24304-1-ND; MFR (none) -> Texas Instruments; MPN (none) -> TS5A21366DCUR
Connections:
- net OPD_PWR: now also R133.1; no longer R133.2
- net VPD-Q4: now also R133.2; no longer R133.1
Other:
- note added: "250 ms inhibit on power up"
- note added: "Allows ~ 4.0 A continuous"
- note added: "Circuit breaker switch with ~10 ms soft start"
- note added: "Main Power Switch Vbus = (6.0, 7.2, 8.4) V"
- note added: "ON/~{OFF} signal powers MAX4211 + TS5A Saves quiescent OPD power draw"
- note added: "RW Q4 has OPD Address 0x23"
- note added: "UART switch"
- note removed: "(3.3V)"
- note removed: "Address selection for Card (See MAX7310 datasheet)"
- note removed: "CLEANUP - CHANGE: all VPD to VPD-Qn VBUSP to VBUSP-Qn BOOT_CONFIG to BOOTCFG-Qn SW-COM1 to RW-UART-TX-Qn SW-COM2 to RW-UART-RX-Qn Fit in sheet boundaries"
- note removed: "FIXME - ?A"
- note removed: "Main Power Switch"
- note removed: "OPD Address 0x1A"
- note removed: "To MCXN digitally configued boot pin"
- note removed: "Vbus = (6.0,7.2,8.4)V"
- moved on the sheet: C36, C37, Q17, Q18, R133, R156, R157, R158, R159, R160, R174, R176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

Commit message: Better BOM
Parts:
- C28, C29, C35, C37: DIS (none) -> DigiKey; DPN (none) -> 399-6856-1-ND; MFR (none) -> KEMET; MPN (none) -> C0603C104K5RACAUTO
- C33, C34, C36, C38: DIS (none) -> DigiKey; DPN (none) -> 490-GRT188R71E105KE13DCT-ND; MFR (none) -> Murata Electronics; MPN (none) -> GRT188R71E105KE13D
- C41: DIS (none) -> DigiKey; DPN (none) -> 399-12983-1-ND; MFR (none) -> KEMET; MPN (none) -> C0603C103J5RACAUTO
- C42: DIS (none) -> DigiKey; DPN (none) -> 399-C0603C474K3RACAUTOCT-ND; MFR (none) -> KEMET; MPN (none) -> C0603C474K3RACAUTO
- D10: DIS (none) -> DigiKey; DPN (none) -> 732-150060AS75000CT-ND; MFR (none) -> Wurth; MPN (none) -> 150060AS75000
- D12: DIS (none) -> DigiKey; DPN (none) -> 732-4971-1-ND; MFR (none) -> Wurth; MPN (none) -> 150060GS75000
- Q16, U19: DIS Digi-Key -> DigiKey
- Q17, Q20: DIS Digi-Key -> DigiKey; DPN 1727-2307-1-ND -> 31-DMN3028LQ-7CT-ND; MFR Nexperia -> Diodes Inc.; MPN PMV45EN2R -> DMN3028LQ-7
- Q18, Q19: DIS Digi-Key -> DigiKey; DPN DMP3050LVT-7DICT-ND -> 31-DMP2035UQ-7CT-ND; MPN DMP3050LVT-7 -> DMP2035UQ-7
- R133: DPN (none) -> RMCF0603FT10R0CT-ND; MPN (none) -> RMCF0603FT10R0
- R150, R155, R156, R158, R162, R166, R168, R170, R171, R172, R173, R174, R176: DIS (none) -> DigiKey; DPN (none) -> RMCF0603FT10K0CT-ND; MFR (none) -> Stackpole Electronics; MPN (none) -> RMCF0603FT10K0
- R151, R152: DIS (none) -> DigiKey; DPN (none) -> RMCF0603FT330KCT-ND; MFR (none) -> Stackpole Electronics; MPN (none) -> RMCF0603FT330K
- R153, R154: DIS (none) -> DigiKey; DPN (none) -> RMCF0603FT1M00CT-ND; MFR (none) -> Stackpole Electronics; MPN (none) -> RMCF0603FT1M00
- R157: DIS (none) -> DigiKey; DPN (none) -> RMCF0603FT4K70CT-ND; MFR (none) -> Stackpole Electronics; MPN (none) -> RMCF0603FT4K70
- R161: DIS (none) -> DigiKey; DPN (none) -> RMCF0603FT100KCT-ND; MFR (none) -> Stackpole Electronics; MPN (none) -> RMCF0603FT100K
- R163: DIS (none) -> DigiKey; DPN (none) -> 738-CSS0805FT15L0CT-ND; MFR (none) -> Stackpole Electronics; MPN (none) -> CSS0805FT15L0
- R167: DIS (none) -> DigiKey; DPN (none) -> RMCF0603ZT0R00CT-ND; MFR (none) -> Stackpole Electronics; MPN (none) -> RMCF0603ZT0R00
- U20, U21: DIS (none) -> DigiKey; DPN (none) -> 576-2927-1-ND; MFR (none) -> Microchip; MPN (none) -> MIC842LYC5-TR
- U23: DIS Digi-Key -> DigiKey; MFR Maxim -> Analog Devices

Commit message: Fixed a few small BOM issues, checked everything, ready for fab.
Parts:
- Q16: MPN DMP2240UDM -> DMP2240UDM-7
Changed lines of the file:
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@@
 			)
 		)
-		(property "Datasheet" "~"
+		(property "Datasheet" "https://www.diodes.com/assets/Datasheets/ds31197.pdf"
 			(at 59.69 184.15 0)
 			(effects
@@
 			)
 		)
-		(property "Description" "Dual PMOS transistor, 6 pin package"
+		(property "Description" "Mosfet Array 2 P-Channel (Dual) 20V 2A 600mW Surface Mount SOT-26"
 			(at 59.69 185.42 0)
 			(effects
@@
 			)
 		)
-		(property "MPN" "DMP2240UDM"
+		(property "MPN" "DMP2240UDM-7"
 			(at 59.69 185.42 0)
 			(effects
@@
 			)
 		)
-		(property "Datasheet" "~"
+		(property "Datasheet" "https://www.diodes.com/assets/Datasheets/ds31197.pdf"
 			(at 59.69 228.6 0)
 			(effects
@@
 			)
 		)
-		(property "Description" "Dual PMOS transistor, 6 pin package"
+		(property "Description" "Mosfet Array 2 P-Channel (Dual) 20V 2A 600mW Surface Mount SOT-26"
 			(at 59.69 229.87 0)
 			(effects
@@
 			)
 		)
-		(property "MPN" "DMP2240UDM"
+		(property "MPN" "DMP2240UDM-7"
 			(at 59.69 229.87 0)
 			(effects

Commit message: Sent off for fabrication.
Last sweep of BOM, ground stitching, and inner layer planes. Lots of small tweaks.
Parts:
- Q16: value DMP2240UDM -> DMP2240UDM-7
- Q17, Q20: value PMV45EN -> DMN3028LQ-7
- Q18, Q19: value DMP3050LVT-7 -> DMPH2040UVTQ-7; DPN 31-DMP2035UQ-7CT-ND -> 31-DMPH2040UVTQ-7CT-ND; MFR Diodes Inc -> Diodes Incorporated; MPN DMP2035UQ-7 -> DMPH2040UVTQ-7
Other:
- moved on the sheet: C28, C29, C33, C34, C35, C36, C37, C38, C41, C42, D10, D12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

Commit message: Fix BOM - some packages were wrong size, caught by CM.
Parts:
- R163: DPN 738-CSS0805FT15L0CT-ND -> CSNL1206FT15L0CT-ND; MPN CSS0805FT15L0 -> CSNL1206FT15L0
Changed lines of the file:
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@@
 			)
 		)
-		(property "Datasheet" "https://www.seielect.com/catalog/SEI-CSS_CSSH.PDF"
+		(property "Datasheet" "https://www.seielect.com/catalog/SEI-CSNL.pdf"
 			(at 273.05 39.37 0)
 			(effects
@@
 			)
 		)
-		(property "Description" "15 mOhms ±1% 0.5W, 1/2W Chip Resistor 0805 (2012 Metric) Automotive AEC-Q200, Current Sense Metal Element"
+		(property "Description" "15 mOhms ±1% 1W Chip Resistor 1206 (3216 Metric) Current Sense, Moisture Resistant Metal Element"
 			(at 273.05 39.37 0)
 			(effects
@@
 			)
 		)
-		(property "DPN" "738-CSS0805FT15L0CT-ND"
+		(property "DPN" "CSNL1206FT15L0CT-ND"
 			(at 273.05 39.37 90)
 			(effects
@@
 			)
 		)
-		(property "MPN" "CSS0805FT15L0"
+		(property "MPN" "CSNL1206FT15L0"
 			(at 273.05 39.37 90)
 			(effects
